File: Nosecone/Nose Board.sch (KiCad schematic (older format))
At the start: 41 parts, among them J1 Conn_01x02, J2 Conn_01x06, J3 Conn_02x03_Odd_Even, J4 Conn_01x04, Q1 Q_PMOS_DGS, Q2 Q_PMOS_DGS, U1 RS485_converter_ISL83488, U10 MS5803-14BA, U11 MS5803-14BA, U2 ATXMEGA16A4U-AU, U3 3.3V_DCDC_Conv_TPS62056DGS, U4 GPS_UBX_CAM_M8C, U5 GPS_UBX_CAM_M8C, U6 XBEE, U7 OpenLog, U8 BNO055, U9 LTC4412

Commit message: PCB Routed
Parts:
- removed J2: Conn_01x06, Pin_Headers:Pin_Header_Straight_1x06_Pitch1.27mm, symbol Conn_01x06
- removed J4: Conn_01x04, Pin_Headers:Pin_Header_Straight_1x04_Pitch1.27mm, symbol Conn_01x04
- removed U5: GPS_UBX_CAM_M8C, Misc components:UBX_CAM-M8C, symbol GPS_UBX_CAM_M8C
- added C11: 4.7uF, Capacitors_SMD:C_0603_HandSoldering, symbol C
- added J2: Conn_02x04_Odd_Even, Connectors_JST:JST_PUD_B08B-PUDSS_2x04x2.00mm_Straight, symbol Conn_02x04_Odd_Even
- added J4: Conn_Coaxial, Connectors:SMA_THT_Jack_Straight, symbol Conn_Coaxial
- added R11, R12: 220, Resistors_SMD:R_0603_HandSoldering, symbol R
- added U12, U13, U5: Via-stitch, Misc components:Small-via, symbol Via-stitch
Connections:
- net GPS2_EXTINT is gone; now on net IMU_INT: U2.21 (PD1/OC0B/XCK0)
- net +3V3: now also C11.1
- net GND: now also C11.2, J2.2 (Pin_2), J4.2 (Ext), U12.1 (TO-STITCH), U13.1 (TO-STITCH), U5.1 (TO-STITCH)
- net GPS1_RXD: now also R12.2; no longer U4.26 (RXD/SPI_MOSI)
- net GPS1_TXD: now also R11.2; no longer U4.25 (TXD/SPI_MISO)
- net IMU_INT: no longer U2.3 (AC0OUT/AC7/ADC7/PA7)
- net VBUS: now also J2.1 (Pin_1)
- net at U1.5 (Y): now also J2.6 (Pin_6)
- net at U1.6 (Z): now also J2.5 (Pin_5)
- net at U1.7 (B): now also J2.4 (Pin_4)
- net at U1.8 (A): now also J2.3 (Pin_3)
- net at U4.16 (RF_OUT): no longer U4.17 (RF_IN)
- net GPS2_PPS: no longer names the net of U2.29 (PE1/OC0B/XCK0/SCL)
- net GPS2_RXD renamed Debug_TX
- net Debug_TX: now also J2.7 (Pin_7)
- net GPS2_TXD renamed Debug_RX
- net Debug_RX: now also J2.8 (Pin_8)
- new net: J4.1 (In), U4.17 (RF_IN)
- new net: R11.1, U4.25 (TXD/SPI_MISO)
- new net: R12.1, U4.26 (RXD/SPI_MOSI)
Other:
- note removed: "Serial Debug Connection"
- moved on the sheet: U1, U4

Commit message: Minor board adjustments, BoM work
Parts:
- added BZ1: Buzzer, Misc components:Buzzer-CUI_CEP-2242, symbol Buzzer
- added J5: Conn_01x02, Pin_Headers:Pin_Header_Straight_1x02_Pitch2.54mm, symbol Conn_01x02
- C1, C2, C3: value C -> 100nF
- C7: footprint Capacitors_SMD:C_0603_HandSoldering -> Capacitors_SMD:C_0805_HandSoldering
- C8: value C -> 22uF
- J1: footprint Pin_Headers:Pin_Header_Straight_1x02_Pitch1.27mm -> Connectors_JST:JST_PH_B2B-PH-K_02x2.00mm_Straight
- R1: value R -> 90.9k
- R2: value R -> 10k
- R6, R7: value R -> 220
Connections:
- net GND: now also BZ1.2 (+)
- net Buzzer_drive: now reaches U2.29 (PE1/OC0B/XCK0/SCL)
- net Buzzer_drive: now also BZ1.1 (-)
- net A1: now reaches U2.41 (AC1/ADC1/PA1)
- net A1: now also J5.1 (Pin_1)
- net A2: now reaches U2.42 (AC2/ADC2/PA2)
- net A2: now also J5.2 (Pin_2)
