File: Middle Board/Middle Board.sch (KiCad schematic (older format))
At the start: 4 parts

Commit message: Finished GNC section schematic
Still need to find digikey part numbers
Parts:
- removed U?: ATXMEGA128A4U-AU, TQFP44, symbol ATXMEGA128A4U-AU
- added C?: 4.7 uF, symbol C_Small
- added C? (x12): 100 nF, symbol C_Small
- added C?: 2.2 uF, symbol C_Small
- added J?: JTAG Connector, symbol Conn_02x05_Odd_Even
- added R? (x4): 100k, symbol R
- added R? (x2): 39, symbol R
- added R? (x2): 10k, symbol R
- added SW?: SW_SPST, symbol SW_SPST
Connections:
- net labels added: +3V3, BNO055_RST, GNC_RX, GNC_TX, GND, SCL, SDA, TCK, TDI, TDO, TMS, nRST
- wire segments 0 -> 89
- no-connect marks 0 -> 8
Other:
- moved on the sheet: U?
