File: Middle Board/_saved_Middle Board.sch (KiCad schematic (older format))
At the start: 40 parts, among them J1 JTAG Connector, SW1 SW_SPST, U1 ATSAMG55, U2 BNO055_Breakout, U3 MS5803, U4 XBee_PRO_SX

Commit message: Added XBee to Mainboard
Parts:
- added D? (x2): LED_R, symbol LED
- added D?: LED_G, symbol LED
- added D?: LED_B, symbol LED
- added R? (x4): 270, symbol R
- gave numbers to parts that had none: 4
- renumbered R9 to R10, R10 to R11, R11 to R12, U4 to U5
Connections:
- net +3V3: now also D?.2 (A), D?.2 (A), D?.2 (A), D?.2 (A)
- net GND: now also R?.2
- net at U1.6 (PA0): now also R?.2
- net at U1.61 (PA2): now also R?.2
- net at U1.7 (PA1): now also R?.2
- new net: D?.1 (K), R?.1 (x4)
Other:
- note added: "50 Ω"
- note added: "Might need more antenna connectors, 2 might not be enough\n"

Commit message: Added GPS to mainboard schematic
Went with a different GPS module than the one Daniel picked out since
we're going with external antennas
Parts:
- added BT?: CR_1220, symbol Battery_Cell
- added FL?: B39162B3520U410, symbol B39162B3520U410
- added J? (x2): Conn_Coaxial, symbol Conn_Coaxial
- added R?: 100, symbol R
- added U?: PD0922J5050S2HF, symbol PD0922J5050S2HF
- added U?: UBX_NEO_M8Q, symbol UBX_NEO_M8Q
- gave numbers to parts that had none: 8
- renumbered D1 to D5, D2 to D6, D3 to D7, R6 to R10, R7 to R11, R8 to R12, R9 to R13, R10 to R14, R11 to R15, R12 to R16, R1 to R5, R2 to R6, R3 to R7, R4 to R8, R5 to R9
Connections:
- net GND: now also BT?.2 (-), FL?.1 (GND), FL?.3 (GND), FL?.4 (GND), FL?.6 (GND), J?.2 (Ext), J?.2 (Ext), U?.10 (GND), U?.12 (GND), U?.13 (GND), U?.24 (GND)
- net XBEE_RF_50Ω: now reaches U4.1, U5.36 (RF_PAD)
- net ANT1_RF_50Ω: now reaches J2.1 (In), R13.1, U4.2
- net ANT2_RF_50Ω: now reaches J3.1 (In), R13.2, U4.3
- new net: BT?.1 (+), U?.22 (V_BCKP)
- new net ANT3_RF_50Ω: J?.1 (In), R?.1, U?.2
- new net ANT4_RF_50Ω: J?.1 (In), R?.2, U?.3
- new net GPS_FILT_RF_50Ω: FL?.2 (IN), U?.1
- new net GPS_RF_50Ω: FL?.5 (OUT), U?.11 (RF_IN)
Other:
- note removed: "50 Ω"
- moved on the sheet: C1, C10, C11, C12, C13, C14, C15, C16, C2, C3, C4, C5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

Commit message: Small changes
Parts:
- added R18, R19: 20, symbol R
- gave numbers to parts that had none: 7
Connections:
- net +3V3: now also U7.23 (VCC)
- net GND: now also U7.7 (VDD_USB)
- net at U7.20 (TxD): now also R18.1
- net at U7.21 (RxD): now also R19.1
- new net GPS_RX: R19.2
- new net GPS_TX: R18.2
- no-connect marks 24 -> 34
Other:
- moved on the sheet: BT1, FL1, J4, J5, R17, U6, U7

Commit message: Apparently I forgot to save everything earlier
Connections:
- net GND: now also C14.2, U3.2 (GND), U3.3 (CSB)
Changed lines of the file:
@@
 NoConn ~ 4000 19050
 NoConn ~ 4000 19150
+$Comp
+L GND #PWR?
+U 1 1 5A716165
+P 4150 14450
+F 0 "#PWR?" H 4150 14200 50  0001 C CNN
+F 1 "GND" H 4150 14300 50  0000 C CNN
+F 2 "" H 4150 14450 50  0001 C CNN
+F 3 "" H 4150 14450 50  0001 C CNN
+	1    4150 14450
+	1    0    0    -1
+$EndComp
 $EndSCHEMATC
