File: Control Board/Control Board.sch (KiCad schematic (older format))
At the start: 93 parts, among them J1 Conn_02x10_Odd_Even, J10 Conn_01x03, J11 Conn_01x03, J12 RJ45, J13 Conn_01x03, J14 Conn_01x03, J15 Conn_01x03, J2 Conn_02x03_Odd_Even, J3 RJ45, J4 Conn_01x02, J5 Conn_01x02, J6 Conn_01x03, J7 Conn_01x02, J8 Conn_01x02, J9 Conn_01x02, Q1 STS4DNF60L, U1 ATXMEGA128A3-AU, U10 OPENLOG, U2 LT1797, U3 LT1797, U4 ISL83490, U5 MAX31856, U6 MAX31856, U7 MAX31856, U8 MAX31856, U9 MAX31856

Commit message: Added digikey part numbers
Parts:
- J10, J11, J13, J14, J15, J6: Digikey Part Number (none) -> 455-1720-ND
- J12, J3: Digikey Part Number (none) -> RJHSE-5080-ND
- J4, J5, J7, J8, J9: Digikey Part Number (none) -> 455-1719-ND
- U10: Digikey Part Number (none) -> 1568-1368-ND
Changed lines of the file:
@@
 F 2 "Custom Footprints:OpenLog" H 8900 14400 50  0001 C CNN
 F 3 "" H 8900 14400 50  0001 C CNN
+F 4 "1568-1368-ND" H 0   0   50  0001 C CNN "Digikey Part Number"
 	1    9050 14400
 	1    0    0    -1
@@
 F 2 "Connectors:RJ45_8" H 12150 12200 50  0001 C CNN
 F 3 "" H 12150 12200 50  0001 C CNN
+F 4 "RJHSE-5080-ND" H 0   0   50  0001 C CNN "Digikey Part Number"
 	1    12150 12200
 	1    0    0    -1
@@
 F 2 "Connectors:RJ45_8" H 12150 14250 50  0001 C CNN
 F 3 "" H 12150 14250 50  0001 C CNN
+F 4 "RJHSE-5080-ND" H 0   0   50  0001 C CNN "Digikey Part Number"
 	1    12150 14250
 	1    0    0    -1
@@
 F 2 "Connectors_JST:JST_PH_S2B-PH-K_02x2.00mm_Angled" H 14300 12450 50  0001 C CNN
 F 3 "~" H 14300 12450 50  0001 C CNN
+F 4 "455-1719-ND" H 0   0   50  0001 C CNN "Digikey Part Number"
 	1    14300 12450
 	1    0    0    -1
@@
 F 2 "Connectors_JST:JST_PH_S2B-PH-K_02x2.00mm_Angled" H 14300 12650 50  0001 C CNN
 F 3 "~" H 14300 12650 50  0001 C CNN
+F 4 "455-1719-ND" H 0   0   50  0001 C CNN "Digikey Part Number"
 	1    14300 12650
 	1    0    0    -1
@@
 F 2 "Connectors_JST:JST_PH_S2B-PH-K_02x2.00mm_Angled" H 14300 12850 50  0001 C CNN
 F 3 "~" H 14300 12850 50  0001 C CNN
+F 4 "455-1719-ND" H 0   0   50  0001 C CNN "Digikey Part Number"
 	1    14300 12850
 	1    0    0    -1
@@
 F 2 "Connectors_JST:JST_PH_S2B-PH-K_02x2.00mm_Angled" H 14300 13050 50  0001 C CNN
 F 3 "~" H 14300 13050 50  0001 C CNN
+F 4 "455-1719-ND" H 0   0   50  0001 C CNN "Digikey Part Number"
 	1    14300 13050
 	1    0    0    -1
@@
 F 2 "Connectors_JST:JST_PH_S2B-PH-K_02x2.00mm_Angled" H 14300 13250 50  0001 C CNN
 F 3 "~" H 14300 13250 50  0001 C CNN
+F 4 "455-1719-ND" H 0   0   50  0001 C CNN "Digikey Part Number"
 	1    14300 13250
 	1    0    0    -1
@@
 F 2 "Connectors_JST:JST_PH_S3B-PH-K_03x2.00mm_Angled" H 15850 15450 50  0001 C CNN
 F 3 "~" H 15850 15450 50  0001 C CNN
+F 4 "455-1720-ND" H 0   0   50  0001 C CNN "Digikey Part Number"
 	1    15850 15450
 	1    0    0    -1
@@
 F 2 "Connectors_JST:JST_PH_S3B-PH-K_03x2.00mm_Angled" H 15850 14550 50  0001 C CNN
 F 3 "~" H 15850 14550 50  0001 C CNN
+F 4 "455-1720-ND" H 0   0   50  0001 C CNN "Digikey Part Number"
 	1    15850 14550
 	1    0    0    -1
@@
 F 2 "Connectors_JST:JST_PH_S3B-PH-K_03x2.00mm_Angled" H 15850 14150 50  0001 C CNN
 F 3 "~" H 15850 14150 50  0001 C CNN
+F 4 "455-1720-ND" H 0   0   50  0001 C CNN "Digikey Part Number"
 	1    15850 14150
 	1    0    0    -1
@@
 F 2 "Connectors_JST:JST_PH_S3B-PH-K_03x2.00mm_Angled" H 15850 15050 50  0001 C CNN
 F 3 "~" H 15850 15050 50  0001 C CNN
+F 4 "455-1720-ND" H 0   0   50  0001 C CNN "Digikey Part Number"
 	1    15850 15050
 	1    0    0    -1
@@
 F 2 "Connectors_JST:JST_PH_S2B-PH-K_02x2.00mm_Angled" H 16300 12800 50  0001 C CNN
 F 3 "~" H 16300 12800 50  0001 C CNN
+F 4 "455-1720-ND" H 0   0   50  0001 C CNN "Digikey Part Number"
 	1    16300 12800
 	-1   0    0    1
@@
 F 2 "Connectors_JST:JST_PH_S3B-PH-K_03x2.00mm_Angled" H 16300 13350 50  0001 C CNN
 F 3 "~" H 16300 13350 50  0001 C CNN
+F 4 "455-1720-ND" H 0   0   50  0001 C CNN "Digikey Part Number"
 	1    16300 13350
 	-1   0    0    1

Commit message: More changes
Parts:
- removed J12: RJ45, Connectors:RJ45_8, symbol Connector:RJ45
- added H1, H2, H3, H4: Mounting_Hole, Mounting_Holes:MountingHole_3.2mm_M3, symbol Mechanical:Mounting_Hole
- added SYM1: SYM_Arrow45_Large, Custom Parts:Logo_v3, symbol Graphic:SYM_Arrow45_Large
- J10, J11, J13, J14, J15: footprint Connectors_JST:JST_PH_S3B-PH-K_03x2.00mm_Angled -> Connectors_JST:JST_PH_B3B-PH-K_03x2.00mm_Straight
- J4, J5, J7, J8, J9: footprint Connectors_JST:JST_PH_S2B-PH-K_02x2.00mm_Angled -> Connectors_JST:JST_PH_B2B-PH-K_02x2.00mm_Straight
- J6: footprint Connectors_JST:JST_PH_S2B-PH-K_02x2.00mm_Angled -> Connectors_JST:JST_PH_B3B-PH-K_03x2.00mm_Straight
Other:
- note added: "Needs Crossover Cable"
- note removed: "Aft board only"
- note removed: "Middle board only"
Changed lines of the file:
@@
 $EndComp
 Text Notes 11750 11550 0    50   ~ 0
-Middle board only
-Text Label 11800 14700 3    60   ~ 0
-BOARD_RX+
-Text Label 12000 14700 3    60   ~ 0
-BOARD_TX+
-Text Label 11900 14700 3    60   ~ 0
-BOARD_RX-
-Text Label 12300 14700 3    60   ~ 0
-BOARD_TX-
-$Comp
-L power:GND #PWR091
-U 1 1 5AAC768D
-P 12700 13900
-F 0 "#PWR091" H 12700 13650 50  0001 C CNN
-F 1 "GND" V 12700 13700 50  0000 C CNN
-F 2 "" H 12700 13900 50  0001 C CNN
-F 3 "" H 12700 13900 50  0001 C CNN
-	1    12700 13900
-	0    -1   1    0
-$EndComp
-$Comp
-L Connector:RJ45 J12
-U 1 1 5AAC7693
-P 12150 14250
-F 0 "J12" H 12226 14867 50  0000 C CNN
-F 1 "RJ45" H 12226 14776 50  0000 C CNN
-F 2 "Connectors:RJ45_8" H 12150 14250 50  0001 C CNN
-F 3 "" H 12150 14250 50  0001 C CNN
-F 4 "RJHSE-5080-ND" H 0   0   50  0001 C CNN "Digikey Part Number"
-	1    12150 14250
-	1    0    0    -1
-$EndComp
-Text Notes 11750 13600 0    50   ~ 0
-Aft board only
+Needs Crossover Cable
 $Comp
 L Connector:Conn_01x02 J4
@@
 F 0 "J4" H 14380 12442 50  0000 L CNN
 F 1 "Conn_01x02" H 14380 12351 50  0000 L CNN
-F 2 "Connectors_JST:JST_PH_S2B-PH-K_02x2.00mm_Angled" H 14300 12450 50  0001 C CNN
+F 2 "Connectors_JST:JST_PH_B2B-PH-K_02x2.00mm_Straight" H 14300 12450 50  0001 C CNN
 F 3 "~" H 14300 12450 50  0001 C CNN
 F 4 "455-1719-ND" H 0   0   50  0001 C CNN "Digikey Part Number"
@@
 F 0 "J5" H 14380 12642 50  0000 L CNN
 F 1 "Conn_01x02" H 14380 12551 50  0000 L CNN
-F 2 "Connectors_JST:JST_PH_S2B-PH-K_02x2.00mm_Angled" H 14300 12650 50  0001 C CNN
+F 2 "Connectors_JST:JST_PH_B2B-PH-K_02x2.00mm_Straight" H 14300 12650 50  0001 C CNN
 F 3 "~" H 14300 12650 50  0001 C CNN
 F 4 "455-1719-ND" H 0   0   50  0001 C CNN "Digikey Part Number"
@@
 F 0 "J7" H 14380 12842 50  0000 L CNN
 F 1 "Conn_01x02" H 14380 12751 50  0000 L CNN
-F 2 "Connectors_JST:JST_PH_S2B-PH-K_02x2.00mm_Angled" H 14300 12850 50  0001 C CNN
+F 2 "Connectors_JST:JST_PH_B2B-PH-K_02x2.00mm_Straight" H 14300 12850 50  0001 C CNN
 F 3 "~" H 14300 12850 50  0001 C CNN
 F 4 "455-1719-ND" H 0   0   50  0001 C CNN "Digikey Part Number"
@@
 F 0 "J8" H 14380 13042 50  0000 L CNN
 F 1 "Conn_01x02" H 14380 12951 50  0000 L CNN
-F 2 "Connectors_JST:JST_PH_S2B-PH-K_02x2.00mm_Angled" H 14300 13050 50  0001 C CNN
+F 2 "Connectors_JST:JST_PH_B2B-PH-K_02x2.00mm_Straight" H 14300 13050 50  0001 C CNN
 F 3 "~" H 14300 13050 50  0001 C CNN
 F 4 "455-1719-ND" H 0   0   50  0001 C CNN "Digikey Part Number"
@@
 F 0 "J9" H 14380 13242 50  0000 L CNN
 F 1 "Conn_01x02" H 14380 13151 50  0000 L CNN
-F 2 "Connectors_JST:JST_PH_S2B-PH-K_02x2.00mm_Angled" H 14300 13250 50  0001 C CNN
+F 2 "Connectors_JST:JST_PH_B2B-PH-K_02x2.00mm_Straight" H 14300 13250 50  0001 C CNN
 F 3 "~" H 14300 13250 50  0001 C CNN
 F 4 "455-1719-ND" H 0   0   50  0001 C CNN "Digikey Part Number"
@@
 F 0 "J15" H 15930 15492 50  0000 L CNN
 F 1 "Conn_01x03" H 15930 15401 50  0000 L CNN
-F 2 "Connectors_JST:JST_PH_S3B-PH-K_03x2.00mm_Angled" H 15850 15450 50  0001 C CNN
+F 2 "Connectors_JST:JST_PH_B3B-PH-K_03x2.00mm_Straight" H 15850 15450 50  0001 C CNN
 F 3 "~" H 15850 15450 50  0001 C CNN
 F 4 "455-1720-ND" H 0   0   50  0001 C CNN "Digikey Part Number"
@@
 F 0 "J13" H 15930 14592 50  0000 L CNN
 F 1 "Conn_01x03" H 15930 14501 50  0000 L CNN
-F 2 "Connectors_JST:JST_PH_S3B-PH-K_03x2.00mm_Angled" H 15850 14550 50  0001 C CNN
+F 2 "Connectors_JST:JST_PH_B3B-PH-K_03x2.00mm_Straight" H 15850 14550 50  0001 C CNN
 F 3 "~" H 15850 14550 50  0001 C CNN
 F 4 "455-1720-ND" H 0   0   50  0001 C CNN "Digikey Part Number"
@@
 F 0 "J11" H 15930 14192 50  0000 L CNN
 F 1 "Conn_01x03" H 15930 14101 50  0000 L CNN
-F 2 "Connectors_JST:JST_PH_S3B-PH-K_03x2.00mm_Angled" H 15850 14150 50  0001 C CNN
+F 2 "Connectors_JST:JST_PH_B3B-PH-K_03x2.00mm_Straight" H 15850 14150 50  0001 C CNN
 F 3 "~" H 15850 14150 50  0001 C CNN
 F 4 "455-1720-ND" H 0   0   50  0001 C CNN "Digikey Part Number"
@@
 F 0 "J14" H 15930 15092 50  0000 L CNN
 F 1 "Conn_01x03" H 15930 15001 50  0000 L CNN
-F 2 "Connectors_JST:JST_PH_S3B-PH-K_03x2.00mm_Angled" H 15850 15050 50  0001 C CNN
+F 2 "Connectors_JST:JST_PH_B3B-PH-K_03x2.00mm_Straight" H 15850 15050 50  0001 C CNN
 F 3 "~" H 15850 15050 50  0001 C CNN
 F 4 "455-1720-ND" H 0   0   50  0001 C CNN "Digikey Part Number"
@@
 F 0 "J6" H 16220 12475 50  0000 C CNN
 F 1 "Conn_01x03" H 16220 12566 50  0000 C CNN
-F 2 "Connectors_JST:JST_PH_S2B-PH-K_02x2.00mm_Angled" H 16300 12800 50  0001 C CNN
+F 2 "Connectors_JST:JST_PH_B3B-PH-K_03x2.00mm_Straight" H 16300 12800 50  0001 C CNN
 F 3 "~" H 16300 12800 50  0001 C CNN
 F 4 "455-1720-ND" H 0   0   50  0001 C CNN "Digikey Part Number"
@@
 F 0 "J10" H 16220 13025 50  0000 C CNN
 F 1 "Conn_01x03" H 16220 13116 50  0000 C CNN
-F 2 "Connectors_JST:JST_PH_S3B-PH-K_03x2.00mm_Angled" H 16300 13350 50  0001 C CNN
+F 2 "Connectors_JST:JST_PH_B3B-PH-K_03x2.00mm_Straight" H 16300 13350 50  0001 C CNN
 F 3 "~" H 16300 13350 50  0001 C CNN
 F 4 "455-1720-ND" H 0   0   50  0001 C CNN "Digikey Part Number"
@@
 Connection ~ 3650 6200
 Connection ~ 3650 6400
+$Comp
+L Mechanical:Mounting_Hole H1
+U 1 1 5AF1AB95
+P 11900 14200
+F 0 "H1" H 12000 14246 50  0000 L CNN
+F 1 "Mounting_Hole" H 12000 14155 50  0000 L CNN
+F 2 "Mounting_Holes:MountingHole_3.2mm_M3" H 11900 14200 50  0001 C CNN
+F 3 "" H 11900 14200 50  0001 C CNN
+	1    11900 14200
+	1    0    0    -1
+$EndComp
+$Comp
+L Mechanical:Mounting_Hole H2
+U 1 1 5AF1AFD9
+P 11900 14400
+F 0 "H2" H 12000 14446 50  0000 L CNN
+F 1 "Mounting_Hole" H 12000 14355 50  0000 L CNN
+F 2 "Mounting_Holes:MountingHole_3.2mm_M3" H 11900 14400 50  0001 C CNN
+F 3 "" H 11900 14400 50  0001 C CNN
+	1    11900 14400
+	1    0    0    -1
+$EndComp
+$Comp
+L Mechanical:Mounting_Hole H3
+U 1 1 5AF1B0A9
+P 11900 14600
+F 0 "H3" H 12000 14646 50  0000 L CNN
+F 1 "Mounting_Hole" H 12000 14555 50  0000 L CNN
+F 2 "Mounting_Holes:MountingHole_3.2mm_M3" H 11900 14600 50  0001 C CNN
+F 3 "" H 11900 14600 50  0001 C CNN
+	1    11900 14600
+	1    0    0    -1
+$EndComp
+$Comp
+L Mechanical:Mounting_Hole H4
+U 1 1 5AF1B185
+P 11900 14800
+F 0 "H4" H 12000 14846 50  0000 L CNN
+F 1 "Mounting_Hole" H 12000 14755 50  0000 L CNN
+F 2 "Mounting_Holes:MountingHole_3.2mm_M3" H 11900 14800 50  0001 C CNN
+F 3 "" H 11900 14800 50  0001 C CNN
+	1    11900 14800
+	1    0    0    -1
+$EndComp
+$Comp
+L Graphic:SYM_Arrow45_Large SYM1
+U 1 1 5AF1C901
+P 11900 15400
+F 0 "SYM1" H 11900 15560 50  0001 C CNN
+F 1 "SYM_Arrow45_Large" H 11900 15260 50  0001 C CNN
+F 2 "Custom Parts:Logo_v3" H 11900 15400 50  0001 C CNN
+F 3 "~" H 11900 15400 50  0001 C CNN
+	1    11900 15400
+	0    -1   -1   0
+$EndComp
 $EndSCHEMATC
