File: Control Board/Control Board.sch (KiCad schematic (older format))
At the start: 97 parts, among them J1 Conn_02x10_Odd_Even, J10 Conn_01x03, J11 Conn_01x03, J13 Conn_01x03, J14 Conn_01x03, J15 Conn_01x03, J2 Conn_02x03_Odd_Even, J3 RJ45, J4 Conn_01x02, J5 Conn_01x02, J6 Conn_01x03, J7 Conn_01x02, J8 Conn_01x02, J9 Conn_01x02, Q1 STS4DNF60L, U1 ATXMEGA128A3-AU, U10 OPENLOG, U2 LT1797, U3 LT1797, U4 ISL83490, U5 MAX31856, U6 MAX31856, U7 MAX31856, U8 MAX31856, U9 MAX31856

Commit message: Added Heatsink, changed umbilical voltage
10.5 volts is technically above the max reccomended supply for the lipo balancer, but it's set to that to make sure the supply doesn't come in and out if it's at 10 volts
Parts:
- C1, C10, C11, C12, C13, C14, C15, C16, C17, C18, C19, C2, C20, C21, C22, C23, C24, C25, C26, C27, C28, C29, C3, C30, C31, C32, C33, C34, C35, C4, C5, C6, C7, C8, C9: symbol device:C_Small -> Control-Board-rescue:C_Small-device
- D1, D2, D3, D4: symbol device:LED -> Control-Board-rescue:LED-device
- H1, H2, H3, H4: symbol Mechanical:Mounting_Hole -> Control-Board-rescue:Mounting_Hole-Mechanical
- J1: symbol Connector:Conn_02x10_Odd_Even -> Control-Board-rescue:Conn_02x10_Odd_Even-Connector
- J10, J11, J13, J14, J15, J6: symbol Connector:Conn_01x03 -> Control-Board-rescue:Conn_01x03-Connector
- J3: symbol Connector:RJ45 -> Control-Board-rescue:RJ45-Connector
- J4, J5, J7, J8, J9: symbol Connector:Conn_01x02 -> Control-Board-rescue:Conn_01x02-Connector
- L1: symbol device:L_Small -> Control-Board-rescue:L_Small-device
- R1, R10, R11, R12, R13, R14, R15, R16, R17, R18, R19, R2, R20, R21, R23, R24, R25, R3, R4, R5: symbol device:R_Small -> Control-Board-rescue:R_Small-device
- R22, R6, R7, R8, R9: symbol device:R -> Control-Board-rescue:R-device
- RN1, RN2: symbol device:Voltage_Divider_CenterPin3 -> Control-Board-rescue:Voltage_Divider_CenterPin3-device
- U1: symbol atmel:ATXMEGA128A3-AU -> Control-Board-rescue:ATXMEGA128A3-AU-atmel

Commit message: Actually making the changes in the last commit because I forgot to save first
Parts:
- removed J2: Conn_02x03_Odd_Even, Pin_Headers:Pin_Header_Angled_2x03_Pitch1.27mm, symbol Control-Board-rescue:Conn_02x03_Odd_Even
- removed R10, R12, R13, R18, R20: 20 kΩ, Resistors_SMD:R_0603, symbol Control-Board-rescue:R_Small-device
- removed R11, R14, R15, R17, R19, R21: 1 kΩ, Resistors_SMD:R_0603, symbol Control-Board-rescue:R_Small-device
- removed R16: 4.99 kΩ, Resistors_SMD:R_0603, symbol Control-Board-rescue:R_Small-device
- added C? (x2): 0.1 uF, Capacitors_SMD:C_0603, symbol Control-Board-rescue:C_Small-device
- added J?: Conn_02x03_Odd_Even, symbol Connector_Generic:Conn_02x03_Odd_Even
- added RN? (x2): 1 kΩ, 5 kΩ, TO_SOT_Packages_SMD:SOT-23, symbol Control-Board-rescue:Voltage_Divider_CenterPin3-device
- added U? (x2): LT1797, TO_SOT_Packages_SMD:TSOT-23-5, symbol Custom-Parts:LT1797
Connections:
- net labels added: PT3_ADC, PT3_IN, PT4_ADC, PT4_IN
- net labels removed: V_3.3_ADC, V_BAT1_ADC, V_BAT2_ADC, V_PT_ADC, V_SUPPLY_ADC, V_UMB_ADC
- wire segments 301 -> 297
- no-connect marks 3 -> 5

Commit message: Changed to 2x7 header from 2x10
Parts:
- removed J1: Conn_02x10_Odd_Even, Pin_Headers:Pin_Header_Straight_2x10_Pitch1.27mm, symbol Control-Board-rescue:Conn_02x10_Odd_Even-Connector
- removed U10: OPENLOG, Custom Footprints:OpenLog, symbol Custom-Parts:OPENLOG
- added J?: Conn_02x07_Counter_Clockwise, symbol Connector_Generic:Conn_02x07_Counter_Clockwise
Connections:
- net labels added: PWR_SCL, PWR_SDA
- net labels removed: BAT_BAK_VCC, BAT_VCC, UMB_VCC
- no-connect marks 5 -> 4
Changed lines of the file:
@@
-$EndComp
-$Comp
-L power:+3V3 #PWR075
-U 1 1 5A835285
-P 14350 10750
-F 0 "#PWR075" H 14350 10600 50  0001 C CNN
-F 1 "+3V3" V 14350 10950 50  0000 C CNN
-F 2 "" H 14350 10750 50  0001 C CNN
-F 3 "" H 14350 10750 50  0001 C CNN
-	1    14350 10750
-	0    -1   -1   0
 $EndComp
 $Comp
@@
 Text Label 4650 3300 0    60   ~ 0
 TC4_DRDY
-Text Label 4650 3450 0    60   ~ 0
+Text Label 4650 2350 0    60   ~ 0
 TC5_CS
-Text Label 4650 3550 0    60   ~ 0
+Text Label 4650 2450 0    60   ~ 0
 TC5_DRDY
 Text Label 4650 4300 0    60   ~ 0
@@
 Text Label 14550 14250 2    60   ~ 0
 SERVO2_CL_SW
-Text Label 13800 10950 2    60   ~ 0
+Text Label 13800 11050 2    60   ~ 0
 GNC_INST
 Text Label 14550 15050 2    60   ~ 0
@@
 Text Label 14550 14150 2    60   ~ 0
 SERVO2_OP_SW
-Text Label 14850 11150 0    60   ~ 0
-BAT_BAK_VCC
-Text Label 14850 11050 0    60   ~ 0
-BAT_VCC
-Text Label 14850 10950 0    60   ~ 0
-UMB_VCC
 Wire Wire Line
 	15950 1750 15050 1750
@@
 Connection ~ 8750 1850
 Connection ~ 8750 3500
-Text Label 14850 10850 0    60   ~ 0
-VCC_IN
-$Comp
-L power:GND #PWR090
-U 1 1 5A9D5527
-P 14850 10750
-F 0 "#PWR090" H 14850 10500 50  0001 C CNN
-F 1 "GND" V 14850 10550 50  0000 C CNN
-F 2 "" H 14850 10750 50  0001 C CNN
-F 3 "" H 14850 10750 50  0001 C CNN
-	1    14850 10750
-	0    -1   1    0
-$EndComp
 Text Label 15650 15350 2    60   ~ 0
 SERVO1_CTRL
@@
 OPENLOG_RX
 $Comp
-L Custom-Parts:OPENLOG U10
-U 1 1 5ACDDD81
-P 9050 14400
-F 0 "U10" H 9478 14540 50  0000 L CNN
-F 1 "OPENLOG" H 9478 14449 50  0000 L CNN
-F 2 "Custom Footprints:OpenLog" H 8900 14400 50  0001 C CNN
-F 3 "" H 8900 14400 50  0001 C CNN
-F 4 "1568-1368-ND" H 0   0   50  0001 C CNN "Digikey Part Number"
-	1    9050 14400
-	1    0    0    -1
-$EndComp
-NoConn ~ 8800 14600
-$Comp
 L power:GND #PWR096
 U 1 1 5ACFC32F
-P 9300 14600
-F 0 "#PWR096" H 9300 14350 50  0001 C CNN
-F 1 "GND" H 9300 14450 50  0000 C CNN
-F 2 "" H 9300 14600 50  0001 C CNN
-F 3 "" H 9300 14600 50  0001 C CNN
-	1    9300 14600
+P 3450 11600
+F 0 "#PWR096" H 3450 11350 50  0001 C CNN
+F 1 "GND" H 3450 11450 50  0000 C CNN
+F 2 "" H 3450 11600 50  0001 C CNN
+F 3 "" H 3450 11600 50  0001 C CNN
+	1    3450 11600
 	-1   0    0    -1
 $EndComp
 Wire Wire Line
-	9200 14600 9300 14600
-Connection ~ 9300 14600
-Wire Wire Line
-	9100 14600 9100 15050
-Wire Wire Line
-	9100 15050 9300 15050
+	3350 11600 3450 11600
+Wire Wire Line
+	3250 11600 3250 12050
+Wire Wire Line
+	3250 12050 3450 12050
 $Comp
 L power:+3V3 #PWR098
 U 1 1 5AD38C00
-P 9300 15050
-F 0 "#PWR098" H 9300 14900 50  0001 C CNN
-F 1 "+3V3" H 9300 15190 50  0000 C CNN
-F 2 "" H 9300 15050 50  0001 C CNN
-F 3 "" H 9300 15050 50  0001 C CNN
-	1    9300 15050
-	1    0    0    -1
-$EndComp
-Wire Wire Line
-	9000 14600 9000 15050
-Wire Wire Line
-	9000 15050 8150 15050
-Wire Wire Line
-	8900 14600 8900 14950
-Wire Wire Line
-	8900 14950 8150 14950
-Text Label 8150 15050 2    60   ~ 0
+P 3450 12050
+F 0 "#PWR098" H 3450 11900 50  0001 C CNN
+F 1 "+3V3" H 3450 12190 50  0000 C CNN
+F 2 "" H 3450 12050 50  0001 C CNN
+F 3 "" H 3450 12050 50  0001 C CNN
+	1    3450 12050
+	1    0    0    -1
+$EndComp
+Wire Wire Line
+	3150 11600 3150 12050
+Wire Wire Line
+	3150 12050 2300 12050
+Wire Wire Line
+	3050 11600 3050 11950
+Wire Wire Line
+	3050 11950 2300 11950
+Text Label 2300 12050 2    60   ~ 0
 OPENLOG_TX
-Text Label 8150 14950 2    60   ~ 0
+Text Label 2300 11950 2    60   ~ 0
 OPENLOG_RX
 Text Label 2150 3750 2    60   ~ 0
@@
 $EndComp
 $Comp
-L Control-Board-rescue:Conn_02x10_Odd_Even-Connector J1
-U 1 1 5AD96437
-P 14550 11150
-F 0 "J1" H 14600 11767 50  0000 C CNN
-F 1 "Conn_02x10_Odd_Even" H 14600 11676 50  0000 C CNN
-F 2 "Pin_Headers:Pin_Header_Straight_2x10_Pitch1.27mm" H 14550 11150 50  0001 C CNN
-F 3 "~" H 14550 11150 50  0001 C CNN
-	1    14550 11150
-	1    0    0    -1
-$EndComp
-$Comp
 L Control-Board-rescue:RJ45-Connector J3
 U 1 1 5ADD31C9
@@
 L power:+3V3 #PWR078
 U 1 1 5AB9D0A9
+P 14850 11650
+F 0 "#PWR078" H 14850 11500 50  0001 C CNN
+F 1 "+3V3" V 14850 11850 50  0000 C CNN
+F 2 "" H 14850 11650 50  0001 C CNN
+F 3 "" H 14850 11650 50  0001 C CNN
+	1    14850 11650
+	0    1    1    0
+$EndComp
+$Comp
+L power:+12V #PWR080
+U 1 1 5AB9D729
 P 14850 11350
-F 0 "#PWR078" H 14850 11200 50  0001 C CNN
-F 1 "+3V3" V 14850 11550 50  0000 C CNN
+F 0 "#PWR080" H 14850 11200 50  0001 C CNN
+F 1 "+12V" V 14850 11550 50  0000 C CNN
 F 2 "" H 14850 11350 50  0001 C CNN
 F 3 "" H 14850 11350 50  0001 C CNN
 	1    14850 11350
-	0    1    1    0
-$EndComp
-$Comp
-L power:+12V #PWR080
-U 1 1 5AB9D729
-P 14850 11550
-F 0 "#PWR080" H 14850 11400 50  0001 C CNN
-F 1 "+12V" V 14850 11750 50  0000 C CNN
-F 2 "" H 14850 11550 50  0001 C CNN
-F 3 "" H 14850 11550 50  0001 C CNN
-	1    14850 11550
 	0    1    1    0
 $EndComp
@@
 $EndComp
 $Comp
-L power:GND #PWR081
-U 1 1 5AB9D89B
-P 14850 11650
-F 0 "#PWR081" H 14850 11400 50  0001 C CNN
-F 1 "GND" V 14850 11450 50  0000 C CNN
-F 2 "" H 14850 11650 50  0001 C CNN
-F 3 "" H 14850 11650 50  0001 C CNN
-	1    14850 11650
-	0    -1   1    0
-$EndComp
-$Comp
 L power:GND #PWR065
 U 1 1 5ABBF318
-P 13900 11150
-F 0 "#PWR065" H 13900 10900 50  0001 C CNN
-F 1 "GND" V 13900 10950 50  0000 C CNN
-F 2 "" H 13900 11150 50  0001 C CNN
-F 3 "" H 13900 11150 50  0001 C CNN
-	1    13900 11150
+P 13900 11250
+F 0 "#PWR065" H 13900 11000 50  0001 C CNN
+F 1 "GND" V 13900 11050 50  0000 C CNN
+F 2 "" H 13900 11250 50  0001 C CNN
+F 3 "" H 13900 11250 50  0001 C CNN
+	1    13900 11250
 	-1   0    0    -1
 $EndComp
@@
 L Control-Board-rescue:R_Small-device R1
 U 1 1 5ABC0525
-P 13900 11050
-F 0 "R1" H 13930 11070 50  0000 L CNN
-F 1 "10 kΩ" H 13930 11010 50  0000 L CNN
-F 2 "Resistors_SMD:R_0603" H 13900 11050 50  0001 C CNN
-F 3 "" H 13900 11050 50  0001 C CNN
-F 4 "311-10.0KHRCT-ND" H 13930 11170 50  0001 C CNN "Digikey Part Number"
-	1    13900 11050
+P 13900 11150
+F 0 "R1" H 13930 11170 50  0000 L CNN
+F 1 "10 kΩ" H 13930 11110 50  0000 L CNN
+F 2 "Resistors_SMD:R_0603" H 13900 11150 50  0001 C CNN
+F 3 "" H 13900 11150 50  0001 C CNN
+F 4 "311-10.0KHRCT-ND" H 13930 11270 50  0001 C CNN "Digikey Part Number"
+	1    13900 11150
 	-1   0    0    1
 $EndComp
 Wire Wire Line
-	13800 10950 13900 10950
-Connection ~ 13900 10950
-Wire Wire Line
-	13900 10950 14350 10950
-$Comp
-L power:GND #PWR063
-U 1 1 5AC1B6BF
-P 14350 10850
-F 0 "#PWR063" H 14350 10600 50  0001 C CNN
-F 1 "GND" V 14350 10650 50  0000 C CNN
-F 2 "" H 14350 10850 50  0001 C CNN
-F 3 "" H 14350 10850 50  0001 C CNN
-	1    14350 10850
-	0    1    -1   0
-$EndComp
-$Comp
-L power:GND #PWR064
-U 1 1 5AC1B82A
-P 14350 11050
-F 0 "#PWR064" H 14350 10800 50  0001 C CNN
-F 1 "GND" V 14350 10850 50  0000 C CNN
-F 2 "" H 14350 11050 50  0001 C CNN
-F 3 "" H 14350 11050 50  0001 C CNN
-	1    14350 11050
-	0    1    -1   0
-$EndComp
+	13800 11050 13900 11050
+Connection ~ 13900 11050
+Wire Wire Line
+	13900 11050 14350 11050
 $Comp
 L Control-Board-rescue:Conn_01x03-Connector J6
@@
 Wire Wire Line
 	8750 6850 8750 7000
+Text Label 14850 11550 0    60   ~ 0
+VCC_IN
+Text Label 14850 11050 0    50   ~ 0
+PWR_SDA
+Text Label 14850 11150 0    50   ~ 0
+PWR_SCL
+Text Label 4650 3450 0    50   ~ 0
+PWR_SDA
+Text Label 4650 3550 0    50   ~ 0
+PWR_SCL
+$Comp
+L Connector_Generic:Conn_02x07_Counter_Clockwise J?
+U 1 1 5C07DC16
+P 14550 11350
+F 0 "J?" H 14600 11867 50  0000 C CNN
+F 1 "Conn_02x07_Counter_Clockwise" H 14600 11776 50  0000 C CNN
+F 2 "" H 14550 11350 50  0001 C CNN
+F 3 "~" H 14550 11350 50  0001 C CNN
+	1    14550 11350
+	1    0    0    -1
+$EndComp
 $EndSCHEMATC

Commit message: Removed openlog breakout, duplicated openlog
I copied the schematic from https://github.com/sparkfun/OpenLog/tree/master/hardware. This was done to save some vertical space, since headers are pretty tall. It should also be more robust.
Parts:
- added C? (x2): 0.1 uF, Capacitors_SMD:C_0603, symbol Control-Board-rescue:C_Small-device
- added D?: LED_G, LEDs:LED_0603, symbol Control-Board-rescue:LED-device
- added D?: LED_B, LEDs:LED_0603, symbol Control-Board-rescue:LED-device
- added J?: Micro_SD_Card_SPI_MODE_Det, symbol Custom-Parts:Micro_SD_Card_SPI_MODE_Det
- added R?: 10 kΩ, symbol Device:R_Small
- added R?: 1 kΩ, symbol Device:R_Small
- added R?: 330 Ω, symbol Device:R_Small
- added U?: ATmega328P-AU, Package_QFP:TQFP-32_7x7mm_P0.8mm, symbol MCU_Microchip_ATmega:ATmega328P-AU
- added Y?: 16 MHz, symbol Device:Resonator_Small
Connections:
- net labels added: SD_CD, SD_CS, SD_MISO, SD_MOSI, SD_SCK
- wire segments 297 -> 324
- no-connect marks 4 -> 6
Other:
- note added: "Basically putting an OpenLog on the board instead of a breakout"
- note added: "From Sparkfun OpenLog"
- note added: "Not a generic ATMEGA328P! Chip must be desoldered from OpenLog.\nThis is because it must be preprogrammed with the Arduino bootloader\nand OpenLog firmware. (I could add components to be able to flash the\nbootloader and firmware but I'm lazy and this is easier)"

Commit message: Remembered to add connectors for the new PTs
Parts:
- added J? (x2): Conn_01x03, Connectors_JST:JST_PH_B3B-PH-K_03x2.00mm_Straight, symbol Control-Board-rescue:Conn_01x03-Connector
Changed lines of the file:
@@
 Text Notes 3900 13950 0    50   ~ 0
 Not a generic ATMEGA328P! Chip must be desoldered from OpenLog.\nThis is because it must be preprogrammed with the Arduino bootloader\nand OpenLog firmware. (I could add components to be able to flash the\nbootloader and firmware but I'm lazy and this is easier)
+$Comp
+L power:+12V #PWR?
+U 1 1 5C58D70F
+P 17600 12800
+F 0 "#PWR?" H 17600 12650 50  0001 C CNN
+F 1 "+12V" V 17600 13000 50  0000 C CNN
+F 2 "" H 17600 12800 50  0001 C CNN
+F 3 "" H 17600 12800 50  0001 C CNN
+	1    17600 12800
+	0    1    1    0
+$EndComp
+$Comp
+L power:GND #PWR?
+U 1 1 5C58D715
+P 17600 12700
+F 0 "#PWR?" H 17600 12450 50  0001 C CNN
+F 1 "GND" V 17600 12500 50  0000 C CNN
+F 2 "" H 17600 12700 50  0001 C CNN
+F 3 "" H 17600 12700 50  0001 C CNN
+	1    17600 12700
+	0    -1   1    0
+$EndComp
+Text Label 17600 12900 0    60   ~ 0
+PT3_IN
+Text Label 17600 13450 0    60   ~ 0
+PT4_IN
+$Comp
+L power:+12V #PWR?
+U 1 1 5C58D71D
+P 17600 13350
+F 0 "#PWR?" H 17600 13200 50  0001 C CNN
+F 1 "+12V" V 17600 13550 50  0000 C CNN
+F 2 "" H 17600 13350 50  0001 C CNN
+F 3 "" H 17600 13350 50  0001 C CNN
+	1    17600 13350
+	0    1    1    0
+$EndComp
+$Comp
+L power:GND #PWR?
+U 1 1 5C58D723
+P 17600 13250
+F 0 "#PWR?" H 17600 13000 50  0001 C CNN
+F 1 "GND" V 17600 13050 50  0000 C CNN
+F 2 "" H 17600 13250 50  0001 C CNN
+F 3 "" H 17600 13250 50  0001 C CNN
+	1    17600 13250
+	0    -1   1    0
+$EndComp
+$Comp
+L Control-Board-rescue:Conn_01x03-Connector J?
+U 1 1 5C58D72A
+P 17400 12800
+F 0 "J?" H 17320 12475 50  0000 C CNN
+F 1 "Conn_01x03" H 17320 12566 50  0000 C CNN
+F 2 "Connectors_JST:JST_PH_B3B-PH-K_03x2.00mm_Straight" H 17400 12800 50  0001 C CNN
+F 3 "~" H 17400 12800 50  0001 C CNN
+F 4 "455-1720-ND" H 1100 0   50  0001 C CNN "Digikey Part Number"
+	1    17400 12800
+	-1   0    0    1
+$EndComp
+$Comp
+L Control-Board-rescue:Conn_01x03-Connector J?
+U 1 1 5C58D731
+P 17400 13350
+F 0 "J?" H 17320 13025 50  0000 C CNN
+F 1 "Conn_01x03" H 17320 13116 50  0000 C CNN
+F 2 "Connectors_JST:JST_PH_B3B-PH-K_03x2.00mm_Straight" H 17400 13350 50  0001 C CNN
+F 3 "~" H 17400 13350 50  0001 C CNN
+F 4 "455-1720-ND" H 1100 0   50  0001 C CNN "Digikey Part Number"
+	1    17400 13350
+	-1   0    0    1
+$EndComp
 $EndSCHEMATC

Commit message: Removed servo control MOSFETs
Now connected directly. They can work with a 3.3v PWM signal according to https://www.servocity.com/hs-m7990th-servo
Parts:
- removed Q1: STS4DNF60L, Housings_SOIC:SOIC-8_3.9x4.9mm_Pitch1.27mm, symbol Custom-Parts:STS4DNF60L
- removed R3, R4: 1 kΩ, Resistors_SMD:R_0603, symbol Control-Board-rescue:R_Small-device
Connections:
- net labels removed: VCC_IN
- wire segments 324 -> 315
Other:
- note added: "Not sure if this part is necessary, ask James\nif the servos work with 3.3V control signal\n\nTurns out it isn't necessary!"
Changed lines of the file:
@@
-$EndComp
-$Comp
-L Custom-Parts:STS4DNF60L Q1
-U 1 1 5A819BE3
-P 3200 6250
-F 0 "Q1" H 3200 6550 60  0000 C CNN
-F 1 "STS4DNF60L" H 3200 5950 60  0000 C CNN
-F 2 "Housings_SOIC:SOIC-8_3.9x4.9mm_Pitch1.27mm" H 3200 6100 60  0001 C CNN
-F 3 "" H 3200 6100 60  0001 C CNN
-F 4 "497-3226-1-ND" H 3200 6650 50  0001 C CNN "Digikey Part Number"
-	1    3200 6250
-	1    0    0    -1
-$EndComp
-$Comp
-L power:GND #PWR061
-U 1 1 5A81AB94
-P 2750 6100
-F 0 "#PWR061" H 2750 5850 50  0001 C CNN
-F 1 "GND" H 2750 5950 50  0000 C CNN
-F 2 "" H 2750 6100 50  0001 C CNN
-F 3 "" H 2750 6100 50  0001 C CNN
-	1    2750 6100
-	0    1    1    0
-$EndComp
-$Comp
-L power:GND #PWR062
-U 1 1 5A81AD05
-P 2750 6300
-F 0 "#PWR062" H 2750 6050 50  0001 C CNN
-F 1 "GND" H 2750 6150 50  0000 C CNN
-F 2 "" H 2750 6300 50  0001 C CNN
-F 3 "" H 2750 6300 50  0001 C CNN
-	1    2750 6300
-	0    1    1    0
 $EndComp
 $Comp
@@
 	2400 3450 2150 3450
 Wire Wire Line
-	2750 6200 2100 6200
-Wire Wire Line
-	2750 6400 2100 6400
-Wire Wire Line
-	3650 6100 3650 6200
-Wire Wire Line
-	3650 6200 4000 6200
-Wire Wire Line
-	3650 6300 3650 6400
-Wire Wire Line
 	2350 7050 2950 7050
 Wire Wire Line
@@
 Connection ~ 9350 2350
 Connection ~ 9350 4000
-Connection ~ 4000 6200
 Connection ~ 2800 7250
 Connection ~ 9550 11850
@@
 Wire Wire Line
 	9350 4000 9750 4000
-Wire Wire Line
-	4000 6200 4200 6200
 Wire Wire Line
 	2800 7250 2950 7250
@@
 Text Label 2150 3750 2    60   ~ 0
 XBEE_RX
-Wire Wire Line
-	3800 5550 4000 5550
-$Comp
-L Control-Board-rescue:R_Small-device R4
-U 1 1 5A81B850
-P 4000 5650
-F 0 "R4" H 4030 5670 50  0000 L CNN
-F 1 "1 kΩ" H 4030 5610 50  0000 L CNN
-F 2 "Resistors_SMD:R_0603" H 4000 5650 50  0001 C CNN
-F 3 "" H 4000 5650 50  0001 C CNN
-F 4 "311-1.00KHRCT-ND" H 4030 5770 50  0001 C CNN "Digikey Part Number"
-	1    4000 5650
-	1    0    0    1
-$EndComp
-$Comp
-L Control-Board-rescue:R_Small-device R3
-U 1 1 5A81B773
-P 3800 5650
-F 0 "R3" H 3830 5670 50  0000 L CNN
-F 1 "1 kΩ" H 3830 5610 50  0000 L CNN
-F 2 "Resistors_SMD:R_0603" H 3800 5650 50  0001 C CNN
-F 3 "" H 3800 5650 50  0001 C CNN
-F 4 "311-1.00KHRCT-ND" H 3830 5770 50  0001 C CNN "Digikey Part Number"
-	1    3800 5650
-	-1   0    0    -1
-$EndComp
-Wire Wire Line
-	4000 5750 4000 6200
-Wire Wire Line
-	3800 6400 4200 6400
-Wire Wire Line
-	3650 6400 3800 6400
-Connection ~ 3800 6400
-Wire Wire Line
-	3800 5750 3800 6400
-Text Label 3900 5550 0    60   ~ 0
-VCC_IN
 $Comp
 L power:GND #PWR082
@@
 	14750 14250 14550 14250
 Connection ~ 3900 7050
-Connection ~ 3650 6200
-Connection ~ 3650 6400
 $Comp
 L Control-Board-rescue:Mounting_Hole-Mechanical H1
@@
 Wire Wire Line
 	8750 6850 8750 7000
-Text Label 14850 11550 0    60   ~ 0
-VCC_IN
 Text Label 14850 11050 0    50   ~ 0
 PWR_SDA
@@
 	-1   0    0    1
 $EndComp
+Text Notes 1750 5850 0    50   ~ 0
+Not sure if this part is necessary, ask James\nif the servos work with 3.3V control signal\n\nTurns out it isn't necessary!
+Wire Wire Line
+	2100 6200 4200 6200
+Wire Wire Line
+	2100 6400 4200 6400
+$Comp
+L power:+3V3 #PWR?
+U 1 1 5C653C57
+P 14850 11550
+F 0 "#PWR?" H 14850 11400 50  0001 C CNN
+F 1 "+3V3" V 14850 11750 50  0000 C CNN
+F 2 "" H 14850 11550 50  0001 C CNN
+F 3 "" H 14850 11550 50  0001 C CNN
+	1    14850 11550
+	0    1    1    0
+$EndComp
 $EndSCHEMATC

Commit message: Added some series resistors to the servo control lines
Parts:
- added R? (x2): 220 Ω, symbol Device:R_Small
Connections:
- wire segments 315 -> 316
Changed lines of the file:
@@
 Text Label 2150 3650 2    60   ~ 0
 XBEE_TX
-Text Label 2150 3550 2    60   ~ 0
-GNC_INST
 Text Label 2150 3450 2    60   ~ 0
 MODE_SW
@@
 	2400 4400 2150 4400
 Wire Wire Line
-	2150 3550 2400 3550
-Wire Wire Line
 	2400 3450 2150 3450
 Wire Wire Line
@@
 Not sure if this part is necessary, ask James\nif the servos work with 3.3V control signal\n\nTurns out it isn't necessary!
 Wire Wire Line
-	2100 6200 4200 6200
-Wire Wire Line
-	2100 6400 4200 6400
+	2100 6200 3100 6200
+Wire Wire Line
+	2100 6400 3100 6400
 $Comp
 L power:+3V3 #PWR?
@@
 	0    1    1    0
 $EndComp
+$Comp
+L Device:R_Small R?
+U 1 1 5C69A738
+P 3200 6200
+F 0 "R?" V 3004 6200 50  0000 C CNN
+F 1 "220 Ω" V 3095 6200 50  0000 C CNN
+F 2 "" H 3200 6200 50  0001 C CNN
+F 3 "~" H 3200 6200 50  0001 C CNN
+	1    3200 6200
+	0    1    1    0
+$EndComp
+Wire Wire Line
+	3300 6200 4200 6200
+Wire Wire Line
+	3300 6400 4200 6400
+$Comp
+L Device:R_Small R?
+U 1 1 5C69AF52
+P 3200 6400
+F 0 "R?" V 3396 6400 50  0000 C CNN
+F 1 "220 Ω" V 3305 6400 50  0000 C CNN
+F 2 "" H 3200 6400 50  0001 C CNN
+F 3 "~" H 3200 6400 50  0001 C CNN
+	1    3200 6400
+	0    -1   -1   0
+$EndComp
+Text Label 4650 2250 0    60   ~ 0
+GNC_INST
 $EndSCHEMATC
