File: Control Board/Control Board.sch (KiCad schematic (older format))
At the start: 101 parts, among them J10 Conn_01x03, J11 Conn_01x03, J13 Conn_01x03, J14 Conn_01x03, J15 Conn_01x03, J3 RJ45, J4 Conn_01x02, J5 Conn_01x02, J6 Conn_01x03, J7 Conn_01x02, J8 Conn_01x02, J9 Conn_01x02, U1 ATXMEGA128A3-AU, U2 LT1797, U3 LT1797, U4 ISL83490, U5 MAX31856, U6 MAX31856, U7 MAX31856, U8 MAX31856, U9 MAX31856

Commit message: Added safety radio to control board
Uses LoRa, which is has a lower data rate than XBees, but much longer range for a given power consumption. Should be able to reach 6000 ft with low gain antennas. It's also way cheaper.
Parts:
- added C?: 0.1 uF, Capacitors_SMD:C_0603, symbol Control-Board-rescue:C_Small-device
- added J?: U.FL, U.FL, symbol SparkFun-Connectors:U.FL
- added R?: 10 kΩ, Resistors_SMD:R_0603, symbol Control-Board-rescue:R_Small-device
- added U?: RFM96W-315S2, symbol RF_AM_FM:RFM96W-315S2
Connections:
- net labels added: LORA_CS, LORA_IRQ, LORA_RST
- net labels removed: MODE_SW
- wire segments 316 -> 331
- no-connect marks 6 -> 11
Changed lines of the file:
@@
 Text Label 2150 3650 2    60   ~ 0
 XBEE_TX
-Text Label 2150 3450 2    60   ~ 0
-MODE_SW
 Text Notes 12200 1700 0    60   ~ 0
 EXT
@@
 	2400 4400 2150 4400
 Wire Wire Line
-	2400 3450 2150 3450
-Wire Wire Line
 	2350 7050 2950 7050
 Wire Wire Line
@@
 Text Label 4650 2250 0    60   ~ 0
 GNC_INST
+$Comp
+L RF_AM_FM:RFM96W-315S2 U?
+U 1 1 5C761F8F
+P 19800 2000
+F 0 "U?" H 19950 2550 50  0000 C CNN
+F 1 "RFM96W-315S2" H 20150 2450 50  0000 C CNN
+F 2 "" H 16500 3650 50  0001 C CNN
+F 3 "http://www.hoperf.com/upload/rf/RFM95_96_97_98W.pdf" H 16500 3650 50  0001 C CNN
+	1    19800 2000
+	1    0    0    -1
+$EndComp
+Text Label 19300 1700 2    60   ~ 0
+SCK1
+Text Label 19300 1800 2    60   ~ 0
+MOSI1
+Text Label 19300 1900 2    60   ~ 0
+MISO1
+Wire Wire Line
+	19700 2600 19700 2700
+Wire Wire Line
+	19700 2700 19800 2700
+Wire Wire Line
+	19900 2700 19900 2600
+Wire Wire Line
+	19800 2600 19800 2700
+Connection ~ 19800 2700
+Wire Wire Line
+	19800 2700 19900 2700
+$Comp
+L power:GND #PWR?
+U 1 1 5C7D3705
+P 19800 2700
+F 0 "#PWR?" H 19800 2450 50  0001 C CNN
+F 1 "GND" H 19800 2550 50  0000 C CNN
+F 2 "" H 19800 2700 50  0001 C CNN
+F 3 "" H 19800 2700 50  0001 C CNN
+	1    19800 2700
+	1    0    0    -1
+$EndComp
+$Comp
+L SparkFun-Connectors:U.FL J?
+U 1 1 5C7D391F
+P 20900 1700
+F 0 "J?" H 20950 2060 45  0000 C CNN
+F 1 "U.FL" H 20950 1976 45  0000 C CNN
+F 2 "U.FL" H 20900 1950 20  0001 C CNN
+F 3 "" H 20900 1700 50  0001 C CNN
+F 4 "CONN-09193" H 20950 1881 60  0000 C CNN "Field4"
+	1    20900 1700
+	-1   0    0    -1
+$EndComp
+Wire Wire Line
+	20300 1700 20700 1700
+Wire Wire Line
+	21000 1900 21100 1900
+Wire Wire Line
+	21100 1900 21100 2000
+Wire Wire Line
+	21100 2000 21000 2000
+$Comp
+L power:GND #PWR?
+U 1 1 5C81F7C4
+P 21100 2000
+F 0 "#PWR?" H 21100 1750 50  0001 C CNN
+F 1 "GND" H 21100 1850 50  0000 C CNN
+F 2 "" H 21100 2000 50  0001 C CNN
+F 3 "" H 21100 2000 50  0001 C CNN
+	1    21100 2000
+	1    0    0    -1
+$EndComp
+Connection ~ 21100 2000
+$Comp
+L Control-Board-rescue:R_Small-device R?
+U 1 1 5C82075A
+P 18600 2100
+F 0 "R?" H 18630 2120 50  0000 L CNN
+F 1 "10 kΩ" H 18630 2060 50  0000 L CNN
+F 2 "Resistors_SMD:R_0603" H 18600 2100 50  0001 C CNN
+F 3 "" H 18600 2100 50  0001 C CNN
+F 4 "311-10.0KHRCT-ND" H 18630 2220 50  0001 C CNN "Digikey Part Number"
+	1    18600 2100
+	-1   0    0    1
+$EndComp
+Wire Wire Line
+	19300 2200 18600 2200
+Connection ~ 18600 2200
+Wire Wire Line
+	18600 2200 18300 2200
+$Comp
+L power:+3V3 #PWR?
+U 1 1 5C847A2E
+P 19800 1300
+F 0 "#PWR?" H 19800 1150 50  0001 C CNN
+F 1 "+3V3" H 19800 1440 50  0000 C CNN
+F 2 "" H 19800 1300 50  0001 C CNN
+F 3 "" H 19800 1300 50  0001 C CNN
+	1    19800 1300
+	1    0    0    -1
+$EndComp
+Wire Wire Line
+	19800 1300 19800 1350
+$Comp
+L power:+3V3 #PWR?
+U 1 1 5C86EE1C
+P 18600 2000
+F 0 "#PWR?" H 18600 1850 50  0001 C CNN
+F 1 "+3V3" H 18600 2140 50  0000 C CNN
+F 2 "" H 18600 2000 50  0001 C CNN
+F 3 "" H 18600 2000 50  0001 C CNN
+	1    18600 2000
+	1    0    0    -1
+$EndComp
+Text Label 18300 2200 2    50   ~ 0
+LORA_RST
+Text Label 19300 2000 2    50   ~ 0
+LORA_CS
+Text Label 2150 3850 2    50   ~ 0
+LORA_RST
+Text Label 2150 3950 2    50   ~ 0
+LORA_CS
+Wire Wire Line
+	2150 3950 2400 3950
+Wire Wire Line
+	2400 3850 2150 3850
+Text Label 20300 2400 0    50   ~ 0
+LORA_IRQ
+Text Label 2150 3550 2    50   ~ 0
+LORA_IRQ
+Wire Wire Line
+	2150 3550 2400 3550
+NoConn ~ 20300 2300
+NoConn ~ 20300 2200
+NoConn ~ 20300 2100
+NoConn ~ 20300 2000
+NoConn ~ 20300 1900
+$Comp
+L Control-Board-rescue:C_Small-device C?
+U 1 1 5C9B0AE5
+P 19700 1350
+F 0 "C?" V 19800 1300 50  0000 L CNN
+F 1 "0.1 uF" V 19600 1400 50  0000 L CNN
+F 2 "Capacitors_SMD:C_0603" H 19700 1350 50  0001 C CNN
+F 3 "" H 19700 1350 50  0001 C CNN
+F 4 "445-5667-1-ND" H 19800 1400 50  0001 C CNN "Digikey Part Number"
+	1    19700 1350
+	0    -1   1    0
+$EndComp
+Connection ~ 19800 1350
+Wire Wire Line
+	19800 1350 19800 1500
+$Comp
+L power:GND #PWR?
+U 1 1 5C9B0F4C
+P 19600 1350
+F 0 "#PWR?" H 19600 1100 50  0001 C CNN
+F 1 "GND" H 19600 1200 50  0000 C CNN
+F 2 "" H 19600 1350 50  0001 C CNN
+F 3 "" H 19600 1350 50  0001 C CNN
+	1    19600 1350
+	0    1    -1   0
+$EndComp
 $EndSCHEMATC
