File: Control Board/Control Board.sch (KiCad schematic (older format))
At the start: 105 parts, among them J10 Conn_01x03, J11 Conn_01x03, J13 Conn_01x03, J14 Conn_01x03, J15 Conn_01x03, J3 RJ45, J4 Conn_01x02, J5 Conn_01x02, J6 Conn_01x03, J7 Conn_01x02, J8 Conn_01x02, J9 Conn_01x02, U1 ATXMEGA128A3-AU, U2 LT1797, U3 LT1797, U4 ISL83490, U5 MAX31856, U6 MAX31856, U7 MAX31856, U8 MAX31856, U9 MAX31856

Commit message: Actually saved the file this time
Parts:
- C1, C10, C12, C14, C15, C17, C19, C2, C20, C22, C24, C25, C27, C29, C3, C30, C32, C34, C35, C4, C5, C7, C8, C9, C? (x4): value 0.1 uF -> 0.1 µF
- C11, C13, C16, C18, C21, C23, C26, C28, C31, C33: value 0.01 uF -> 0.01 µF
- C6: value 10 uF -> 10 µF
- C?: value 0.1 uF -> 10 µF; Digikey Part Number 445-5667-1-ND -> (none)
Changed lines of the file:
@@
 P 15100 2250
 F 0 "C15" H 15110 2320 50  0000 L CNN
-F 1 "0.1 uF" H 15110 2170 50  0000 L CNN
+F 1 "0.1 µF" H 15110 2170 50  0000 L CNN
 F 2 "Capacitors_SMD:C_0603" H 15100 2250 50  0001 C CNN
 F 3 "" H 15100 2250 50  0001 C CNN
@@
 P 13800 2050
 F 0 "C14" H 13810 2120 50  0000 L CNN
-F 1 "0.1 uF" H 13810 1970 50  0000 L CNN
+F 1 "0.1 µF" H 13810 1970 50  0000 L CNN
 F 2 "Capacitors_SMD:C_0603" H 13800 2050 50  0001 C CNN
 F 3 "" H 13800 2050 50  0001 C CNN
@@
 P 13200 1800
 F 0 "C12" H 13210 1870 50  0000 L CNN
-F 1 "0.1 uF" H 13210 1720 50  0000 L CNN
+F 1 "0.1 µF" H 13210 1720 50  0000 L CNN
 F 2 "Capacitors_SMD:C_0603" H 13200 1800 50  0001 C CNN
 F 3 "" H 13200 1800 50  0001 C CNN
@@
 P 13200 1600
 F 0 "C11" H 13210 1670 50  0000 L CNN
-F 1 "0.01 uF" H 13210 1520 50  0000 L CNN
+F 1 "0.01 µF" H 13210 1520 50  0000 L CNN
 F 2 "Capacitors_SMD:C_0603" H 13200 1600 50  0001 C CNN
 F 3 "" H 13200 1600 50  0001 C CNN
@@
 P 13200 2000
 F 0 "C13" H 13210 2070 50  0000 L CNN
-F 1 "0.01 uF" H 13210 1920 50  0000 L CNN
+F 1 "0.01 µF" H 13210 1920 50  0000 L CNN
 F 2 "Capacitors_SMD:C_0603" H 13200 2000 50  0001 C CNN
 F 3 "" H 13200 2000 50  0001 C CNN
@@
 P 15100 3950
 F 0 "C20" H 15110 4020 50  0000 L CNN
-F 1 "0.1 uF" H 15110 3870 50  0000 L CNN
+F 1 "0.1 µF" H 15110 3870 50  0000 L CNN
 F 2 "Capacitors_SMD:C_0603" H 15100 3950 50  0001 C CNN
 F 3 "" H 15100 3950 50  0001 C CNN
@@
 P 13800 3750
 F 0 "C19" H 13810 3820 50  0000 L CNN
-F 1 "0.1 uF" H 13810 3670 50  0000 L CNN
+F 1 "0.1 µF" H 13810 3670 50  0000 L CNN
 F 2 "Capacitors_SMD:C_0603" H 13800 3750 50  0001 C CNN
 F 3 "" H 13800 3750 50  0001 C CNN
@@
 P 13200 3500
 F 0 "C17" H 13210 3570 50  0000 L CNN
-F 1 "0.1 uF" H 13210 3420 50  0000 L CNN
+F 1 "0.1 µF" H 13210 3420 50  0000 L CNN
 F 2 "Capacitors_SMD:C_0603" H 13200 3500 50  0001 C CNN
 F 3 "" H 13200 3500 50  0001 C CNN
@@
 P 13200 3300
 F 0 "C16" H 13210 3370 50  0000 L CNN
-F 1 "0.01 uF" H 13210 3220 50  0000 L CNN
+F 1 "0.01 µF" H 13210 3220 50  0000 L CNN
 F 2 "Capacitors_SMD:C_0603" H 13200 3300 50  0001 C CNN
 F 3 "" H 13200 3300 50  0001 C CNN
@@
 P 13200 3700
 F 0 "C18" H 13210 3770 50  0000 L CNN
-F 1 "0.01 uF" H 13210 3620 50  0000 L CNN
+F 1 "0.01 µF" H 13210 3620 50  0000 L CNN
 F 2 "Capacitors_SMD:C_0603" H 13200 3700 50  0001 C CNN
 F 3 "" H 13200 3700 50  0001 C CNN
@@
 P 15100 5650
 F 0 "C25" H 15110 5720 50  0000 L CNN
-F 1 "0.1 uF" H 15110 5570 50  0000 L CNN
+F 1 "0.1 µF" H 15110 5570 50  0000 L CNN
 F 2 "Capacitors_SMD:C_0603" H 15100 5650 50  0001 C CNN
 F 3 "" H 15100 5650 50  0001 C CNN
@@
 P 13800 5450
 F 0 "C24" H 13810 5520 50  0000 L CNN
-F 1 "0.1 uF" H 13810 5370 50  0000 L CNN
+F 1 "0.1 µF" H 13810 5370 50  0000 L CNN
 F 2 "Capacitors_SMD:C_0603" H 13800 5450 50  0001 C CNN
 F 3 "" H 13800 5450 50  0001 C CNN
@@
 P 13200 5200
 F 0 "C22" H 13210 5270 50  0000 L CNN
-F 1 "0.1 uF" H 13210 5120 50  0000 L CNN
+F 1 "0.1 µF" H 13210 5120 50  0000 L CNN
 F 2 "Capacitors_SMD:C_0603" H 13200 5200 50  0001 C CNN
 F 3 "" H 13200 5200 50  0001 C CNN
@@
 P 13200 5000
 F 0 "C21" H 13210 5070 50  0000 L CNN
-F 1 "0.01 uF" H 13210 4920 50  0000 L CNN
+F 1 "0.01 µF" H 13210 4920 50  0000 L CNN
 F 2 "Capacitors_SMD:C_0603" H 13200 5000 50  0001 C CNN
 F 3 "" H 13200 5000 50  0001 C CNN
@@
 P 13200 5400
 F 0 "C23" H 13210 5470 50  0000 L CNN
-F 1 "0.01 uF" H 13210 5320 50  0000 L CNN
+F 1 "0.01 µF" H 13210 5320 50  0000 L CNN
 F 2 "Capacitors_SMD:C_0603" H 13200 5400 50  0001 C CNN
 F 3 "" H 13200 5400 50  0001 C CNN
@@
 P 15100 7350
 F 0 "C30" H 15110 7420 50  0000 L CNN
-F 1 "0.1 uF" H 15110 7270 50  0000 L CNN
+F 1 "0.1 µF" H 15110 7270 50  0000 L CNN
 F 2 "Capacitors_SMD:C_0603" H 15100 7350 50  0001 C CNN
 F 3 "" H 15100 7350 50  0001 C CNN
@@
 P 13800 7150
 F 0 "C29" H 13810 7220 50  0000 L CNN
-F 1 "0.1 uF" H 13810 7070 50  0000 L CNN
+F 1 "0.1 µF" H 13810 7070 50  0000 L CNN
 F 2 "Capacitors_SMD:C_0603" H 13800 7150 50  0001 C CNN
 F 3 "" H 13800 7150 50  0001 C CNN
@@
 P 13200 6900
 F 0 "C27" H 13210 6970 50  0000 L CNN
-F 1 "0.1 uF" H 13210 6820 50  0000 L CNN
+F 1 "0.1 µF" H 13210 6820 50  0000 L CNN
 F 2 "Capacitors_SMD:C_0603" H 13200 6900 50  0001 C CNN
 F 3 "" H 13200 6900 50  0001 C CNN
@@
 P 13200 6700
 F 0 "C26" H 13210 6770 50  0000 L CNN
-F 1 "0.01 uF" H 13210 6620 50  0000 L CNN
+F 1 "0.01 µF" H 13210 6620 50  0000 L CNN
 F 2 "Capacitors_SMD:C_0603" H 13200 6700 50  0001 C CNN
 F 3 "" H 13200 6700 50  0001 C CNN
@@
 P 13200 7100
 F 0 "C28" H 13210 7170 50  0000 L CNN
-F 1 "0.01 uF" H 13210 7020 50  0000 L CNN
+F 1 "0.01 µF" H 13210 7020 50  0000 L CNN
 F 2 "Capacitors_SMD:C_0603" H 13200 7100 50  0001 C CNN
 F 3 "" H 13200 7100 50  0001 C CNN
@@
 P 15100 9050
 F 0 "C35" H 15110 9120 50  0000 L CNN
-F 1 "0.1 uF" H 15110 8970 50  0000 L CNN
+F 1 "0.1 µF" H 15110 8970 50  0000 L CNN
 F 2 "Capacitors_SMD:C_0603" H 15100 9050 50  0001 C CNN
 F 3 "" H 15100 9050 50  0001 C CNN
@@
 P 13800 8850
 F 0 "C34" H 13810 8920 50  0000 L CNN
-F 1 "0.1 uF" H 13810 8770 50  0000 L CNN
+F 1 "0.1 µF" H 13810 8770 50  0000 L CNN
 F 2 "Capacitors_SMD:C_0603" H 13800 8850 50  0001 C CNN
 F 3 "" H 13800 8850 50  0001 C CNN
@@
 P 13200 8600
 F 0 "C32" H 13210 8670 50  0000 L CNN
-F 1 "0.1 uF" H 13210 8520 50  0000 L CNN
+F 1 "0.1 µF" H 13210 8520 50  0000 L CNN
 F 2 "Capacitors_SMD:C_0603" H 13200 8600 50  0001 C CNN
 F 3 "" H 13200 8600 50  0001 C CNN
@@
 P 13200 8400
 F 0 "C31" H 13210 8470 50  0000 L CNN
-F 1 "0.01 uF" H 13210 8320 50  0000 L CNN
+F 1 "0.01 µF" H 13210 8320 50  0000 L CNN
 F 2 "Capacitors_SMD:C_0603" H 13200 8400 50  0001 C CNN
 F 3 "" H 13200 8400 50  0001 C CNN
@@
 P 13200 8800
 F 0 "C33" H 13210 8870 50  0000 L CNN
-F 1 "0.01 uF" H 13210 8720 50  0000 L CNN
+F 1 "0.01 µF" H 13210 8720 50  0000 L CNN
 F 2 "Capacitors_SMD:C_0603" H 13200 8800 50  0001 C CNN
 F 3 "" H 13200 8800 50  0001 C CNN
@@
 P 3150 1200
 F 0 "C1" H 3100 1750 50  0000 L CNN
-F 1 "0.1 uF" V 3150 1400 50  0000 L CNN
+F 1 "0.1 µF" V 3150 1400 50  0000 L CNN
 F 2 "Capacitors_SMD:C_0603" H 3150 1200 50  0001 C CNN
 F 3 "" H 3150 1200 50  0001 C CNN
@@
 P 2400 1350
 F 0 "C6" H 2410 1420 50  0000 L CNN
-F 1 "10 uF" V 2300 1150 50  0000 L CNN
+F 1 "10 µF" V 2300 1150 50  0000 L CNN
 F 2 "Capacitors_SMD:C_0603" H 2400 1350 50  0001 C CNN
 F 3 "" H 2400 1350 50  0001 C CNN
@@
 P 3250 1200
 F 0 "C2" H 3200 1750 50  0000 L CNN
-F 1 "0.1 uF" V 3250 1400 50  0000 L CNN
+F 1 "0.1 µF" V 3250 1400 50  0000 L CNN
 F 2 "Capacitors_SMD:C_0603" H 3250 1200 50  0001 C CNN
 F 3 "" H 3250 1200 50  0001 C CNN
@@
 P 3350 1200
 F 0 "C3" H 3300 1750 50  0000 L CNN
-F 1 "0.1 uF" V 3350 1400 50  0000 L CNN
+F 1 "0.1 µF" V 3350 1400 50  0000 L CNN
 F 2 "Capacitors_SMD:C_0603" H 3350 1200 50  0001 C CNN
 F 3 "" H 3350 1200 50  0001 C CNN
@@
 P 3450 1200
 F 0 "C4" H 3400 1750 50  0000 L CNN
-F 1 "0.1 uF" V 3450 1400 50  0000 L CNN
+F 1 "0.1 µF" V 3450 1400 50  0000 L CNN
 F 2 "Capacitors_SMD:C_0603" H 3450 1200 50  0001 C CNN
 F 3 "" H 3450 1200 50  0001 C CNN
@@
 P 3550 1200
 F 0 "C5" H 3500 1750 50  0000 L CNN
-F 1 "0.1 uF" V 3550 1400 50  0000 L CNN
+F 1 "0.1 µF" V 3550 1400 50  0000 L CNN
 F 2 "Capacitors_SMD:C_0603" H 3550 1200 50  0001 C CNN
 F 3 "" H 3550 1200 50  0001 C CNN
@@
 P 3850 1400
 F 0 "C7" V 3900 1600 50  0000 L CNN
-F 1 "0.1 uF" V 3850 1600 50  0000 L CNN
+F 1 "0.1 µF" V 3850 1600 50  0000 L CNN
 F 2 "Capacitors_SMD:C_0603" H 3850 1400 50  0001 C CNN
 F 3 "" H 3850 1400 50  0001 C CNN
@@
 P 8650 1850
 F 0 "C8" V 8750 1800 50  0000 L CNN
-F 1 "0.1 uF" V 8550 1900 50  0000 L CNN
+F 1 "0.1 µF" V 8550 1900 50  0000 L CNN
 F 2 "Capacitors_SMD:C_0603" H 8650 1850 50  0001 C CNN
 F 3 "" H 8650 1850 50  0001 C CNN
@@
 P 8650 3500
 F 0 "C9" V 8750 3450 50  0000 L CNN
-F 1 "0.1 uF" V 8550 3550 50  0000 L CNN
+F 1 "0.1 µF" V 8550 3550 50  0000 L CNN
 F 2 "Capacitors_SMD:C_0603" H 8650 3500 50  0001 C CNN
 F 3 "" H 8650 3500 50  0001 C CNN
@@
 P 8450 11250
 F 0 "C10" H 8400 11800 50  0000 L CNN
-F 1 "0.1 uF" V 8450 11450 50  0000 L CNN
+F 1 "0.1 µF" V 8450 11450 50  0000 L CNN
 F 2 "Capacitors_SMD:C_0603" H 8450 11250 50  0001 C CNN
 F 3 "" H 8450 11250 50  0001 C CNN
@@
 P 8650 5200
 F 0 "C?" V 8750 5150 50  0000 L CNN
-F 1 "0.1 uF" V 8550 5250 50  0000 L CNN
+F 1 "0.1 µF" V 8550 5250 50  0000 L CNN
 F 2 "Capacitors_SMD:C_0603" H 8650 5200 50  0001 C CNN
 F 3 "" H 8650 5200 50  0001 C CNN
@@
 P 8650 6850
 F 0 "C?" V 8750 6800 50  0000 L CNN
-F 1 "0.1 uF" V 8550 6900 50  0000 L CNN
+F 1 "0.1 µF" V 8550 6900 50  0000 L CNN
 F 2 "Capacitors_SMD:C_0603" H 8650 6850 50  0001 C CNN
 F 3 "" H 8650 6850 50  0001 C CNN
@@
 P 2750 14000
 F 0 "C?" H 2400 14000 50  0000 L CNN
-F 1 "0.1 uF" H 2400 14100 50  0000 L CNN
+F 1 "0.1 µF" H 2400 14100 50  0000 L CNN
 F 2 "Capacitors_SMD:C_0603" H 2750 14000 50  0001 C CNN
 F 3 "" H 2750 14000 50  0001 C CNN
@@
 P 2600 14000
 F 0 "C?" H 2250 14000 50  0000 L CNN
-F 1 "0.1 uF" H 2250 14100 50  0000 L CNN
+F 1 "0.1 µF" H 2250 14100 50  0000 L CNN
 F 2 "Capacitors_SMD:C_0603" H 2600 14000 50  0001 C CNN
 F 3 "" H 2600 14000 50  0001 C CNN
@@
 P 19700 1350
 F 0 "C?" V 19800 1300 50  0000 L CNN
-F 1 "0.1 uF" V 19600 1400 50  0000 L CNN
+F 1 "10 µF" V 19600 1400 50  0000 L CNN
 F 2 "Capacitors_SMD:C_0603" H 19700 1350 50  0001 C CNN
 F 3 "" H 19700 1350 50  0001 C CNN
-F 4 "445-5667-1-ND" H 19800 1400 50  0001 C CNN "Digikey Part Number"
 	1    19700 1350
 	0    -1   1    0

Commit message: Create Safing Remote Project
Parts:
- added AE?: Antenna, symbol Device:Antenna
- U?: value RFM96W-315S2 -> RFM95W-915S2; Digikey Part Number (none) -> RFM95W-915S2-ND
Changed lines of the file:
@@
 P 19800 2000
 F 0 "U?" H 19950 2550 50  0000 C CNN
-F 1 "RFM96W-315S2" H 20150 2450 50  0000 C CNN
+F 1 "RFM95W-915S2" H 20150 2450 50  0000 C CNN
 F 2 "" H 16500 3650 50  0001 C CNN
 F 3 "http://www.hoperf.com/upload/rf/RFM95_96_97_98W.pdf" H 16500 3650 50  0001 C CNN
+F 4 "RFM95W-915S2-ND" H 19800 2000 50  0001 C CNN "Digikey Part Number"
 	1    19800 2000
 	1    0    0    -1
@@
 	0    1    -1   0
 $EndComp
+$Comp
+L Device:Antenna AE?
+U 1 1 5C9B331C
+P 21500 1500
+F 0 "AE?" H 21580 1491 50  0000 L CNN
+F 1 "Antenna" H 21580 1400 50  0000 L CNN
+F 2 "" H 21500 1500 50  0001 C CNN
+F 3 "~" H 21500 1500 50  0001 C CNN
+F 4 "WM9671-ND" H 21500 1500 50  0001 C CNN "Digikey Part Number"
+	1    21500 1500
+	1    0    0    -1
+$EndComp
 $EndSCHEMATC

Commit message: Finished annotating
Other:
- note added: "Backup Radio:\nSends critical safety information so that the rocket state is known even if\nthe main comms fail. Uses a low cost, low power, long range LoRa\ntransciever. Capable of recieving commands too, if that functionality ends\nup being needed."
- note added: "Connector:\nConnects to the other boards in the avionics stack"
- note added: "Data Logger:\nLogs data to an SD card, kinda like a black box. If it blows up hopefully\nthis will tell us why."
- note added: "Inter-Board Comms:\nRS422 transciever to communicate between uper and lower avionics.\nUses Cat5 cable, which isn't standard for RS422, so the design had to be\nmodified a bit from standard."
- note added: "LEDs:\nBlinky blinky"
- note added: "MCU:\nDoes all the controlly thinky mathy stuff"
- note added: "Mounting holes and logo:\nMounting holes and logo"
- note added: "PT Op-Amps:\nThe Pressure Transducers (PTs) like to have a very high input impedance\non the device connected to their output in order to output the right\nvoltage. (Think of input impedance as the resistance between the input\nand ground. That's a major oversimplification for a lot of circuits, but\nworks okay enough here.) The voltage they output is too high for the\nMCU, so it has to go into a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"
- note added: "PT and TC Connectors:\nConnects to the pressure transducers and thermocouples"
- note added: "Servo Connections:\nConnecting the PWM outputs of the MCU to the servo inputs. There used\nto be a lot more here."
- note added: "Servo Connectors:\nConnectors for the servos and associated limit switches"
- note added: "Thermocouple Amplifiers:\nThese configurable thermocouple amplifiers output the temperature on\nthe connected thermocouples, and are configurable to use almost any\ntype of thermocouple."
- moved on the sheet: U?

Commit message: Added KiBOM, started work on control board
Parts:
- R11: renamed from R?; footprint (none) -> Resistors_SMD:R_0603; Digikey Part Number (none) -> 311-10.0KHRCT-ND
- gave numbers to parts that had none: 26

Commit message: Started control board part numbering
Parts:
- C38: Digikey Part Number (none) -> 1276-1038-1-ND
- C6: Digikey Part Number 490-12323-1-ND -> 1276-1038-1-ND
Changed lines of the file:
@@
 F 2 "Capacitors_SMD:C_0603" H 2400 2300 50  0001 C CNN
 F 3 "" H 2400 2300 50  0001 C CNN
-F 4 "490-12323-1-ND" H 2410 2470 50  0001 C CNN "Digikey Part Number"
+F 4 "1276-1038-1-ND" H 2410 2470 50  0001 C CNN "Digikey Part Number"
 	1    2400 2300
 	0    1    1    0
@@
 F 2 "Capacitors_SMD:C_0603" H 11500 12850 50  0001 C CNN
 F 3 "" H 11500 12850 50  0001 C CNN
+F 4 "1276-1038-1-ND" H 0   0   50  0001 C CNN "Digikey Part Number"
 	1    11500 12850
 	0    -1   1    0
@@
 F 1 "Antenna" H 13380 12900 50  0000 L CNN
 F 2 "" H 13300 13000 50  0001 C CNN
-F 3 "~" H 13300 13000 50  0001 C CNN
+F 3 "" H 13300 13000 50  0001 C CNN
 F 4 "WM9671-ND" H 13300 13000 50  0001 C CNN "Digikey Part Number"
 	1    13300 13000

Commit message: Finished Control Board Part Numbers
Parts:
- C1, C10, C12, C14, C15, C17, C19, C2, C20, C22, C24, C25, C27, C29, C3, C30, C32, C34, C35, C36, C37, C39, C4, C40, C5, C7, C8, C9: Digikey Part Number 445-5667-1-ND -> 1276-6717-6-ND
- C11, C13, C16, C18, C21, C23, C26, C28, C31, C33: Digikey Part Number 399-1091-1-ND -> 1276-1921-1-ND
- J1: Digikey Part Number (none) -> 609-3693-1-ND
- J12: Digikey Part Number (none) -> WM24066CT-ND
- J18: Digikey Part Number (none) -> 952-2217-ND
- J2: Digikey Part Number (none) -> H9161CT-ND
- R1, R10, R11, R2, R23, R24, R25, R5: Digikey Part Number 311-10.0KHRCT-ND -> P10.0KHCT-ND
- R12: Digikey Part Number (none) -> P330HCT-ND
- R13: Digikey Part Number (none) -> P1.00KHCT-ND
- R22: Digikey Part Number 311-100HRCT-ND -> P100HCT-ND
- R3, R4: Digikey Part Number (none) -> P220HCT-ND
- R6, R7, R8, R9: Digikey Part Number 311-100GRCT-ND -> P100HCT-ND
- U10, U11, U2, U3: value LT1797 -> LT6200; footprint TO_SOT_Packages_SMD:TSOT-23-5 -> TO_SOT_Packages_SMD:TSOT-23-6; symbol Custom-Parts:LT1797 -> Custom-Parts:LT6200; Digikey Part Number LT1797CS5#TRMPBFCT-ND -> LT6200CS6-5#TRMPBFCT-ND

Commit message: Associated a few control board footprints
Parts:
- J18: footprint (none) -> Pin_Headers:Pin_Header_Straight_1x07_Pitch2.54mm
- J2: footprint U.FL -> (none)
- R12, R13, R3, R4: footprint (none) -> Resistors_SMD:R_0603
Changed lines of the file:
@@
 F 0 "J18" H 13950 20967 50  0000 C CNN
 F 1 "Conn_02x07_Counter_Clockwise" H 13950 20876 50  0000 C CNN
-F 2 "" H 13900 20450 50  0001 C CNN
+F 2 "Pin_Headers:Pin_Header_Straight_1x07_Pitch2.54mm" H 13900 20450 50  0001 C CNN
 F 3 "~" H 13900 20450 50  0001 C CNN
 F 4 "952-2217-ND" H 0   0   50  0001 C CNN "Digikey Part Number"
@@
 F 0 "R13" H 5609 20296 50  0000 L CNN
 F 1 "1 kΩ" H 5609 20205 50  0000 L CNN
-F 2 "" H 5550 20250 50  0001 C CNN
+F 2 "Resistors_SMD:R_0603" H 5550 20250 50  0001 C CNN
 F 3 "~" H 5550 20250 50  0001 C CNN
 F 4 "P1.00KHCT-ND" H 0   0   50  0001 C CNN "Digikey Part Number"
@@
 F 0 "R12" H 5209 20296 50  0000 L CNN
 F 1 "330 Ω" H 5209 20205 50  0000 L CNN
-F 2 "" H 5150 20250 50  0001 C CNN
+F 2 "Resistors_SMD:R_0603" H 5150 20250 50  0001 C CNN
 F 3 "~" H 5150 20250 50  0001 C CNN
 F 4 "P330HCT-ND" H 0   0   50  0001 C CNN "Digikey Part Number"
@@
 F 0 "R3" V 3454 9600 50  0000 C CNN
 F 1 "220 Ω" V 3545 9600 50  0000 C CNN
-F 2 "" H 3650 9600 50  0001 C CNN
+F 2 "Resistors_SMD:R_0603" H 3650 9600 50  0001 C CNN
 F 3 "~" H 3650 9600 50  0001 C CNN
 F 4 "P220HCT-ND" H 0   0   50  0001 C CNN "Digikey Part Number"
@@
 F 0 "R4" V 3846 9800 50  0000 C CNN
 F 1 "220 Ω" V 3755 9800 50  0000 C CNN
-F 2 "" H 3650 9800 50  0001 C CNN
+F 2 "Resistors_SMD:R_0603" H 3650 9800 50  0001 C CNN
 F 3 "~" H 3650 9800 50  0001 C CNN
 F 4 "P220HCT-ND" H 0   0   50  0001 C CNN "Digikey Part Number"
@@
 F 0 "J2" H 12750 13560 45  0000 C CNN
 F 1 "U.FL" H 12750 13476 45  0000 C CNN
-F 2 "U.FL" H 12700 13450 20  0001 C CNN
+F 2 "" H 12700 13450 20  0001 C CNN
 F 3 "" H 12700 13200 50  0001 C CNN
 F 4 "CONN-09193" H 12750 13381 60  0000 C CNN "Field4"

Commit message: Started on control board footprints
Parts:
- J1: footprint (none) -> Control_Board_Footprints:PDI_CONNECTOR
- J2: footprint (none) -> Control_Board_Footprints:U.FL_SMD_CONNECTOR
Changed lines of the file:
@@
 F 0 "J1" H 3500 7467 50  0000 C CNN
 F 1 "Conn_02x03_Odd_Even" H 3500 7376 50  0000 C CNN
-F 2 "" H 3450 7150 50  0001 C CNN
+F 2 "Control_Board_Footprints:PDI_CONNECTOR" H 3450 7150 50  0001 C CNN
 F 3 "~" H 3450 7150 50  0001 C CNN
 F 4 "609-3693-1-ND" H 0   0   50  0001 C CNN "Digikey Part Number"
@@
 F 0 "J2" H 12750 13560 45  0000 C CNN
 F 1 "U.FL" H 12750 13476 45  0000 C CNN
-F 2 "" H 12700 13450 20  0001 C CNN
+F 2 "Control_Board_Footprints:U.FL_SMD_CONNECTOR" H 12700 13450 20  0001 C CNN
 F 3 "" H 12700 13200 50  0001 C CNN
 F 4 "CONN-09193" H 12750 13381 60  0000 C CNN "Field4"
