File: Control Board/Control Board.kicad_pcb (KiCad board)
At the start: 2 copper layers, 135 parts, among them J1 Conn_02x03_Odd_Even, J2 Conn_02x35_Counter_Clockwise, Q1 SI7135DP, Q2 SI7135DP, Q3 SI7135DP, Q4 SI7135DP, Q5 SI7135DP, Q6 SI7135DP, Q7 STS4DNF60L, Q8 STS4DNF60L, SW1 SW_SPDT, U1 LTC4417CGN, U10 MAX31856, U11 MAX31856, U12 MAX31856, U13 MAX31856, U2 TPS54308DDC, U3 TPS54308DDC, U4 TPS54308DDC, U5 ATXMEGA128A3-AU, U6 LT1797, U7 LT1797, U8 ISL83490, U9 MAX31856

Commit message: Routed Or Controller
Parts:
- added REF**: VIA_0.52mm, Custom Footprints:VIA_0.52mm, F.Cu at (64.3, 110.7)
- added REF**: VIA_0.52mm, Custom Footprints:VIA_0.52mm, F.Cu at (61.7, 97.5)
- added REF**: VIA_0.52mm, Custom Footprints:VIA_0.52mm, F.Cu at (60.2, 97.5)
- added REF**: VIA_0.52mm, Custom Footprints:VIA_0.52mm, F.Cu at (60.2, 96.3)
- added REF**: VIA_0.52mm, Custom Footprints:VIA_0.52mm, F.Cu at (59.2, 96.3)
- added REF**: VIA_0.52mm, Custom Footprints:VIA_0.52mm, F.Cu at (59.2, 97.5)
- added REF**: VIA_0.52mm, Custom Footprints:VIA_0.52mm, F.Cu at (57.1, 129.0)
- added REF**: VIA_0.52mm, Custom Footprints:VIA_0.52mm, F.Cu at (56.1, 129.0)
- added REF**: VIA_0.52mm, Custom Footprints:VIA_0.52mm, F.Cu at (56.1, 128.0)
- added REF**: VIA_0.52mm, Custom Footprints:VIA_0.52mm, F.Cu at (57.1, 128.0)
- added REF**: VIA_0.52mm, Custom Footprints:VIA_0.52mm, F.Cu at (57.1, 127.0)
- added REF**: VIA_0.52mm, Custom Footprints:VIA_0.52mm, F.Cu at (65.3, 110.7)
- added REF**: VIA_0.52mm, Custom Footprints:VIA_0.52mm, F.Cu at (56.1, 127.0)
- added REF**: VIA_0.52mm, Custom Footprints:VIA_0.52mm, F.Cu at (72.9, 115.6)
- added REF**: VIA_0.52mm, Custom Footprints:VIA_0.52mm, F.Cu at (71.9, 115.6)
- added REF**: VIA_0.52mm, Custom Footprints:VIA_0.52mm, F.Cu at (71.9, 114.6)
- added REF**: VIA_0.52mm, Custom Footprints:VIA_0.52mm, F.Cu at (72.9, 114.6)
- added REF**: VIA_0.52mm, Custom Footprints:VIA_0.52mm, F.Cu at (72.9, 113.5)
- added REF**: VIA_0.52mm, Custom Footprints:VIA_0.52mm, F.Cu at (71.9, 113.5)
- added REF**: VIA_0.52mm, Custom Footprints:VIA_0.52mm, F.Cu at (62.9, 116.2)
- added REF**: VIA_0.52mm, Custom Footprints:VIA_0.52mm, F.Cu at (61.7, 116.2)
- added REF**: VIA_0.52mm, Custom Footprints:VIA_0.52mm, F.Cu at (60.2, 116.2)
- added REF**: VIA_0.52mm, Custom Footprints:VIA_0.52mm, F.Cu at (64.3, 108.7)
- added REF**: VIA_0.52mm, Custom Footprints:VIA_0.52mm, F.Cu at (59.1, 116.2)
- added REF**: VIA_0.52mm, Custom Footprints:VIA_0.52mm, F.Cu at (62.9, 114.9)
- added REF**: VIA_0.52mm, Custom Footprints:VIA_0.52mm, F.Cu at (61.7, 114.9)
- added REF**: VIA_0.52mm, Custom Footprints:VIA_0.52mm, F.Cu at (60.2, 114.9)
- added REF**: VIA_0.52mm, Custom Footprints:VIA_0.52mm, F.Cu at (59.1, 114.9)
- added REF**: VIA_0.52mm, Custom Footprints:VIA_0.52mm, F.Cu at (65.3, 108.7)
- added REF**: VIA_0.52mm, Custom Footprints:VIA_0.52mm, F.Cu at (65.3, 109.7)
- added REF**: VIA_0.52mm, Custom Footprints:VIA_0.52mm, F.Cu at (64.3, 109.7)
- added REF**: VIA_0.52mm, Custom Footprints:VIA_0.52mm, F.Cu at (62.7, 97.5)
- added REF**: VIA_0.52mm, Custom Footprints:VIA_0.52mm, F.Cu at (62.7, 96.3)
- added REF**: VIA_0.52mm, Custom Footprints:VIA_0.52mm, F.Cu at (61.7, 96.3)
- moved C6 212.4 mm to (81.8, 106.2), turned to 270 degrees
- moved C4 199.8 mm to (88.6, 104.9), turned to 90 degrees
- moved C2 197.3 mm to (85.3, 106.2), turned to 90 degrees
- moved D3 195.5 mm to (70.2, 123.8), turned to 180 degrees
- moved C3 191.7 mm to (86.9, 104.9), turned to 90 degrees
- moved D1 191.4 mm to (74.5, 118.1)
- moved C5 186.6 mm to (80.0, 106.2), turned to 270 degrees
- moved D4 185.6 mm to (62.0, 118.1), turned to 180 degrees
- moved R2 177.8 mm to (86.2, 117.7)
- moved R29 158.9 mm to (133.1, 118.4)
- moved C7 156.4 mm to (83.6, 106.2), turned to 270 degrees
- moved R30 154.8 mm to (133.1, 113.5)
- moved Q3 149.8 mm to (68.6, 110.5), turned to 270 degrees
- moved R8 149.2 mm to (90.1, 122.8)
- moved R27 149.1 mm to (133.4, 122.2)
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Connections:
- J2 pad 10: /BAT_VCC -> /UMB_VCC
- J2 pad 11: /BAT_VCC -> /UMB_VCC
- J2 pad 12: /BAT_VCC -> /UMB_VCC
- J2 pad 5: /UMB_VCC -> /BAT_VCC
- J2 pad 6: /UMB_VCC -> /BAT_VCC
- J2 pad 7: /UMB_VCC -> /BAT_VCC
- J2 pad 8: /UMB_VCC -> /BAT_VCC
- J2 pad 9: /BAT_VCC -> /UMB_VCC
Routing:
- net /BAT_BAK_VCC: track 0.00 -> 53.7 mm, vias 0 -> 2
- net /BAT_VCC: track 0.00 -> 42.8 mm, vias 0 -> 3
- net Net-(Q5-Pad2): track 0.00 -> 37.7 mm, vias 0 -> 3
- net Net-(C4-Pad1): track 0.00 -> 32.6 mm, vias 0 -> 2
- net +14V: track 0.00 -> 30.3 mm, vias 0 -> 2
- net /UMB_VCC: track 0.00 -> 30.0 mm, vias 0 -> 2
- net Net-(Q3-Pad2): track 0.00 -> 27.9 mm, vias 0 -> 3
- net Net-(C3-Pad1): track 0.00 -> 22.6 mm, vias 0 -> 2
- net Net-(Q1-Pad2): track 0.00 -> 18.3 mm, vias 0 -> 3
- net Net-(R8-Pad2): track 0.00 -> 11.0 mm, vias 0 -> 2
- net Net-(R7-Pad1): track 0.00 -> 10.3 mm, vias 0 -> 2
- net Net-(C2-Pad1): track 0.00 -> 10.1 mm, vias 0 -> 2
- net Net-(R5-Pad2): track 0.00 -> 8.40 mm, vias 0 -> 2
- net Net-(R4-Pad1): track 0.00 -> 7.85 mm, vias 0 -> 2
- net Net-(R2-Pad2): track 0.00 -> 5.34 mm
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- added copper zone on B.Cu, net +14V
- added copper zone on F.Cu, net +14V
- added copper zone on B.Cu, net /BAT_BAK_VCC
- added copper zone on F.Cu, net /BAT_BAK_VCC
- added copper zone on F.Cu, net /BAT_VCC
- added copper zone on F.Cu, net /UMB_VCC
- added copper zone on B.Cu, net GND
- added copper zone on F.Cu, net GND
- added copper zone on F.Cu, net Net-(C2-Pad1)
- added copper zone on F.Cu, net Net-(C3-Pad1)
- added copper zone on F.Cu, net Net-(C4-Pad1)
Other:
- net class Default: trace_width 0.25 -> 0.2; via_dia 0.6 -> 0.66
- net class High Power added: clearance 0.2, trace_width 5, via_dia 0.66, via_drill 0.4
- net class Low Power added: clearance 0.2, trace_width 1, via_dia 0.66, via_drill 0.4
- net class Mid Power added: clearance 0.2, trace_width 0.3, via_dia 0.66, via_drill 0.4
- net class Small added: clearance 0.13, trace_width 0.13, via_dia 0.52, via_drill 0.25
- rule trace_min: 0.2 -> 0.13
- rule via_min_drill: 0.3 -> 0.25
- rule via_min_size: 0.4 -> 0.51

Commit message: More routing
Parts:
- added REF**: VIA_0.52mm, Custom Footprints:VIA_0.52mm, F.Cu at (52.7, 129.2)
- added REF**: VIA_0.66mm, Custom Footprints:VIA_0.66mm, F.Cu at (61.3, 87.9)
- added REF**: VIA_0.52mm, Custom Footprints:VIA_0.52mm, F.Cu at (51.8, 129.2)
- added REF**: VIA_0.52mm, Custom Footprints:VIA_0.52mm, F.Cu at (53.7, 130.2)
- added REF**: VIA_0.52mm, Custom Footprints:VIA_0.52mm, F.Cu at (51.8, 128.3)
- added REF**: VIA_0.66mm, Custom Footprints:VIA_0.66mm, F.Cu at (61.3, 87.0)
- added REF**: VIA_0.52mm, Custom Footprints:VIA_0.52mm, F.Cu at (51.8, 130.2)
- added REF**: VIA_0.52mm, Custom Footprints:VIA_0.52mm, F.Cu at (52.7, 130.2)
- added REF**: VIA_0.66mm, Custom Footprints:VIA_0.66mm, F.Cu at (61.3, 69.8)
- added REF**: VIA_0.66mm, Custom Footprints:VIA_0.66mm, F.Cu at (61.3, 89.9)
- added REF**: VIA_0.66mm, Custom Footprints:VIA_0.66mm, F.Cu at (61.3, 88.9)
- moved C17 224.8 mm to (67.0, 61.0)
- moved R11 222.2 mm to (73.7, 82.9), turned to 180 degrees
- moved L2 215.6 mm to (58.1, 66.0), turned to 90 degrees
- moved R13 214.4 mm to (73.7, 65.7), turned to 180 degrees
- moved C16 213.0 mm to (67.0, 63.5)
- moved C14 196.4 mm to (66.7, 71.4), turned to 90 degrees
- moved C10 194.8 mm to (68.9, 88.6), turned to 90 degrees
- moved C9 193.6 mm to (66.7, 88.6), turned to 90 degrees
- moved C15 190.1 mm to (68.9, 71.4), turned to 90 degrees
- moved C13 188.5 mm to (73.0, 67.9), turned to 180 degrees
- moved C12 187.1 mm to (67.0, 80.6)
- moved C8 185.0 mm to (73.0, 85.1), turned to 180 degrees
- moved C11 184.6 mm to (67.0, 78.1)
- moved R12 174.9 mm to (73.7, 63.8)
- moved U4 164.2 mm to (69.7, 28.9)
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Routing:
- net +3V3: track 0.00 -> 18.5 mm, vias 0 -> 2
- net /XBEE_VCC: track 0.00 -> 16.3 mm, vias 0 -> 2
- net Net-(R10-Pad2): track 0.00 -> 10.2 mm
- net Net-(R12-Pad2): track 0.00 -> 9.96 mm
- net +14V: track 30.3 -> 36.6 mm
- net Net-(C8-Pad2): track 0.00 -> 5.67 mm, vias 0 -> 4
- net Net-(C13-Pad2): track 0.00 -> 5.67 mm, vias 0 -> 4
- net /TC2_T+: track 0.00 -> 4.25 mm
- net Net-(C13-Pad1): track 0.00 -> 2.98 mm
- net Net-(C8-Pad1): track 0.00 -> 2.98 mm
- net /TC1_T-: track 0.00 -> 1.31 mm
- added copper zone on F.Cu, net +3V3
- added copper zone on F.Cu, net /XBEE_VCC
- added copper zone on B.Cu, net Net-(C13-Pad2)
- added copper zone on F.Cu, net Net-(C13-Pad2)
- added copper zone on B.Cu, net Net-(C8-Pad2)
- added copper zone on F.Cu, net Net-(C8-Pad2)
Other:
- board outline added: 91.4 x 53.3 mm

Commit message: More routing
Parts:
- moved C18 249.3 mm to (39.1, 23.9)
- moved C21 244.0 mm to (39.6, 40.6)
- moved C20 241.2 mm to (39.4, 35.6)
- moved C19 231.0 mm to (39.1, 29.2)
- moved R14 220.2 mm to (34.0, 31.5)
- moved SW1 200.2 mm to (101.6, 25.4), turned to 180 degrees
- moved D2 189.9 mm to (83.8, 94.0)
- moved R15 181.7 mm to (33.8, 35.8)
- moved C1 180.3 mm to (102.9, 91.9), turned to 180 degrees
- moved R21 162.6 mm to (170.2, 15.5), turned to 270 degrees
- moved R23 161.8 mm to (113.8, 100.3)
- moved R20 159.4 mm to (132.8, 55.4), turned to 180 degrees
- moved R22 157.2 mm to (170.2, 18.3), turned to 270 degrees
- moved C54 148.5 mm to (236.0, 7.87), turned to 90 degrees
- moved C52 144.1 mm to (236.0, 10.9), turned to 90 degrees
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Connections:
- C29 pad 2: Net-(C29-Pad2) -> +12V
- C30 pad 2: Net-(C30-Pad2) -> +12V
Routing:
- net +3V3: track 18.5 -> 23.8 mm
- net /TC2_T+: track 4.25 -> 0.00 mm

Commit message: Removed power supply from control board
Parts:
- removed the C1 at (102.9, 91.9)
- removed the C10 at (118.6, 90.2)
- removed the C11 at (120.5, 100.7)
- removed the C12 at (120.5, 98.2)
- removed the C13 at (114.4, 110.9)
- removed the C14 at (120.8, 107.4)
- removed the C15 at (118.6, 107.4)
- removed the C16 at (120.5, 115.3)
- removed the C17 at (120.5, 117.9)
- removed the C18 at (39.1, 23.9)
- removed the C19 at (39.1, 29.2)
- removed the C2 at (85.3, 106.2)
- removed the C20 at (39.4, 35.6)
- removed the C21 at (39.6, 40.6)
- removed the C3 at (86.9, 104.9)
- removed the C4 at (88.6, 104.9)
- removed the C5 at (80.0, 106.2)
- removed the C6 at (81.8, 106.2)
- removed the C7 at (83.6, 106.2)
- removed the C8 at (114.4, 93.7)
- removed the C9 at (120.8, 90.2)
- removed the D2 at (83.8, 94.0)
- removed the D3 at (70.2, 123.8)
- removed the D4 at (62.0, 118.1)
- removed D5: LED_R, LEDs:LED_0603
- removed the L1 at (129.3, 95.6)
- removed L2: 18 uH, Inductors_SMD:L_Wuerth_HCI-1365
- removed L3: 16 uH, Inductors_SMD:L_Wuerth_HCI-1050
- removed the Q1 at (76.2, 110.5)
- removed the Q2 at (76.2, 101.6)
- removed Q3, Q4, Q5, Q6: SI7135DP, Custom Footprints:PowerPAK_SO-8
- removed the R1 at (83.0, 117.7)
- removed the R10 at (113.8, 97.9)
- removed the R11 at (113.8, 95.9)
- removed the R12 at (113.8, 115.0)
- removed the R13 at (113.8, 113.1)
- removed the R14 at (34.0, 31.5)
- removed the R15 at (33.8, 35.8)
- removed the R2 at (86.2, 117.7)
- removed the R23 at (113.8, 100.3)
- removed the R3 at (89.4, 117.7)
- removed the R4 at (85.0, 120.3)
- removed the R5 at (88.2, 120.3)
- removed the R6 at (91.3, 120.3)
- removed the R7 at (86.9, 122.8)
- removed the R9 at (93.3, 122.8)
- removed REF** (x40): VIA_0.52mm, Custom Footprints:VIA_0.52mm
- removed REF** (x5): VIA_0.66mm, Custom Footprints:VIA_0.66mm
- removed the U1 at (87.1, 111.8)
- removed the U2 at (113.5, 90.2)
- removed the U3 at (113.5, 107.4)
- removed the U4 at (31.0, 40.1)
- D1: value SMBJ26CA -> LED_R; footprint Diodes_SMD:D_SMB -> LEDs:LED_0603
- J2: value Conn_02x35_Counter_Clockwise -> Conn_02x25_Counter_Clockwise; footprint Custom Footprints:CONN_CARD_02x35_MALE -> Custom Footprints:CONN_CARD_02x25_MALE
- R8: value 2.49 kΩ -> 100 Ω
- moved D1 36.1 mm to (94.0, 148.5)
- moved R8 26.0 mm to (94.0, 148.5)
- renumbered C22 to C1, C31 to C10, C32 to C11, C33 to C12, C34 to C13, C35 to C14, C36 to C15, C37 to C16, C38 to C17, C39 to C18, C40 to C19, C23 to C2, C41 to C20, C42 to C21, C43 to C22, C44 to C23, C45 to C24, C46 to C25, C47 to C26, C48 to C27, C49 to C28, C50 to C29, C24 to C3, C51 to C30, C52 to C31, C53 to C32, C54 to C33, C55 to C34, C56 to C35, C25 to C4, C26 to C5, C27 to C6, C28 to C7, C29 to C8, C30 to C9, D6 to D2, D7 to D3, D8 to D4, L4 to L1, Q7 to Q1, Q8 to Q2, R16 to R1, R25 to R10, R26 to R11, R27 to R12, R28 to R13, R29 to R14, R30 to R15, R31 to R16, R32 to R17, R33 to R18, R34 to R19, R17 to R2, R35 to R20, R36 to R21, R37 to R22, R38 to R23, R39 to R24, R18 to R3, R19 to R4, R20 to R5, R21 to R6, R22 to R7, R24 to R9, U5 to U1, U6 to U2, U7 to U3, U8 to U4, U9 to U5, U10 to U6, U11 to U7, U12 to U8, U13 to U9
Connections:
- D1 pad 1: GND -> Net-(D1-Pad1)
- D1 pad 2: /UMB_VCC -> +3V3
- J1 pad 3: Net-(J1-Pad3) -> (no net)
- J1 pad 4: Net-(J1-Pad4) -> (no net)
- J2 pad 1: +3V3 -> +12V
- J2 pad 10: /UMB_VCC -> GND
- J2 pad 11: /UMB_VCC -> /GPS_RX
- J2 pad 12: /UMB_VCC -> /GPS_TX
- J2 pad 13: GND -> /GNC_RX
- J2 pad 14: /BOARD_TX+ -> /GNC_TX
- J2 pad 15: GND -> /XBEE_RX
- J2 pad 16: /BOARD_RX+ -> /XBEE_TX
- J2 pad 18: /GPS_RX -> GND
- J2 pad 19: /GPS_TX -> /TC1_T-
- J2 pad 20: GND -> /TC1_T+
- J2 pad 21: /GNC_RX -> /TC2_T-
- J2 pad 22: /GNC_TX -> /TC2_T+
- J2 pad 23: GND -> /TC3_T-
- J2 pad 24: /XBEE_RX -> /TC3_T+
- J2 pad 25: /XBEE_TX -> GND
- J2 pad 27: GND -> /TC5_T+
- J2 pad 28: GND -> /TC5_T-
- J2 pad 29: /TC1_T- -> /TC4_T+
- J2 pad 3: /XBEE_VCC -> (no net)
- J2 pad 30: /TC1_T+ -> /TC4_T-
- J2 pad 31: /TC2_T- -> /PT2_IN
- J2 pad 32: /TC2_T+ -> /PT1_IN
- J2 pad 33: /TC3_T- -> GND
- J2 pad 34: /TC3_T+ -> GND
- J2 pad 35: GND -> /SERVO1_CL_SW
- J2 pad 36: GND -> /SERVO1_OP_SW
- J2 pad 37: /TC5_T+ -> /SERVO2_CL_SW
- J2 pad 38: /TC5_T- -> /SERVO2_OP_SW
- J2 pad 39: /TC4_T+ -> /GNC_INST
- J2 pad 4: GND -> /BAT_VCC
- J2 pad 40: /TC4_T- -> GND
- J2 pad 41: /PT2_IN -> GND
- J2 pad 42: /PT1_IN -> /BOARD_RX-
- J2 pad 44: +12V -> /BOARD_TX-
- J2 pad 46: GND -> /BAT_BAK_VCC
- J2 pad 47: GND -> /VCC_IN
- J2 pad 48: /SERVO1_CL_SW -> GND
- J2 pad 49: /SERVO1_OP_SW -> +3V3
- J2 pad 5: /BAT_VCC -> /UMB_VCC
- J2 pad 50: /SERVO2_CL_SW -> GND
- J2 pad 6: /BAT_VCC -> GND
- J2 pad 7: /BAT_VCC -> /BOARD_TX+
- J2 pad 8: /BAT_VCC -> GND
- J2 pad 9: /UMB_VCC -> /BOARD_RX+
- R20 pad 1: +14V -> /VCC_IN
- R8 pad 1: Net-(R7-Pad1) -> Net-(D1-Pad1)
- R8 pad 2: Net-(R8-Pad2) -> GND
- U1 pad 58: Net-(U5-Pad58) -> (no net)
- U1 pad 59: Net-(U5-Pad59) -> (no net)
- U1 pad 7: Net-(U5-Pad7) -> (no net)
Routing:
- net /BAT_BAK_VCC: track 53.7 -> 0.00 mm, vias 2 -> 0
- net /BAT_VCC: track 42.8 -> 0.00 mm, vias 3 -> 0
- net Net-(Q5-Pad2): track 37.7 -> 0.00 mm, vias 3 -> 0
- net +14V: track 36.4 -> 0.00 mm, vias 2 -> 0
- net Net-(C4-Pad1): track 32.6 -> 0.00 mm, vias 2 -> 0
- net /UMB_VCC: track 30.0 -> 0.00 mm, vias 2 -> 0
- net Net-(Q3-Pad2): track 27.9 -> 0.00 mm, vias 3 -> 0
- net +3V3: track 23.8 -> 0.00 mm, vias 2 -> 0
- net Net-(C3-Pad1): track 22.6 -> 0.00 mm, vias 2 -> 0
- net Net-(Q1-Pad2): track 18.3 -> 0.00 mm, vias 3 -> 0
- net /XBEE_VCC: track 16.3 -> 0.00 mm, vias 2 -> 0
- net Net-(R8-Pad2): track 11.0 -> 0.00 mm, vias 2 -> 0
- net Net-(R7-Pad1): track 10.3 -> 0.00 mm, vias 2 -> 0
- net Net-(R10-Pad2): track 10.2 -> 0.00 mm
- net Net-(C2-Pad1): track 10.1 -> 0.00 mm, vias 2 -> 0
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- removed copper zone on B.Cu, net +14V
- removed copper zone on F.Cu, net +14V
- removed copper zone on F.Cu, net +3V3
- removed copper zone on B.Cu, net /BAT_BAK_VCC
- removed copper zone on F.Cu, net /BAT_BAK_VCC
- removed copper zone on F.Cu, net /BAT_VCC
- removed copper zone on F.Cu, net /UMB_VCC
- removed copper zone on F.Cu, net /XBEE_VCC
- removed copper zone on B.Cu, net Net-(C13-Pad2)
- removed copper zone on F.Cu, net Net-(C13-Pad2)
- removed copper zone on F.Cu, net Net-(C2-Pad1)
- removed copper zone on F.Cu, net Net-(C3-Pad1)
- removed copper zone on F.Cu, net Net-(C4-Pad1)
- removed copper zone on B.Cu, net Net-(C8-Pad2)
- removed copper zone on F.Cu, net Net-(C8-Pad2)

Commit message: Removed buzzer, changed board sizes
Parts:
- removed BZ1: AI-1223-TWT-12V-R, Buzzers_Beepers:Buzzer_12x9.5RM7.6
- removed BZ2: AI-1441-TWT-12V-R, Buzzers_Beepers:Buzzer_12x9.5RM7.6
- removed Q2: STS4DNF60L, Housings_SOIC:SOIC-8_3.9x4.9mm_Pitch1.27mm
- removed the R6 at (170.2, 15.5)
- removed the R7 at (170.2, 18.3)
- moved C6 236.3 mm to (50.8, 125.7), turned to 180 degrees
- moved C1 235.5 mm to (57.8, 98.4), turned to 180 degrees
- moved C2 225.1 mm to (52.1, 108.6), turned to 270 degrees
- moved R17 216.5 mm to (79.4, 102.9), turned to 90 degrees
- moved C3 214.3 mm to (57.8, 118.7)
- moved C5 209.8 mm to (73.0, 111.8), turned to 90 degrees
- moved R21 196.2 mm to (97.2, 102.9), turned to 90 degrees
- moved C7 187.3 mm to (73.7, 105.4), turned to 90 degrees
- moved R20 187.1 mm to (97.2, 106.0), turned to 90 degrees
- moved C4 186.5 mm to (66.0, 118.7)
- moved R19 185.6 mm to (94.6, 102.9), turned to 90 degrees
- moved R18 181.0 mm to (94.6, 105.9), turned to 90 degrees
- moved RN1 170.1 mm to (77.1, 116.6), turned to 270 degrees
- moved C11 167.2 mm to (89.8, 122.8), turned to 0 degrees
- moved C13 166.1 mm to (92.8, 122.8), turned to 0 degrees
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- renumbered R12 to R10, R13 to R11, R14 to R12, R15 to R13, R16 to R14, R17 to R15, R18 to R16, R19 to R17, R20 to R18, R21 to R19, R22 to R20, R23 to R21, R24 to R22, R8 to R6, R9 to R7, R10 to R8, R11 to R9
Connections:
- J2 pad 1: +12V -> +3V3
- J2 pad 10: GND -> /GNC_TX
- J2 pad 11: /GPS_RX -> /XBEE_RX
- J2 pad 12: /GPS_TX -> /XBEE_TX
- J2 pad 13: /GNC_RX -> GND
- J2 pad 14: /GNC_TX -> /SERVO2_CTRL
- J2 pad 15: /XBEE_RX -> GND
- J2 pad 16: /XBEE_TX -> (no net)
- J2 pad 17: GND -> /BAT_VCC
- J2 pad 18: GND -> +12V
- J2 pad 19: /TC1_T- -> GND
- J2 pad 20: /TC1_T+ -> /TC1_T-
- J2 pad 21: /TC2_T- -> /TC1_T+
- J2 pad 22: /TC2_T+ -> /TC2_T-
- J2 pad 23: /TC3_T- -> /TC2_T+
- J2 pad 24: /TC3_T+ -> /TC3_T-
- J2 pad 25: GND -> /TC3_T+
- J2 pad 26: GND -> /TC5_T+
- J2 pad 27: /TC5_T+ -> /TC5_T-
- J2 pad 28: /TC5_T- -> /TC4_T+
- J2 pad 29: /TC4_T+ -> /TC4_T-
- J2 pad 3: (no net) -> /BOARD_TX+
- J2 pad 30: /TC4_T- -> /PT2_IN
- J2 pad 31: /PT2_IN -> /PT1_IN
- J2 pad 32: /PT1_IN -> GND
- J2 pad 33: GND -> /BAT_BAK_VCC
- J2 pad 34: GND -> /UMB_VCC
- J2 pad 35: /SERVO1_CL_SW -> /VCC_IN
- J2 pad 36: /SERVO1_OP_SW -> GND
- J2 pad 37: /SERVO2_CL_SW -> /SERVO1_CTRL
- J2 pad 38: /SERVO2_OP_SW -> GND
- J2 pad 39: /GNC_INST -> /SERVO1_CL_SW
- J2 pad 4: /BAT_VCC -> GND
- J2 pad 40: GND -> /SERVO1_OP_SW
- J2 pad 41: GND -> /SERVO2_CL_SW
- J2 pad 42: /BOARD_RX- -> /SERVO2_OP_SW
- J2 pad 43: GND -> /GNC_INST
- J2 pad 44: /BOARD_TX- -> GND
- J2 pad 46: /BAT_BAK_VCC -> /BOARD_RX-
- J2 pad 47: /VCC_IN -> GND
- J2 pad 48: GND -> /BOARD_TX-
- J2 pad 49: +3V3 -> GND
- J2 pad 5: /UMB_VCC -> /BOARD_RX+
- J2 pad 7: /BOARD_TX+ -> /GPS_RX
- J2 pad 8: GND -> /GPS_TX
- J2 pad 9: /BOARD_RX+ -> /GNC_RX
- U1 pad 40: /BUZZER1 -> (no net)
- U1 pad 41: /BUZZER2 -> (no net)
Other:
- board size 91.4 x 53.3 mm -> 80 x 45.7 mm

Commit message: A whole lot of changes
Kinda forgot what they all were
Parts:
- removed J2: Conn_02x25_Counter_Clockwise, Custom Footprints:CONN_CARD_02x25_MALE
- removed SW1: SW_SPDT, Buttons_Switches_SMD:SW_SPDT_CK-JS102011SAQN
- added J1: Conn_02x10_Odd_Even, Pin_Headers:Pin_Header_Straight_2x10_Pitch1.27mm, B.Cu at (179.7, 135.3)
- added SYM1: SYM_Arrow45_XLarge, Custom Parts:Logo_v3, B.Cu at (212.7, 132.7)
- moved C6 195.0 mm to (245.7, 127.6)
- moved R22 164.7 mm to (222.9, 105.2), turned to 270 degrees
- moved U4 160.5 mm to (218.2, 106.4), turned to 0 degrees
- moved C3 155.4 mm to (212.7, 107.3), turned to 90 degrees
- moved C10 155.2 mm to (216.4, 102.6), turned to 0 degrees
- moved RN1 151.0 mm to (224.5, 149.0), turned to 0 degrees
- moved U2 147.4 mm to (219.7, 149.0), turned to 0 degrees
- moved C8 144.4 mm to (220.2, 146.2), turned to 0 degrees
- moved Q1 143.5 mm to (218.6, 125.2)
- moved R1 143.5 mm to (223.9, 126.8)
- moved R2 143.5 mm to (223.9, 123.7)
- moved R3 143.5 mm to (225.9, 126.8)
- moved R4 143.5 mm to (225.9, 123.7)
- moved RN2 143.1 mm to (224.8, 142.1), turned to 0 degrees
- moved U3 139.3 mm to (220.0, 142.1), turned to 0 degrees
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Routing:
- removed copper zone on B.Cu, net GND
- removed copper zone on F.Cu, net GND
Other:
- board size 80 x 45.7 mm -> 55.9 x 58.4 mm
- board text added: "Control Board v0.1 UAH SHC Spaceport America Cup 2018 Designed by Thomas Bennett Daniel Corey, Kyle Daigle, Jacob Klingbeil, Brendan Luke"
