File: Control Board/Control Board.kicad_pcb (KiCad board)
At the start: 2 copper layers, 55.9 x 58.4 mm, 77 parts, among them J1 Conn_02x03_Odd_Even, J1 Conn_02x10_Odd_Even, Q1 STS4DNF60L, U1 ATXMEGA128A3-AU, U2 LT1797, U3 LT1797, U4 ISL83490, U5 MAX31856, U6 MAX31856, U7 MAX31856, U8 MAX31856, U9 MAX31856

Commit message: More changes
Parts:
- added H1: Mounting_Hole, Mounting_Holes:MountingHole_3.2mm_M3, F.Cu at (180.8, 104.6)
- added H2: Mounting_Hole, Mounting_Holes:MountingHole_3.2mm_M3, F.Cu at (228.1, 104.6)
- added H3: Mounting_Hole, Mounting_Holes:MountingHole_3.2mm_M3, F.Cu at (228.1, 154.4)
- added H4: Mounting_Hole, Mounting_Holes:MountingHole_3.2mm_M3, F.Cu at (180.8, 154.4)
- added J10: Conn_01x03, Connectors_JST:JST_PH_B3B-PH-K_03x2.00mm_Straight, F.Cu at (245.1, 146.8)
- added J11: Conn_01x03, Connectors_JST:JST_PH_B3B-PH-K_03x2.00mm_Straight, F.Cu at (245.1, 137.9)
- added J13: Conn_01x03, Connectors_JST:JST_PH_B3B-PH-K_03x2.00mm_Straight, F.Cu at (237.7, 137.9)
- added J14: Conn_01x03, Connectors_JST:JST_PH_B3B-PH-K_03x2.00mm_Straight, F.Cu at (245.1, 129.0)
- added J15: Conn_01x03, Connectors_JST:JST_PH_B3B-PH-K_03x2.00mm_Straight, F.Cu at (237.7, 129.0)
- added J3: RJ45, Connectors:RJ45_8, F.Cu at (241.6, 113.3)
- added J4: Conn_01x02, Connectors_JST:JST_PH_B2B-PH-K_02x2.00mm_Straight, F.Cu at (252.5, 155.7)
- added J5: Conn_01x02, Connectors_JST:JST_PH_B2B-PH-K_02x2.00mm_Straight, F.Cu at (252.5, 148.7)
- added J6: Conn_01x03, Connectors_JST:JST_PH_B3B-PH-K_03x2.00mm_Straight, F.Cu at (245.1, 155.7)
- added J7: Conn_01x02, Connectors_JST:JST_PH_B2B-PH-K_02x2.00mm_Straight, F.Cu at (252.5, 141.7)
- added J8: Conn_01x02, Connectors_JST:JST_PH_B2B-PH-K_02x2.00mm_Straight, F.Cu at (252.5, 134.7)
- added J9: Conn_01x02, Connectors_JST:JST_PH_B2B-PH-K_02x2.00mm_Straight, F.Cu at (252.5, 127.8)
- added R23: 10 kΩ, Resistors_SMD:R_0603, F.Cu at (227.8, 128.3)
- added R24: 10 kΩ, Resistors_SMD:R_0603, F.Cu at (230.4, 128.3)
- added R25: 10 kΩ, Resistors_SMD:R_0603, F.Cu at (225.3, 128.3)
- added U10: OPENLOG, Custom Footprints:OpenLog, F.Cu at (222.5, 123.8)
- J1: moved to F.Cu
- R1, R2: value 1.8 kΩ -> 10 kΩ
- SYM1: value SYM_Arrow45_XLarge -> SYM_Arrow45_Large
- moved C6 57.1 mm to (188.7, 125.7)
- moved R1 40.0 mm to (185.4, 137.7)
- moved R14 37.4 mm to (180.8, 148.5), turned to 180 degrees
- moved D1 35.3 mm to (203.8, 103.4)
- moved R12 33.6 mm to (180.8, 146.6), turned to 0 degrees
- moved R15 29.8 mm to (180.8, 144.7), turned to 180 degrees
- moved R6 28.8 mm to (203.8, 106.7), turned to 270 degrees
- moved R13 26.0 mm to (180.8, 142.7), turned to 0 degrees
- moved R17 22.2 mm to (180.8, 140.8), turned to 180 degrees
- moved R16 18.4 mm to (180.8, 138.9), turned to 0 degrees
- moved C10 14.5 mm to (228.9, 110.0)
- moved C3 14.5 mm to (225.2, 114.7)
- moved R22 14.5 mm to (235.3, 112.5)
- moved U4 14.5 mm to (230.6, 113.8)
- moved J1 10.2 mm to (179.7, 125.1)
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- renumbered J1 to J2
Connections:
- J1 pad 1: (no net) -> +3V3
- J1 pad 10: (no net) -> /BAT_BAK_VCC
- J1 pad 11: (no net) -> /GNC_RX
- J1 pad 12: (no net) -> GND
- J1 pad 13: (no net) -> /XBEE_TX
- J1 pad 14: (no net) -> +3V3
- J1 pad 15: (no net) -> /XBEE_RX
- J1 pad 16: (no net) -> GND
- J1 pad 17: (no net) -> /GPS_TX
- J1 pad 18: (no net) -> +12V
- J1 pad 19: (no net) -> /GPS_RX
- J1 pad 2: (no net) -> GND
- J1 pad 20: (no net) -> GND
- J1 pad 3: (no net) -> GND
- J1 pad 4: (no net) -> /VCC_IN
- J1 pad 5: (no net) -> /GNC_INST
- J1 pad 6: (no net) -> /UMB_VCC
- J1 pad 7: (no net) -> GND
- J1 pad 8: (no net) -> /BAT_VCC
- J1 pad 9: (no net) -> /GNC_TX
- J2 pad 3: (no net) -> Net-(J2-Pad3)
- J2 pad 4: (no net) -> Net-(J2-Pad4)
- R1 pad 1: +14V -> GND
- R1 pad 2: /SERVO2_CTRL -> /GNC_INST
- R2 pad 1: +14V -> GND
- R2 pad 2: /SERVO1_CTRL -> /SERVO2_OP_SW
- R3 pad 1: GND -> /VCC_IN
- R4 pad 1: GND -> /SERVO1_CTRL
- R4 pad 2: /SERVO1_CTRL -> /VCC_IN
- U1 pad 1: /TC1_FAULT -> /V_BAT1_ADC
- U1 pad 10: /V_BAT2_ADC -> /TC3_CS
- U1 pad 11: /V_SUPPLY_ADC -> /TC3_DRDY
- U1 pad 12: /V_3.3_ADC -> /TC4_CS
- U1 pad 13: /V_PT_ADC -> /TC4_DRDY
- U1 pad 16: /TC4_CS -> /TC5_CS
- U1 pad 17: /TC4_FAULT -> /TC5_DRDY
- U1 pad 18: /TC4_DRDY -> /OPENLOG_TX
- U1 pad 19: /TC3_CS -> /OPENLOG_RX
- U1 pad 2: /TC1_DRDY -> /V_BAT2_ADC
- U1 pad 20: /TC3_DRDY -> Net-(U1-Pad20)
- U1 pad 3: /TC2_CS -> /V_SUPPLY_ADC
- U1 pad 4: /TC2_FAULT -> /V_3.3_ADC
- U1 pad 40: (no net) -> Net-(U1-Pad40)
- U1 pad 41: (no net) -> Net-(U1-Pad41)
- U1 pad 5: /TC2_DRDY -> /V_PT_ADC
- U1 pad 51: /TC5_CS -> Net-(U1-Pad51)
- U1 pad 54: /TC5_FAULT -> Net-(U1-Pad54)
- U1 pad 55: /TC5_DRDY -> Net-(U1-Pad55)
- U1 pad 58: (no net) -> Net-(U1-Pad58)
- U1 pad 59: (no net) -> Net-(U1-Pad59)
- U1 pad 6: /TC3_FAULT -> /TC1_CS
- U1 pad 64: /TC1_CS -> /V_UMB_ADC
- U1 pad 7: (no net) -> /TC1_DRDY
- U1 pad 8: /V_UMB_ADC -> /TC2_CS
- U1 pad 9: /V_BAT1_ADC -> /TC2_DRDY
- U5 pad 13: /TC1_FAULT -> Net-(U5-Pad13)
- U6 pad 13: /TC2_FAULT -> Net-(U6-Pad13)
- U7 pad 13: /TC3_FAULT -> Net-(U7-Pad13)
- U8 pad 13: /TC4_FAULT -> Net-(U8-Pad13)
- U9 pad 13: /TC5_FAULT -> Net-(U9-Pad13)
Routing:
- net /BOARD_RX-: track 0.00 -> 17.4 mm
- net /BOARD_RX+: track 0.00 -> 9.34 mm
- net /BOARD_TX+: track 0.00 -> 9.22 mm
- net /BOARD_TX-: track 0.00 -> 7.70 mm
- added copper zone on B.Cu, net GND
- added copper zone on F.Cu, net GND
Other:
- board size 55.9 x 58.4 mm -> 80 x 58.4 mm

Commit message: Routed a ton of stuff on the control board
Parts:
- moved R1 26.6 mm to (188.0, 111.2), turned to 0 degrees
- moved L1 25.3 mm to (188.1, 124.0), turned to 0 degrees
- moved C1 22.1 mm to (204.8, 129.6), turned to 0 degrees
- moved C7 21.4 mm to (190.4, 123.2), turned to 270 degrees
- moved C3 20.8 mm to (204.8, 110.4), turned to 180 degrees
- moved C5 20.8 mm to (190.4, 116.8), turned to 270 degrees
- moved C4 20.8 mm to (196.8, 110.4), turned to 180 degrees
- moved C2 20.4 mm to (209.6, 120.0), turned to 90 degrees
- moved J6 10.2 mm to (237.7, 148.6)
- moved C6 10.1 mm to (179.7, 121.2), turned to 90 degrees
- moved RN1 5.69 mm to (225.7, 144.5), turned to 180 degrees
- moved RN2 5.53 mm to (225.7, 139.1), turned to 180 degrees
- moved C9 5.49 mm to (229.9, 141.7), turned to 180 degrees
- moved U2 4.89 mm to (230.4, 144.5), turned to 180 degrees
- moved C8 4.57 mm to (229.9, 147.2), turned to 180 degrees
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Routing:
- net +3V3: track 0.00 -> 311.9 mm, vias 0 -> 24
- net /TC1_T-: track 1.25 -> 85.5 mm
- net +12V: track 0.00 -> 83.1 mm, vias 0 -> 2
- net /MOSI1: track 0.00 -> 81.0 mm, vias 0 -> 8
- net /MISO1: track 0.00 -> 79.0 mm, vias 0 -> 8
- net /SCK1: track 0.00 -> 77.2 mm
- net /TC2_T-: track 0.00 -> 76.6 mm
- net /TC3_T-: track 0.00 -> 74.1 mm
- net /TC1_T+: track 0.00 -> 73.4 mm
- net /TC4_T-: track 0.00 -> 72.2 mm
- net /TC5_T-: track 0.00 -> 70.3 mm
- net /PT2_ADC: track 0.00 -> 70.1 mm
- net /PT1_ADC: track 0.00 -> 68.4 mm
- net /TC2_T+: track 0.00 -> 67.9 mm
- net /TC3_T+: track 0.00 -> 66.0 mm
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Other:
- net class Small: clearance 0.13 -> 0.16; trace_width 0.13 -> 0.16; via_drill 0.25 -> 0.254
- rule trace_min: 0.13 -> 0.1524
- rule via_min_drill: 0.25 -> 0.254
- rule via_min_size: 0.51 -> 0.508
