File: Power Board/Power Board.sch (KiCad schematic (older format))
At the start: 55 parts, among them J1 Conn_02x10_Odd_Even, J2 Conn_01x02, J3 Conn_01x02, J4 Conn_01x02, J5 Conn_01x02, Q1 SI7135DP, Q2 SI7135DP, Q3 SI7135DP, Q4 SI7135DP, Q5 SI7135DP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

Commit message: Started implementing battery charger/balancer, upgraded to KiCad 5 stable
Parts:
- added C?: 0.1 uF, Capacitors_SMD:C_0603, symbol Device:C_Small
- added D?: LED_G, LEDs:LED_0603, symbol Device:LED
- added D? (x4): LED_B, LEDs:LED_0603, symbol Device:LED
- added J?: Conn_01x03, Connectors_JST:JST_XH_S03B-XH-A_03x2.50mm_Angled, symbol Connector_Generic:Conn_01x03
- added Q?: AON7423, symbol Device:Q_PMOS_SGD
- added R?: 0.124Ω, Resistors_SMD:R_2512, symbol Device:R
- added R?: 470 Ω, Resistors_SMD:R_0603, symbol Device:R
- added R? (x4): 1 kΩ, Resistors_SMD:R_0603, symbol Device:R
- added U?: BQ2057WSNTR, symbol Custom-Parts:BQ2057WSNTR
- added U?: BQ29209DRBT, symbol Custom-Parts:BQ29209DRBT
- C1: symbol device:CP1_Small -> Device:CP1_Small
- C10, C11, C12, C13, C14, C15, C16, C17, C18, C2, C3, C4, C5, C6, C7, C8, C9: symbol device:C_Small -> Device:C_Small
- D2: symbol device:D_Zener -> Device:D_Zener
- D5, D6: symbol device:LED -> Device:LED
- H1, H2, H3, H4: symbol Mechanical:Mounting_Hole -> Power-Board-rescue:Mounting_Hole-Mechanical
- J1: symbol Connector:Conn_02x10_Odd_Even -> Power-Board-rescue:Conn_02x10_Odd_Even-Connector
- J2, J3, J4, J5: symbol Connector:Conn_01x02 -> Power-Board-rescue:Conn_01x02-Connector
- L1, L2: symbol device:L_Small -> Device:L_Small
- Q1, Q2, Q3, Q4, Q5, Q6: symbol device:Q_PMOS_DGS -> Device:Q_PMOS_DGS
- R1, R10, R11, R2, R3, R4, R5, R6, R7, R8, R9: symbol device:R_Small -> Device:R_Small
- R12, R13: symbol device:R -> Device:R
Connections:
- net labels added: BAT_CELL_1, BAT_CELL_2, BAT_CELL_GND, CHARGE_STAT
- wire segments 148 -> 185
Other:
- note added: "Charge current 1A"

Commit message: Finished battery charger schematic
still need to fill out BOM, and start cell balancer
Parts:
- removed R?: 470 Ω, Resistors_SMD:R_0603, symbol Device:R
- added J?: Conn_01x02, Connectors_JST:JST_PH_S2B-PH-K_02x2.00mm_Angled, symbol Connector_Generic:Conn_01x02
- added R?: 1 kΩ, Resistors_SMD:R_0603, symbol Device:R
- added R?: 8.25 kΩ, symbol Device:R
- added R?: 22.1 kΩ, symbol Device:R
- added TH?: NXFT15XH103FA2B100, ~, symbol Device:Thermistor_NTC
Connections:
- wire segments 185 -> 198
Other:
- note added: "Not mounted, free hanging"
Changed lines of the file:
@@
 L power:GND #PWR?
 U 1 1 5B825B1A
-P 9700 6350
-F 0 "#PWR?" H 9700 6100 50  0001 C CNN
-F 1 "GND" V 9700 6150 50  0000 C CNN
-F 2 "" H 9700 6350 50  0001 C CNN
-F 3 "" H 9700 6350 50  0001 C CNN
-	1    9700 6350
+P 9700 6400
+F 0 "#PWR?" H 9700 6150 50  0001 C CNN
+F 1 "GND" V 9700 6200 50  0000 C CNN
+F 2 "" H 9700 6400 50  0001 C CNN
+F 3 "" H 9700 6400 50  0001 C CNN
+	1    9700 6400
 	-1   0    0    -1
 $EndComp
@@
 Wire Wire Line
 	11100 5800 11350 5800
-Text Label 12100 5800 0    50   ~ 0
-CHARGE_STAT
 $Comp
 L Device:LED D?
 U 1 1 5B8CB8F0
-P 11350 6150
-F 0 "D?" H 11350 6250 50  0000 C CNN
-F 1 "LED_G" H 11350 6050 50  0000 C CNN
-F 2 "LEDs:LED_0603" H 11350 6150 50  0001 C CNN
-F 3 "" H 11350 6150 50  0001 C CNN
-F 4 "160-1888-1-ND" H 11350 6350 50  0001 C CNN "Digikey Part Number"
-	1    11350 6150
-	0    -1   -1   0
-$EndComp
-$Comp
-L Device:R R?
-U 1 1 5B8CB8F7
-P 11350 6650
-F 0 "R?" V 11430 6650 50  0000 C CNN
-F 1 "470 Ω" V 11350 6650 50  0000 C CNN
-F 2 "Resistors_SMD:R_0603" V 11280 6650 50  0001 C CNN
-F 3 "" H 11350 6650 50  0001 C CNN
-F 4 "311-100GRCT-ND" H 11430 6750 50  0001 C CNN "Digikey Part Number"
-	1    11350 6650
-	1    0    0    -1
+P 11500 6000
+F 0 "D?" H 11500 6100 50  0000 C CNN
+F 1 "LED_G" H 11500 5900 50  0000 C CNN
+F 2 "LEDs:LED_0603" H 11500 6000 50  0001 C CNN
+F 3 "" H 11500 6000 50  0001 C CNN
+F 4 "160-1888-1-ND" H 11500 6200 50  0001 C CNN "Digikey Part Number"
+	1    11500 6000
+	-1   0    0    1
 $EndComp
 $Comp
 L power:GND #PWR?
 U 1 1 5B8CB8FD
-P 11350 6950
-F 0 "#PWR?" H 11350 6700 50  0001 C CNN
-F 1 "GND" H 11350 6800 50  0000 C CNN
-F 2 "" H 11350 6950 50  0001 C CNN
-F 3 "" H 11350 6950 50  0001 C CNN
-	1    11350 6950
-	0    -1   -1   0
-$EndComp
-Wire Wire Line
-	11350 6300 11350 6500
-Wire Wire Line
-	11350 6950 11350 6800
+P 11950 6000
+F 0 "#PWR?" H 11950 5750 50  0001 C CNN
+F 1 "GND" H 11950 5850 50  0000 C CNN
+F 2 "" H 11950 6000 50  0001 C CNN
+F 3 "" H 11950 6000 50  0001 C CNN
+	1    11950 6000
+	1    0    0    -1
+$EndComp
 Wire Wire Line
 	11350 6000 11350 5800
-Connection ~ 11350 5800
-Wire Wire Line
-	11350 5800 12100 5800
 $Comp
 L Device:C_Small C?
@@
 	1    0    0    -1
 $EndComp
-Text Label 10400 6350 0    50   ~ 0
+Text Label 12100 6400 0    50   ~ 0
 BAT_CELL_GND
 Wire Wire Line
 	11100 5700 11200 5700
 Wire Wire Line
-	11200 5700 11200 6350
+	11200 5700 11200 6400
 Wire Wire Line
 	9250 4500 9350 4500
@@
 Wire Wire Line
 	9350 4500 9550 4500
-Wire Wire Line
-	9700 6350 11200 6350
-Connection ~ 9700 6350
 Connection ~ 9700 5700
 Wire Wire Line
 	9350 5700 9700 5700
-Wire Wire Line
-	9700 6150 9700 6350
 Wire Wire Line
 	9700 5700 9700 5950
@@
 	8400 1100 8900 1100
 Connection ~ 8900 1100
+$Comp
+L Device:R R?
+U 1 1 5B9CB7B5
+P 11800 6000
+F 0 "R?" V 11880 6000 50  0000 C CNN
+F 1 "1 kΩ" V 11800 6000 50  0000 C CNN
+F 2 "Resistors_SMD:R_0603" V 11730 6000 50  0001 C CNN
+F 3 "" H 11800 6000 50  0001 C CNN
+F 4 "RHM1.0KDCT-ND" H 11880 6100 50  0001 C CNN "Digikey Part Number"
+	1    11800 6000
+	0    -1   -1   0
+$EndComp
+$Comp
+L Connector_Generic:Conn_01x02 J?
+U 1 1 5B9CEC20
+P 8300 5800
+F 0 "J?" H 8220 6017 50  0000 C CNN
+F 1 "Conn_01x02" H 8220 5926 50  0000 C CNN
+F 2 "Connectors_JST:JST_PH_S2B-PH-K_02x2.00mm_Angled" H 8300 5800 50  0001 C CNN
+F 3 "~" H 8300 5800 50  0001 C CNN
+	1    8300 5800
+	-1   0    0    -1
+$EndComp
+$Comp
+L Device:Thermistor_NTC TH?
+U 1 1 5B9CEDC6
+P 7850 5850
+F 0 "TH?" H 7550 5900 50  0000 L CNN
+F 1 "NXFT15XH103FA2B100" H 6850 5800 50  0000 L CNN
+F 2 "~" H 7850 5900 50  0001 C CNN
+F 3 "~" H 7850 5900 50  0001 C CNN
+F 4 "490-5630-ND" H 7850 5850 50  0001 C CNN "Digikey Part Number"
+	1    7850 5850
+	1    0    0    -1
+$EndComp
+Text Notes 6850 6150 0    50   ~ 0
+Not mounted, free hanging
+Wire Wire Line
+	7850 5700 8050 5700
+Wire Wire Line
+	8050 5700 8050 5800
+Wire Wire Line
+	8050 5800 8150 5800
+Wire Wire Line
+	7850 6000 8050 6000
+Wire Wire Line
+	8050 6000 8050 5900
+Wire Wire Line
+	8050 5900 8150 5900
+$Comp
+L power:GND #PWR?
+U 1 1 5BA07E84
+P 8500 5900
+F 0 "#PWR?" H 8500 5650 50  0001 C CNN
+F 1 "GND" V 8500 5700 50  0000 C CNN
+F 2 "" H 8500 5900 50  0001 C CNN
+F 3 "" H 8500 5900 50  0001 C CNN
+	1    8500 5900
+	-1   0    0    -1
+$EndComp
+$Comp
+L Device:R R?
+U 1 1 5BA12446
+P 8800 5550
+F 0 "R?" H 8870 5596 50  0000 L CNN
+F 1 "8.25 kΩ" H 8870 5505 50  0000 L CNN
+F 2 "" V 8730 5550 50  0001 C CNN
+F 3 "~" H 8800 5550 50  0001 C CNN
+	1    8800 5550
+	1    0    0    -1
+$EndComp
+$Comp
+L Device:R R?
+U 1 1 5BA12507
+P 8800 6050
+F 0 "R?" H 8870 6096 50  0000 L CNN
+F 1 "22.1 kΩ" H 8870 6005 50  0000 L CNN
+F 2 "" V 8730 6050 50  0001 C CNN
+F 3 "~" H 8800 6050 50  0001 C CNN
+	1    8800 6050
+	1    0    0    -1
+$EndComp
+Wire Wire Line
+	8500 5800 8800 5800
+Wire Wire Line
+	8800 5700 8800 5800
+Wire Wire Line
+	8800 5400 8800 5100
+Wire Wire Line
+	8800 5100 9350 5100
+Wire Wire Line
+	9700 6400 8800 6400
+Wire Wire Line
+	8800 6400 8800 6200
+Connection ~ 8800 5800
+Wire Wire Line
+	8800 5800 8800 5900
+Wire Wire Line
+	8800 5800 10200 5800
+Connection ~ 9700 6400
+Wire Wire Line
+	9700 6150 9700 6400
+Wire Wire Line
+	11350 5800 11700 5800
+Connection ~ 11350 5800
+Wire Wire Line
+	12100 6400 11200 6400
+Connection ~ 11200 6400
+Wire Wire Line
+	9700 6400 11200 6400
+Text Label 11700 5800 0    50   ~ 0
+CHARGE_STAT
 $EndSCHEMATC

Commit message: Finished Balancer and charger schematic
Still need to change umbilical voltage input range
Parts:
- removed C10, C9: 15 uF, Capacitors_SMD:C_0805, symbol Device:C_Small
- removed C12: 22 uF, Capacitors_SMD:C_0805, symbol Device:C_Small
- added C20, C21, C22: 0.1 µF, symbol Device:C_Small
- added C23: 0.33 µF, symbol Device:C_Small
- added C?: 22 uF, Capacitors_SMD:C_0805, symbol Device:C_Small
- added R22: 100 Ω, symbol Device:R_Small
- added R?: 140 kΩ, symbol Device:R_Small
- added R? (x2): 10 kΩ, symbol Device:R_Small
- added R? (x3): 100 kΩ, symbol Device:R_Small
- added R?: 10 Ω, symbol Device:R_Small
- added U?: LT6700CS6-1, symbol Custom-Parts:LT6700CS6-1
- added U?: STS8C5H30L, symbol Custom-Parts:STS8C5H30L
- C11: value 22 uF -> 47 uF; Digikey Part Number 1276-6526-1-ND -> 490-13249-1-ND
- L1: value 18 uH -> 2.2 uH; footprint Inductors_SMD:L_Wuerth_HCI-1365 -> (none); Digikey Part Number 732-3880-1-ND -> SRP6540-2R2MCT-ND
- R10: value 100 kΩ -> 33.2 kΩ; Digikey Part Number 311-100KHRCT-ND -> 311-33.2KHRCT-ND
- R11: value 22 kΩ -> 10 kΩ; Digikey Part Number 311-22.0KHRCT-ND -> 311-10.0KHRCT-ND
- U2: value TPS54308DDC -> TPS564208DDCT; Digikey Part Number 296-47880-1-ND -> 296-44123-1-ND
- gave numbers to parts that had none: 20
Connections:
- wire segments 198 -> 260
Other:
- note added: "6V Undervoltage Cutoff"
- note added: "Balance MOSFETs"
- note added: "Cell Balance Controller"

Commit message: Did some digikey part number replacing
Parts:
- C1: value 470 uF -> 470 µF
- C11: value 47 uF -> 47 µF
- C13, C14: Digikey Part Number 399-9043-1-ND -> 399-9044-1-ND
- C15: value 15 uF -> 15 µF; Digikey Part Number 445-14423-1-ND -> 445-14373-1-ND
- C16: value 22 uF -> 22 µF; Digikey Part Number 1276-6526-1-ND -> 1276-6780-1-ND
- C17: value 1 uF -> 1 µF
- C18: value 4.7 uF -> 4.7 µF
- C19, C2, C3, C4, C5, C6, C7: value 0.1 uF -> 0.1 µF; Digikey Part Number 445-5667-1-ND -> 1276-6717-6-ND
- C20, C21, C22: footprint (none) -> Capacitors_SMD:C_0603; Digikey Part Number (none) -> 1276-6717-6-ND
- C23: footprint (none) -> Capacitors_SMD:C_0603; Digikey Part Number (none) -> 445-12479-6-ND
- C8: value 0.1 uF -> 0.1 µF; Digikey Part Number 399-1171-1-ND -> 478-3351-1-ND
- C9: renamed from C?; value 22 uF -> 22 µF
- L1: value 2.2 uH -> 2.2 µH
- L2: value 15 uH -> 15 µH
- Q1, Q2, Q3, Q4, Q5, Q6: Digikey Part Number SI7135DP-T1-GE3CT-ND -> SI7145DP-T1-GE3CT-ND
- R1, R4, R7: Digikey Part Number 311-82.5KHRCT-ND -> P82.5KHCT-ND
- R10: Digikey Part Number 311-33.2KHRCT-ND -> P33.2KHCT-ND
- R11: Digikey Part Number 311-10.0KHRCT-ND -> P10.0KHCT-ND
- R12: Digikey Part Number 311-100GRCT-ND -> P100HCT-ND
- R13: Digikey Part Number 311-100GRCT-ND -> P470HCT-ND
- R19: footprint (none) -> Resistors_SMD:R_0603; Digikey Part Number (none) -> P8.25KDBCT-ND
- R21: footprint (none) -> Resistors_SMD:R_0603; Digikey Part Number (none) -> P22.1KDBCT-ND
- R22: footprint (none) -> Resistors_SMD:R_0603; Digikey Part Number (none) -> P100HCT-ND
- R23, R24, R25: renamed from R?; footprint (none) -> Resistors_SMD:R_0603; Digikey Part Number (none) -> P100KDBCT-ND
- R26: renamed from R?; footprint (none) -> Resistors_SMD:R_0603; Digikey Part Number (none) -> P140KDBCT-ND
- R27: renamed from R?; footprint (none) -> Resistors_SMD:R_0603; Digikey Part Number (none) -> 541-10.0SCT-ND
- R28, R29: renamed from R?; footprint (none) -> Resistors_SMD:R_0603; Digikey Part Number (none) -> P10.0KHCT-ND
- R3, R6, R9: Digikey Part Number 311-11.0KHRCT-ND -> P11.0KHCT-ND
- U6: renamed from U?; Digikey Part Number (none) -> LT6700CS6-1#TRMPBFCT-ND
- gave numbers to parts that had none: 1
Other:
- note added: "MOSFETs will need heatsinks"

Commit message: Added Heatsink, changed umbilical voltage
10.5 volts is technically above the max reccomended supply for the lipo balancer, but it's set to that to make sure the supply doesn't come in and out if it's at 10 volts
Parts:
- added HS1: Heatsink, symbol Mechanical:Heatsink
- R1: value 82.5 kΩ -> 88.7 kΩ; Digikey Part Number P82.5KHCT-ND -> P88.7KHCT-ND
- R2: value 5.49 kΩ -> 1.58 kΩ; Digikey Part Number 311-5.49KHRCT-ND -> P1.58KHCT-ND
- R3: value 11 kΩ -> 9.53 kΩ; Digikey Part Number P11.0KHCT-ND -> P9.53KHCT-ND
Other:
- note added: "9-10.5 V"
Changed lines of the file:
@@
 VCC_IN
 Text Notes 1700 1050 0    60   ~ 0
-6-9 V (actually 8.4 but a little margin of error)
+9-10.5 V
 Text Notes 1700 1450 0    60   ~ 0
 6-9 V (actually 8.4 but a little margin of error)
@@
 P 3650 3100
 F 0 "R1" V 3650 2500 50  0000 L CNN
-F 1 "82.5 kΩ" V 3650 2650 50  0000 L CNN
+F 1 "88.7 kΩ" V 3650 2650 50  0000 L CNN
 F 2 "Resistors_SMD:R_0603" H 3650 3100 50  0001 C CNN
 F 3 "" H 3650 3100 50  0001 C CNN
-F 4 "P82.5KHCT-ND" H 3650 2600 50  0001 C CNN "Digikey Part Number"
+F 4 "P88.7KHCT-ND" H 3650 2600 50  0001 C CNN "Digikey Part Number"
 	1    3650 3100
 	0    1    -1   0
@@
 P 3650 3200
 F 0 "R2" V 3650 2600 50  0000 L CNN
-F 1 "5.49 kΩ" V 3650 2750 50  0000 L CNN
+F 1 "1.58 kΩ" V 3650 2750 50  0000 L CNN
 F 2 "Resistors_SMD:R_0603" H 3650 3200 50  0001 C CNN
 F 3 "" H 3650 3200 50  0001 C CNN
-F 4 "311-5.49KHRCT-ND" H 3650 2700 50  0001 C CNN "Digikey Part Number"
+F 4 "P1.58KHCT-ND" H 3650 2700 50  0001 C CNN "Digikey Part Number"
 	1    3650 3200
 	0    1    -1   0
@@
 P 3650 3300
 F 0 "R3" V 3650 2700 50  0000 L CNN
-F 1 "11 kΩ" V 3650 2900 50  0000 L CNN
+F 1 "9.53 kΩ" V 3650 2900 50  0000 L CNN
 F 2 "Resistors_SMD:R_0603" H 3650 3300 50  0001 C CNN
 F 3 "" H 3650 3300 50  0001 C CNN
-F 4 "P11.0KHCT-ND" H 3650 2800 50  0001 C CNN "Digikey Part Number"
+F 4 "P9.53KHCT-ND" H 3650 2800 50  0001 C CNN "Digikey Part Number"
 	1    3650 3300
 	0    1    -1   0
@@
 Text Notes 5900 1000 0    50   ~ 0
 MOSFETs will need heatsinks
+$Comp
+L Mechanical:Heatsink HS1
+U 1 1 5BBF14DE
+P 7250 950
+F 0 "HS1" H 7392 1071 50  0000 L CNN
+F 1 "Heatsink" H 7392 980 50  0000 L CNN
+F 2 "" H 7262 950 50  0001 C CNN
+F 3 "" H 7262 950 50  0001 C CNN
+F 4 "ATS1099-ND" H 7250 950 50  0001 C CNN "Digikey Part Number"
+	1    7250 950
+	1    0    0    -1
+$EndComp
 $EndSCHEMATC

Commit message: Few changes
Parts:
- added U?: LTC4150, MSOP10, symbol SparkFun-IC-Power:LTC4150
Connections:
- net labels added: THERM1, THERM2, THERM3, THERM4
- wire segments 260 -> 272
Other:
- note added: "Figure out replacement for DS1682S or a way to get it to count down"
- note added: "TODO: MAX6664, LTC4150, DS1682S, MAX11611"
- note added: "TODO: Redo this connector"
Changed lines of the file:
@@
 	1    0    0    -1
 $EndComp
+Text Notes 4200 14600 0    50   ~ 0
+TODO: Redo this connector
+Text Label 9200 11000 0    50   ~ 0
+CHARGE_STAT
+Text Label 9200 11300 0    60   ~ 0
+UMB_VCC
+$Comp
+L power:+12V #PWR?
+U 1 1 5BBFC6B2
+P 9700 11200
+F 0 "#PWR?" H 9700 11050 50  0001 C CNN
+F 1 "+12V" H 9700 11340 50  0000 C CNN
+F 2 "" H 9700 11200 50  0001 C CNN
+F 3 "" H 9700 11200 50  0001 C CNN
+	1    9700 11200
+	1    0    0    -1
+$EndComp
+$Comp
+L power:+3V3 #PWR?
+U 1 1 5BBFCB8D
+P 9900 11100
+F 0 "#PWR?" H 9900 10950 50  0001 C CNN
+F 1 "+3V3" H 9900 11250 50  0000 C CNN
+F 2 "" H 9900 11100 50  0001 C CNN
+F 3 "" H 9900 11100 50  0001 C CNN
+	1    9900 11100
+	1    0    0    -1
+$EndComp
+Text Label 9200 11400 0    60   ~ 0
+BAT_VCC
+Text Label 9200 11500 0    60   ~ 0
+BAT_BAK_VCC
+Text Label 9200 11700 0    50   ~ 0
+BAT_CELL_1
+Text Label 9200 11600 0    60   ~ 0
+VCC_IN
+Text Label 9200 11800 0    50   ~ 0
+THERM1
+Text Label 9200 11900 0    50   ~ 0
+THERM2
+Text Label 9200 12000 0    50   ~ 0
+THERM3
+Text Label 9200 12100 0    50   ~ 0
+THERM4
+Wire Wire Line
+	9900 11100 9000 11100
+Wire Wire Line
+	9200 11000 9000 11000
+Wire Wire Line
+	9700 11200 9000 11200
+Wire Wire Line
+	9200 11300 9000 11300
+Wire Wire Line
+	9200 11400 9000 11400
+Wire Wire Line
+	9200 11500 9000 11500
+Wire Wire Line
+	9200 11600 9000 11600
+Wire Wire Line
+	9200 11700 9000 11700
+Wire Wire Line
+	9200 11800 9000 11800
+Wire Wire Line
+	9200 11900 9000 11900
+Wire Wire Line
+	9200 12000 9000 12000
+Wire Wire Line
+	9200 12100 9000 12100
+$Comp
+L SparkFun-IC-Power:LTC4150 U?
+U 1 1 5BCD2784
+P 9400 9950
+F 0 "U?" H 9400 10710 45  0000 C CNN
+F 1 "LTC4150" H 9400 10626 45  0000 C CNN
+F 2 "MSOP10" H 9400 10550 20  0001 C CNN
+F 3 "" H 9400 9950 60  0001 C CNN
+F 4 "IC-11785" H 9400 10531 60  0000 C CNN "Field4"
+	1    9400 9950
+	1    0    0    -1
+$EndComp
+Text Notes 11100 9400 0    50   ~ 0
+TODO: MAX6664, LTC4150, DS1682S, MAX11611
+Text Notes 11100 9500 0    50   ~ 0
+Figure out replacement for DS1682S or a way to get it to count down
 $EndSCHEMATC

Commit message: Changed power board monitoring strategy
Now has onboard MCU
Parts:
- added C? (x2): 4.7 µF, symbol Device:C_Small
- added R?: R, symbol Device:R
- added R? (x2): R_Small, symbol Device:R_Small
- added U?: ATxmega32E5-AU, Package_QFP:TQFP-32_7x7mm_P0.8mm, symbol MCU_Microchip_ATmega:ATxmega32E5-AU
Connections:
- net labels added: 12V_SENS, 3V3_SENS, BAL_OUT, BAT_BAK_VCC_SENS, BAT_CELL_1_SENS, BAT_CELL_2_CONN, BAT_VCC_CONN, BAT_VCC_SENS, LVL_POL, LVL_~INT~, LVL_~SHDN~, MCU_SCL, MCU_SDA, SEL_~SHDN~, THERM5, THERM6, THERM7, UMB_VCC_SENS, VCC_IN_SENS
- wire segments 272 -> 290
Other:
- note added: "Shunt Resistor\nTODO: Decide Value"
- note added: "TODO: LTC4150, ATXMEGA32E5"
- note added: "TODO: Redo this connector on other boards\n(Also make the footprint bigger)"
- note removed: "Figure out replacement for DS1682S or a way to get it to count down"
- note removed: "TODO: MAX6664, LTC4150, DS1682S, MAX11611"
- note removed: "TODO: Redo this connector"

Commit message: Schematic done (again)
Still needs footprints and part numbers
Parts:
- removed R? (x2): R_Small, symbol Device:R_Small
- added C? (x2): 0.1 µF, Capacitors_SMD:C_0603, symbol Device:C_Small
- added C? (x2): 10 µF, Capacitors_SMD:C_0603, symbol Device:C_Small
- added J?: Conn_02x03_Odd_Even, symbol Connector_Generic:Conn_02x03_Odd_Even
- added L?: 220 Ω @ 100 MHz, symbol Device:Ferrite_Bead_Small
- added L?: 10 µH, symbol Device:L_Small
- added R? (x7): 121 kΩ, symbol Device:R_Small
- added R? (x10): 10 kΩ, symbol Device:R_Small
- added R? (x3): 100 kΩ, Resistors_SMD:R_0603, symbol Device:R_Small
- added R? (x6): 64.9 kΩ, symbol Device:R_Small
- added TH? (x6): NXFT15XH103FA2B100, symbol Device:Thermistor_NTC
- R?: value R -> 2.5 mΩ; Digikey Part Number (none) -> A131768CT-ND
Connections:
- net labels added: SEL_~VALID1~, SEL_~VALID2~, SEL_~VALID3~
- net labels removed: THERM7
- wire segments 290 -> 341
- no-connect marks 0 -> 2
Other:
- note added: "Close to\npower supply"
- note removed: "If this shows up as a box with a question mark\nlook at the exported pdf schematic instead"
- note removed: "Shunt Resistor\nTODO: Decide Value"
- note removed: "TODO: LTC4150, ATXMEGA32E5"
