File: Power Board/Power Board.sch (KiCad schematic (older format))
At the start: 151 parts, among them J1 Conn_02x03_Odd_Even, J2 Conn_01x02, J3 Conn_01x02, J4 Conn_01x02, J5 Conn_01x02, J6 Conn_01x02, J7 Conn_01x03, J8 Conn_02x07_Counter_Clockwise, Q1 SI7157DP, Q2 SI7157DP, Q3 SI7157DP, Q4 SI7157DP, Q5 SI7157DP, Q6 SI7157DP, Q7 AON7423, U1 LTC4417CGN, U10 LMR62014XMF, U2 TPS564208DDCT, U3 LTC3130-1, U4 BQ2057WSNTR, U5 BQ29209DRBT, U6 LT6700CS6-1, U7 STS8C5H30L, U8 LTC4150, U9 ATxmega32E5-AU

Commit message: One more footprint
Parts:
- L5: footprint (none) -> Custom Parts:L_SLF10165
Changed lines of the file:
@@
 F 0 "L5" V 14690 1800 50  0000 C CNN
 F 1 "10 µH" V 14599 1800 50  0000 C CNN
-F 2 "" H 14500 1800 50  0001 C CNN
+F 2 "Custom Parts:L_SLF10165" H 14500 1800 50  0001 C CNN
 F 3 "~" H 14500 1800 50  0001 C CNN
 F 4 "445-6478-1-ND" V 14500 1800 50  0001 C CNN "Digikey Part Number"

Commit message: Apparently connector footprints are odd-even by default, not counterclockwise
Parts:
- removed J8: Conn_02x07_Counter_Clockwise, Pin_Headers:Pin_Header_Straight_2x07_Pitch2.54mm, symbol Power-Board-rescue:Conn_02x07_Counter_Clockwise-Connector_Generic
- added J?: Conn_02x07_Odd_Even, Pin_Headers:Pin_Header_Straight_2x07_Pitch2.54mm, symbol Connector_Generic:Conn_02x07_Odd_Even
- HS1: footprint (none) -> Custom Parts:HS_ATS1099
- J1: footprint (none) -> Pin_Headers:Pin_Header_Straight_2x03_Pitch1.27mm_SMD
Changed lines of the file:
@@
 F 0 "HS1" H 7592 1971 50  0000 L CNN
 F 1 "Heatsink" H 7592 1880 50  0000 L CNN
-F 2 "" H 7462 1850 50  0001 C CNN
+F 2 "Custom Parts:HS_ATS1099" H 7462 1850 50  0001 C CNN
 F 3 "" H 7462 1850 50  0001 C CNN
 F 4 "ATS1099-ND" H 7450 1850 50  0001 C CNN "Digikey Part Number"
@@
 F 0 "J1" H 10500 14900 50  0000 C CNN
 F 1 "Conn_02x03_Odd_Even" H 10100 14800 50  0000 C CNN
-F 2 "" H 10450 15150 50  0001 C CNN
+F 2 "Pin_Headers:Pin_Header_Straight_2x03_Pitch1.27mm_SMD" H 10450 15150 50  0001 C CNN
 F 3 "" H 10450 15150 50  0001 C CNN
 F 4 "609-3693-1-ND" H -400 0   50  0001 C CNN "Digikey Part Number"
@@
 Text Label 13800 19100 2    50   ~ 0
 THERM1
-$Comp
-L Power-Board-rescue:Conn_02x07_Counter_Clockwise-Connector_Generic J8
-U 1 1 5C0B7D8D
-P 3350 16950
-F 0 "J8" H 3400 17467 50  0000 C CNN
-F 1 "Conn_02x07_Counter_Clockwise" H 3400 17376 50  0000 C CNN
-F 2 "Pin_Headers:Pin_Header_Straight_2x07_Pitch2.54mm" H 3350 16950 50  0001 C CNN
-F 3 "" H 3350 16950 50  0001 C CNN
-F 4 "952-1932-ND" H 0   0   50  0001 C CNN "Digikey Part Number"
-	1    3350 16950
-	1    0    0    -1
-$EndComp
 $Comp
 L Power-Board-rescue:+3V3-power #PWR053
@@
 Wire Wire Line
 	11900 14250 11900 14100
+$Comp
+L Connector_Generic:Conn_02x07_Odd_Even J?
+U 1 1 5C438F55
+P 3350 16950
+F 0 "J?" H 3400 17467 50  0000 C CNN
+F 1 "Conn_02x07_Odd_Even" H 3400 17376 50  0000 C CNN
+F 2 "Pin_Headers:Pin_Header_Straight_2x07_Pitch2.54mm" H 3350 16950 50  0001 C CNN
+F 3 "~" H 3350 16950 50  0001 C CNN
+F 4 "952-1932-ND" H 3350 16950 50  0001 C CNN "Digikey Part Number"
+	1    3350 16950
+	1    0    0    -1
+$EndComp
 $EndSCHEMATC

Commit message: Power Board Footprints Done!
Parts:
- J2, J3, J4, J5: footprint (none) -> Custom Parts:XT30_Angled
- TH1, TH2, TH3, TH4, TH5, TH6, TH7: footprint (none) -> Custom Parts:Thermistor_Through_Hole_Tiny
- gave numbers to parts that had none: 11
Changed lines of the file:
@@
 F 0 "J2" H 5080 19042 50  0000 L CNN
 F 1 "Conn_01x02" H 5080 18951 50  0000 L CNN
-F 2 "" H 5000 19050 50  0001 C CNN
+F 2 "Custom Parts:XT30_Angled" H 5000 19050 50  0001 C CNN
 F 3 "" H 5000 19050 50  0001 C CNN
 F 4 "https://www.aliexpress.com/item/AMASS-XT30PW-Banana-golden-XT30-Upgrade-Right-Angle-Plug-Connector-male-female-ESC-Motor-PCB-board/32689137918.html" H 5180 19142 50  0001 C CNN "AliExpress Part Link"
@@
 F 0 "J3" H 5080 19342 50  0000 L CNN
 F 1 "Conn_01x02" H 5080 19251 50  0000 L CNN
-F 2 "" H 5000 19350 50  0001 C CNN
+F 2 "Custom Parts:XT30_Angled" H 5000 19350 50  0001 C CNN
 F 3 "" H 5000 19350 50  0001 C CNN
 F 4 "" H 0   0   50  0001 C CNN "Digikey Part Number"
@@
 F 0 "J4" H 5080 19642 50  0000 L CNN
 F 1 "Conn_01x02" H 5080 19551 50  0000 L CNN
-F 2 "" H 5000 19650 50  0001 C CNN
+F 2 "Custom Parts:XT30_Angled" H 5000 19650 50  0001 C CNN
 F 3 "" H 5000 19650 50  0001 C CNN
 F 4 "" H 0   0   50  0001 C CNN "Digikey Part Number"
@@
 F 0 "J5" H 5080 19942 50  0000 L CNN
 F 1 "Conn_01x02" H 5080 19851 50  0000 L CNN
-F 2 "" H 5000 19950 50  0001 C CNN
+F 2 "Custom Parts:XT30_Angled" H 5000 19950 50  0001 C CNN
 F 3 "" H 5000 19950 50  0001 C CNN
 F 4 "" H 0   0   50  0001 C CNN "Digikey Part Number"
@@
 F 0 "TH1" H 11500 5750 50  0000 L CNN
 F 1 "NXFT15XH103FA2B100" H 10800 5650 50  0000 L CNN
-F 2 "" H 11800 5750 50  0001 C CNN
+F 2 "Custom Parts:Thermistor_Through_Hole_Tiny" H 11800 5750 50  0001 C CNN
 F 3 "" H 11800 5750 50  0001 C CNN
 F 4 "490-5630-ND" H 11800 5700 50  0001 C CNN "Digikey Part Number"
@@
 F 0 "TH2" H 13500 19350 50  0000 L CNN
 F 1 "NXFT15XH103FA2B100" H 12800 19250 50  0000 L CNN
-F 2 "" H 13800 19350 50  0001 C CNN
+F 2 "Custom Parts:Thermistor_Through_Hole_Tiny" H 13800 19350 50  0001 C CNN
 F 3 "" H 13800 19350 50  0001 C CNN
 F 4 "490-5630-ND" H 13800 19300 50  0001 C CNN "Digikey Part Number"
@@
 F 0 "TH4" H 13500 20650 50  0000 L CNN
 F 1 "NXFT15XH103FA2B100" H 12800 20550 50  0000 L CNN
-F 2 "" H 13800 20650 50  0001 C CNN
+F 2 "Custom Parts:Thermistor_Through_Hole_Tiny" H 13800 20650 50  0001 C CNN
 F 3 "" H 13800 20650 50  0001 C CNN
 F 4 "490-5630-ND" H 13800 20600 50  0001 C CNN "Digikey Part Number"
@@
 F 0 "TH6" H 13500 21950 50  0000 L CNN
 F 1 "NXFT15XH103FA2B100" H 12800 21850 50  0000 L CNN
-F 2 "" H 13800 21950 50  0001 C CNN
+F 2 "Custom Parts:Thermistor_Through_Hole_Tiny" H 13800 21950 50  0001 C CNN
 F 3 "" H 13800 21950 50  0001 C CNN
 F 4 "490-5630-ND" H 13800 21900 50  0001 C CNN "Digikey Part Number"
@@
 F 0 "TH3" H 14800 19350 50  0000 L CNN
 F 1 "NXFT15XH103FA2B100" H 14100 19250 50  0000 L CNN
-F 2 "" H 15100 19350 50  0001 C CNN
+F 2 "Custom Parts:Thermistor_Through_Hole_Tiny" H 15100 19350 50  0001 C CNN
 F 3 "" H 15100 19350 50  0001 C CNN
 F 4 "490-5630-ND" H 15100 19300 50  0001 C CNN "Digikey Part Number"
@@
 F 0 "TH5" H 14800 20650 50  0000 L CNN
 F 1 "NXFT15XH103FA2B100" H 14100 20550 50  0000 L CNN
-F 2 "" H 15100 20650 50  0001 C CNN
+F 2 "Custom Parts:Thermistor_Through_Hole_Tiny" H 15100 20650 50  0001 C CNN
 F 3 "" H 15100 20650 50  0001 C CNN
 F 4 "490-5630-ND" H 15100 20600 50  0001 C CNN "Digikey Part Number"
@@
 F 0 "TH7" H 14800 21950 50  0000 L CNN
 F 1 "NXFT15XH103FA2B100" H 14100 21850 50  0000 L CNN
-F 2 "" H 15100 21950 50  0001 C CNN
+F 2 "Custom Parts:Thermistor_Through_Hole_Tiny" H 15100 21950 50  0001 C CNN
 F 3 "" H 15100 21950 50  0001 C CNN
 F 4 "490-5630-ND" H 15100 21900 50  0001 C CNN "Digikey Part Number"
@@
 BAT_CHARGE_EN
 $Comp
-L Custom_Parts:TPS22810 U?
+L Custom_Parts:TPS22810 U11
 U 1 1 5C3F6B0F
 P 17150 2400
-F 0 "U?" H 17150 2865 50  0000 C CNN
+F 0 "U11" H 17150 2865 50  0000 C CNN
 F 1 "TPS22810" H 17150 2774 50  0000 C CNN
 F 2 "TO_SOT_Packages_SMD:SOT-23-6" H 17100 2400 50  0001 C CNN
@@
 	16500 2400 16500 2900
 $Comp
-L Power-Board-rescue:GND-power #PWR?
+L Power-Board-rescue:GND-power #PWR0101
 U 1 1 5C47E10D
 P 16500 2900
-F 0 "#PWR?" H 16500 2650 50  0001 C CNN
+F 0 "#PWR0101" H 16500 2650 50  0001 C CNN
 F 1 "GND" V 16500 2700 50  0000 C CNN
 F 2 "" H 16500 2900 50  0001 C CNN
@@
 High side load switch to prevent the battery charger from\ntrying to run if the step up converter is disabled.
 $Comp
-L Device:D_TVS D?
+L Device:D_TVS D15
 U 1 1 5C50A71C
 P 1800 12250
-F 0 "D?" V 1754 12329 50  0000 L CNN
+F 0 "D15" V 1754 12329 50  0000 L CNN
 F 1 "12V TVS" V 1845 12329 50  0000 L CNN
 F 2 "Custom Parts:TVS_0603" H 1800 12250 50  0001 C CNN
@@
 	1800 12100 2250 12100
 $Comp
-L Power-Board-rescue:GND-power #PWR?
+L Power-Board-rescue:GND-power #PWR0102
 U 1 1 5C50A9C8
 P 1800 12400
-F 0 "#PWR?" H 1800 12150 50  0001 C CNN
+F 0 "#PWR0102" H 1800 12150 50  0001 C CNN
 F 1 "GND" H 1800 12250 50  0000 C CNN
 F 2 "" H 1800 12400 50  0001 C CNN
@@
 $EndComp
 $Comp
-L Device:D_TVS D?
+L Device:D_TVS D16
 U 1 1 5C52CE60
 P 4750 12250
-F 0 "D?" V 4704 12329 50  0000 L CNN
+F 0 "D16" V 4704 12329 50  0000 L CNN
 F 1 "12V TVS" V 4795 12329 50  0000 L CNN
 F 2 "Custom Parts:TVS_0603" H 4750 12250 50  0001 C CNN
@@
 	4750 12100 4950 12100
 $Comp
-L Power-Board-rescue:GND-power #PWR?
+L Power-Board-rescue:GND-power #PWR0103
 U 1 1 5C52CFB6
 P 4750 12400
-F 0 "#PWR?" H 4750 12150 50  0001 C CNN
+F 0 "#PWR0103" H 4750 12150 50  0001 C CNN
 F 1 "GND" H 4750 12250 50  0000 C CNN
 F 2 "" H 4750 12400 50  0001 C CNN
@@
 $EndComp
 $Comp
-L Device:D_TVS D?
+L Device:D_TVS D12
 U 1 1 5C52D0E8
 P 2150 8750
-F 0 "D?" V 2104 8829 50  0000 L CNN
+F 0 "D12" V 2104 8829 50  0000 L CNN
 F 1 "12V TVS" V 2195 8829 50  0000 L CNN
 F 2 "Custom Parts:TVS_0603" H 2150 8750 50  0001 C CNN
@@
 	2150 8600 2450 8600
 $Comp
-L Power-Board-rescue:GND-power #PWR?
+L Power-Board-rescue:GND-power #PWR0104
 U 1 1 5C52DA25
 P 2150 8900
-F 0 "#PWR?" H 2150 8650 50  0001 C CNN
+F 0 "#PWR0104" H 2150 8650 50  0001 C CNN
 F 1 "GND" H 2150 8750 50  0000 C CNN
 F 2 "" H 2150 8900 50  0001 C CNN
@@
 $EndComp
 $Comp
-L Power-Board-rescue:GND-power #PWR?
+L Power-Board-rescue:GND-power #PWR0105
 U 1 1 5C52DCBD
 P 5850 9100
-F 0 "#PWR?" H 5850 8850 50  0001 C CNN
+F 0 "#PWR0105" H 5850 8850 50  0001 C CNN
 F 1 "GND" H 5850 8950 50  0000 C CNN
 F 2 "" H 5850 9100 50  0001 C CNN
@@
 $EndComp
 $Comp
-L Device:D_TVS D?
+L Device:D_TVS D11
 U 1 1 5C52DDF3
 P 5050 2950
-F 0 "D?" V 5004 3029 50  0000 L CNN
+F 0 "D11" V 5004 3029 50  0000 L CNN
 F 1 "12V TVS" V 5095 3029 50  0000 L CNN
 F 2 "Custom Parts:TVS_0603" H 5050 2950 50  0001 C CNN
@@
 	5050 2800 6700 2800
 $Comp
-L Device:D_TVS D?
+L Device:D_TVS D10
 U 1 1 5C52F331
 P 4800 2550
-F 0 "D?" V 4754 2629 50  0000 L CNN
+F 0 "D10" V 4754 2629 50  0000 L CNN
 F 1 "12V TVS" V 4845 2629 50  0000 L CNN
 F 2 "Custom Parts:TVS_0603" H 4800 2550 50  0001 C CNN
@@
 	4800 2400 5900 2400
 $Comp
-L Device:D_TVS D?
+L Device:D_TVS D9
 U 1 1 5C52F47D
 P 4600 2150
-F 0 "D?" V 4554 2229 50  0000 L CNN
+F 0 "D9" V 4554 2229 50  0000 L CNN
 F 1 "12V TVS" V 4645 2229 50  0000 L CNN
 F 2 "Custom Parts:TVS_0603" H 4600 2150 50  0001 C CNN
@@
 	4600 2000 5100 2000
 $Comp
-L Power-Board-rescue:GND-power #PWR?
+L Power-Board-rescue:GND-power #PWR0106
 U 1 1 5C52F5C7
 P 5050 3100
-F 0 "#PWR?" H 5050 2850 50  0001 C CNN
+F 0 "#PWR0106" H 5050 2850 50  0001 C CNN
 F 1 "GND" H 5050 2950 50  0000 C CNN
 F 2 "" H 5050 3100 50  0001 C CNN
@@
 $EndComp
 $Comp
-L Power-Board-rescue:GND-power #PWR?
+L Power-Board-rescue:GND-power #PWR0107
 U 1 1 5C52F702
 P 4800 3100
-F 0 "#PWR?" H 4800 2850 50  0001 C CNN
+F 0 "#PWR0107" H 4800 2850 50  0001 C CNN
 F 1 "GND" H 4800 2950 50  0000 C CNN
 F 2 "" H 4800 3100 50  0001 C CNN
@@
 $EndComp
 $Comp
-L Power-Board-rescue:GND-power #PWR?
+L Power-Board-rescue:GND-power #PWR0108
 U 1 1 5C52F83D
 P 4600 3100
-F 0 "#PWR?" H 4600 2850 50  0001 C CNN
+F 0 "#PWR0108" H 4600 2850 50  0001 C CNN
 F 1 "GND" H 4600 2950 50  0000 C CNN
 F 2 "" H 4600 3100 50  0001 C CNN
@@
 	5550 8800 5850 8800
 $Comp
-L Device:D_TVS D?
+L Device:D_TVS D14
 U 1 1 5C5C1214
 P 5850 8950
-F 0 "D?" V 5804 9029 50  0000 L CNN
+F 0 "D14" V 5804 9029 50  0000 L CNN
 F 1 "3.3V TVS" V 5895 9029 50  0000 L CNN
 F 2 "Custom Parts:TVS_0402" H 5850 8950 50  0001 C CNN
@@
 	5850 8800 6050 8800
 $Comp
-L Device:D_TVS D?
+L Device:D_TVS D18
 U 1 1 5C5C17B0
 P 12050 14250
-F 0 "D?" V 12004 14329 50  0000 L CNN
+F 0 "D18" V 12004 14329 50  0000 L CNN
 F 1 "3.3V TVS" V 12095 14329 50  0000 L CNN
 F 2 "Custom Parts:TVS_0402" H 12050 14250 50  0001 C CNN
@@
 $EndComp
 $Comp
-L Device:D_TVS D?
+L Device:D_TVS D17
 U 1 1 5C5C22E7
 P 12050 14100
-F 0 "D?" V 12004 14179 50  0000 L CNN
+F 0 "D17" V 12004 14179 50  0000 L CNN
 F 1 "3.3V TVS" V 12095 14179 50  0000 L CNN
 F 2 "Custom Parts:TVS_0402" H 12050 14100 50  0001 C CNN
@@
 	12850 14250 12850 13800
 $Comp
-L Power-Board-rescue:GND-power #PWR?
+L Power-Board-rescue:GND-power #PWR0109
 U 1 1 5C654E2B
 P 11900 14400
-F 0 "#PWR?" H 11900 14150 50  0001 C CNN
+F 0 "#PWR0109" H 11900 14150 50  0001 C CNN
 F 1 "GND" H 11800 14300 50  0000 C CNN
 F 2 "" H 11900 14400 50  0001 C CNN
@@
 	11900 14250 11900 14100
 $Comp
-L Connector_Generic:Conn_02x07_Odd_Even J?
+L Connector_Generic:Conn_02x07_Odd_Even J8
 U 1 1 5C438F55
 P 3350 16950
-F 0 "J?" H 3400 17467 50  0000 C CNN
+F 0 "J8" H 3400 17467 50  0000 C CNN
 F 1 "Conn_02x07_Odd_Even" H 3400 17376 50  0000 C CNN
 F 2 "Pin_Headers:Pin_Header_Straight_2x07_Pitch2.54mm" H 3350 16950 50  0001 C CNN

Commit message: Finally ready to redo power PCB
Parts:
- C1: footprint Custom Footprints:CP_Radial_Horiz_D8.0mm_L13.00mm_P3.50mm -> Custom Parts:CP_Radial_Horiz_D8.0mm_L13.00mm_P3.50mm
- L1: footprint Custom Parts:3.3v DC-DC Inductor -> Custom Parts:L_SRP6540
- L2: footprint Custom Footprints:L_Wuerth_7447779115 -> Custom Parts:L_Wuerth_7447779115
- Q1, Q2, Q3, Q4, Q5, Q6: footprint Custom Footprints:PowerPAK_SO-8 -> Custom Parts:PowerPAK_SO-8
- Q7: value AON7423 -> DMG2305UX; footprint Custom Parts:AON7423 -> TO_SOT_Packages_SMD:SOT-23; symbol Power-Board-rescue:Q_PMOS_SGD-Device -> Device:Q_PMOS_GDS; Digikey Part Number 785-1310-1-ND -> DMG2305UX-13DICT-ND
- U10: footprint Package_TO_SOT_SMD:SOT-23-5 -> TO_SOT_Packages_SMD:SOT-23-5
- U9: footprint Package_QFP:TQFP-32_7x7mm_P0.8mm -> Housings_QFP:TQFP-32_7x7mm_Pitch0.8mm
Changed lines of the file:
@@
 F 0 "Q1" H 5500 2150 50  0000 L CNN
 F 1 "SI7157DP" H 5500 2050 50  0000 L CNN
-F 2 "Custom Footprints:PowerPAK_SO-8" H 5500 2200 50  0001 C CNN
+F 2 "Custom Parts:PowerPAK_SO-8" H 5500 2200 50  0001 C CNN
 F 3 "" H 5300 2100 50  0001 C CNN
 F 4 "SI7157DP-T1-GE3CT-ND" H 5500 2250 50  0001 C CNN "Digikey Part Number"
@@
 F 0 "Q2" H 6000 2150 50  0000 L CNN
 F 1 "SI7157DP" H 6000 2050 50  0000 L CNN
-F 2 "Custom Footprints:PowerPAK_SO-8" H 6000 2200 50  0001 C CNN
+F 2 "Custom Parts:PowerPAK_SO-8" H 6000 2200 50  0001 C CNN
 F 3 "" H 5800 2100 50  0001 C CNN
 F 4 "SI7157DP-T1-GE3CT-ND" H 6000 2250 50  0001 C CNN "Digikey Part Number"
@@
 F 0 "Q3" H 6300 2550 50  0000 L CNN
 F 1 "SI7157DP" H 6300 2450 50  0000 L CNN
-F 2 "Custom Footprints:PowerPAK_SO-8" H 6300 2600 50  0001 C CNN
+F 2 "Custom Parts:PowerPAK_SO-8" H 6300 2600 50  0001 C CNN
 F 3 "" H 6100 2500 50  0001 C CNN
 F 4 "SI7157DP-T1-GE3CT-ND" H 6300 2650 50  0001 C CNN "Digikey Part Number"
@@
 F 0 "Q4" H 6800 2550 50  0000 L CNN
 F 1 "SI7157DP" H 6800 2450 50  0000 L CNN
-F 2 "Custom Footprints:PowerPAK_SO-8" H 6800 2600 50  0001 C CNN
+F 2 "Custom Parts:PowerPAK_SO-8" H 6800 2600 50  0001 C CNN
 F 3 "" H 6600 2500 50  0001 C CNN
 F 4 "SI7157DP-T1-GE3CT-ND" H 6800 2650 50  0001 C CNN "Digikey Part Number"
@@
 F 0 "Q5" H 7100 2950 50  0000 L CNN
 F 1 "SI7157DP" H 7100 2850 50  0000 L CNN
-F 2 "Custom Footprints:PowerPAK_SO-8" H 7100 3000 50  0001 C CNN
+F 2 "Custom Parts:PowerPAK_SO-8" H 7100 3000 50  0001 C CNN
 F 3 "" H 6900 2900 50  0001 C CNN
 F 4 "SI7157DP-T1-GE3CT-ND" H 7100 3050 50  0001 C CNN "Digikey Part Number"
@@
 F 0 "Q6" H 7600 2950 50  0000 L CNN
 F 1 "SI7157DP" H 7600 2850 50  0000 L CNN
-F 2 "Custom Footprints:PowerPAK_SO-8" H 7600 3000 50  0001 C CNN
+F 2 "Custom Parts:PowerPAK_SO-8" H 7600 3000 50  0001 C CNN
 F 3 "" H 7400 2900 50  0001 C CNN
 F 4 "SI7157DP-T1-GE3CT-ND" H 7600 3050 50  0001 C CNN "Digikey Part Number"
@@
 F 0 "C1" H 8610 2370 50  0000 L CNN
 F 1 "470 µF" H 8610 2220 50  0000 L CNN
-F 2 "Custom Footprints:CP_Radial_Horiz_D8.0mm_L13.00mm_P3.50mm" H 8600 2300 50  0001 C CNN
+F 2 "Custom Parts:CP_Radial_Horiz_D8.0mm_L13.00mm_P3.50mm" H 8600 2300 50  0001 C CNN
 F 3 "" H 8600 2300 50  0001 C CNN
 F 4 "1189-1733-ND" H 8610 2470 50  0001 C CNN "Digikey Part Number"
@@
 F 0 "L1" H 4580 8840 50  0000 L CNN
 F 1 "2.2 µH" H 4580 8760 50  0000 L CNN
-F 2 "Custom Parts:3.3v DC-DC Inductor" H 4550 8800 50  0001 C CNN
+F 2 "Custom Parts:L_SRP6540" H 4550 8800 50  0001 C CNN
 F 3 "" H 4550 8800 50  0001 C CNN
 F 4 "SRP6540-2R2MCT-ND" H 4550 8800 50  0001 C CNN "Digikey Part Number"
@@
 F 0 "L2" H 3430 11640 50  0000 L CNN
 F 1 "15 µH" H 3430 11560 50  0000 L CNN
-F 2 "Custom Footprints:L_Wuerth_7447779115" H 3400 11600 50  0001 C CNN
+F 2 "Custom Parts:L_Wuerth_7447779115" H 3400 11600 50  0001 C CNN
 F 3 "" H 3400 11600 50  0001 C CNN
 F 4 "732-4180-1-ND" H 3430 11740 50  0001 C CNN "Digikey Part Number"
@@
 $EndComp
 $Comp
-L Power-Board-rescue:Q_PMOS_SGD-Device Q7
+L Device:Q_PMOS_GDS Q7
 U 1 1 5B823DE9
 P 15250 4450
 F 0 "Q7" V 15593 4450 50  0000 C CNN
-F 1 "AON7423" V 15502 4450 50  0000 C CNN
-F 2 "Custom Parts:AON7423" H 15450 4550 50  0001 C CNN
+F 1 "DMG2305UX" V 15502 4450 50  0000 C CNN
+F 2 "TO_SOT_Packages_SMD:SOT-23" H 15450 4550 50  0001 C CNN
 F 3 "" H 15250 4450 50  0001 C CNN
-F 4 "785-1310-1-ND" V 15250 4450 50  0001 C CNN "Digikey Part Number"
+F 4 "DMG2305UX-13DICT-ND" V 15250 4450 50  0001 C CNN "Digikey Part Number"
 	1    15250 4450
 	0    1    -1   0
@@
 F 0 "U9" H 13050 14450 50  0000 C CNN
 F 1 "ATxmega32E5-AU" H 13350 14350 50  0000 C CNN
-F 2 "Package_QFP:TQFP-32_7x7mm_P0.8mm" H 12850 15550 50  0001 C CIN
+F 2 "Housings_QFP:TQFP-32_7x7mm_Pitch0.8mm" H 12850 15550 50  0001 C CIN
 F 3 "http://ww1.microchip.com/downloads/en/DeviceDoc/Atmel-8153-8-and-16-bit-AVR-Microcontroller-XMEGA-E-ATxmega8E5-ATxmega16E5-ATxmega32E5_Datasheet.pdf" H 12850 15550 50  0001 C CNN
 F 4 "ATXMEGA32E5-AU-ND" H 0   0   50  0001 C CNN "Digikey Part Number"
@@
 F 0 "U10" H 14500 2667 50  0000 C CNN
 F 1 "LMR62014XMF" H 14500 2576 50  0000 C CNN
-F 2 "Package_TO_SOT_SMD:SOT-23-5" H 14550 2050 50  0001 L CIN
+F 2 "TO_SOT_Packages_SMD:SOT-23-5" H 14550 2050 50  0001 L CIN
 F 3 "http://www.ti.com/lit/ds/symlink/lmr62014.pdf" H 14500 2400 50  0001 C CNN
 F 4 "LMR62014XMF/NOPBCT-ND" H 14500 2300 50  0001 C CNN "Digikey Part Number"

Commit message: Switching to a screw terminal for power board
Parts:
- removed J2, J3, J4, J5: Conn_01x02, Custom Parts:XT30_Angled, symbol Power-Board-rescue:Conn_01x02-Connector-Power-Board-rescue
- added J?: Screw_Terminal_01x06, symbol Connector:Screw_Terminal_01x06
Changed lines of the file:
@@
 	1    0    0    -1
 $EndComp
-$Comp
-L Power-Board-rescue:Conn_01x02-Connector-Power-Board-rescue J2
-U 1 1 5AA75ED0
-P 5000 19050
-F 0 "J2" H 5080 19042 50  0000 L CNN
-F 1 "Conn_01x02" H 5080 18951 50  0000 L CNN
-F 2 "Custom Parts:XT30_Angled" H 5000 19050 50  0001 C CNN
-F 3 "" H 5000 19050 50  0001 C CNN
-F 4 "https://www.aliexpress.com/item/AMASS-XT30PW-Banana-golden-XT30-Upgrade-Right-Angle-Plug-Connector-male-female-ESC-Motor-PCB-board/32689137918.html" H 5180 19142 50  0001 C CNN "AliExpress Part Link"
-	1    5000 19050
-	1    0    0    -1
-$EndComp
-Text Label 4800 19050 2    60   ~ 0
+Text Label 5100 19150 2    60   ~ 0
 VCC_IN
-$Comp
-L Power-Board-rescue:GND-power #PWR037
-U 1 1 5AA762AB
-P 4800 19150
-F 0 "#PWR037" H 4800 18900 50  0001 C CNN
-F 1 "GND" V 4800 18950 50  0000 C CNN
-F 2 "" H 4800 19150 50  0001 C CNN
-F 3 "" H 4800 19150 50  0001 C CNN
-	1    4800 19150
-	0    1    -1   0
-$EndComp
-$Comp
-L Power-Board-rescue:Conn_01x02-Connector-Power-Board-rescue J3
-U 1 1 5AA7656E
-P 5000 19350
-F 0 "J3" H 5080 19342 50  0000 L CNN
-F 1 "Conn_01x02" H 5080 19251 50  0000 L CNN
-F 2 "Custom Parts:XT30_Angled" H 5000 19350 50  0001 C CNN
-F 3 "" H 5000 19350 50  0001 C CNN
-F 4 "" H 0   0   50  0001 C CNN "Digikey Part Number"
-F 5 "https://www.aliexpress.com/item/AMASS-XT30PW-Banana-golden-XT30-Upgrade-Right-Angle-Plug-Connector-male-female-ESC-Motor-PCB-board/32689137918.html" H 0   0   50  0001 C CNN "AliExpress Part Link"
-	1    5000 19350
-	1    0    0    -1
-$EndComp
-$Comp
-L Power-Board-rescue:Conn_01x02-Connector-Power-Board-rescue J4
-U 1 1 5AA765F7
-P 5000 19650
-F 0 "J4" H 5080 19642 50  0000 L CNN
-F 1 "Conn_01x02" H 5080 19551 50  0000 L CNN
-F 2 "Custom Parts:XT30_Angled" H 5000 19650 50  0001 C CNN
-F 3 "" H 5000 19650 50  0001 C CNN
-F 4 "" H 0   0   50  0001 C CNN "Digikey Part Number"
-F 5 "https://www.aliexpress.com/item/AMASS-XT30PW-Banana-golden-XT30-Upgrade-Right-Angle-Plug-Connector-male-female-ESC-Motor-PCB-board/32689137918.html" H 0   0   50  0001 C CNN "AliExpress Part Link"
-	1    5000 19650
-	1    0    0    -1
-$EndComp
-$Comp
-L Power-Board-rescue:Conn_01x02-Connector-Power-Board-rescue J5
-U 1 1 5AA76683
-P 5000 19950
-F 0 "J5" H 5080 19942 50  0000 L CNN
-F 1 "Conn_01x02" H 5080 19851 50  0000 L CNN
-F 2 "Custom Parts:XT30_Angled" H 5000 19950 50  0001 C CNN
-F 3 "" H 5000 19950 50  0001 C CNN
-F 4 "" H 0   0   50  0001 C CNN "Digikey Part Number"
-F 5 "https://www.aliexpress.com/item/AMASS-XT30PW-Banana-golden-XT30-Upgrade-Right-Angle-Plug-Connector-male-female-ESC-Motor-PCB-board/32689137918.html" H 0   0   50  0001 C CNN "AliExpress Part Link"
-	1    5000 19950
-	1    0    0    -1
-$EndComp
-Text Label 4800 19350 2    60   ~ 0
+Text Label 5100 19350 2    60   ~ 0
 BAT_BAK_VCC
-Text Label 4800 19650 2    60   ~ 0
+Text Label 5100 19450 2    60   ~ 0
 BAT_VCC_CONN
-Text Label 4800 19950 2    60   ~ 0
+Text Label 5100 19650 2    60   ~ 0
 UMB_VCC
-$Comp
-L Power-Board-rescue:GND-power #PWR038
-U 1 1 5AA76884
-P 4800 19450
-F 0 "#PWR038" H 4800 19200 50  0001 C CNN
-F 1 "GND" V 4800 19250 50  0000 C CNN
-F 2 "" H 4800 19450 50  0001 C CNN
-F 3 "" H 4800 19450 50  0001 C CNN
-	1    4800 19450
-	0    1    -1   0
-$EndComp
 $Comp
 L Power-Board-rescue:GND-power #PWR039
 U 1 1 5AA76909
-P 4800 19750
-F 0 "#PWR039" H 4800 19500 50  0001 C CNN
-F 1 "GND" V 4800 19550 50  0000 C CNN
-F 2 "" H 4800 19750 50  0001 C CNN
-F 3 "" H 4800 19750 50  0001 C CNN
-	1    4800 19750
+P 5100 19250
+F 0 "#PWR039" H 5100 19000 50  0001 C CNN
+F 1 "GND" V 5100 19050 50  0000 C CNN
+F 2 "" H 5100 19250 50  0001 C CNN
+F 3 "" H 5100 19250 50  0001 C CNN
+	1    5100 19250
 	0    1    -1   0
 $EndComp
@@
 L Power-Board-rescue:GND-power #PWR040
 U 1 1 5AA7698E
-P 4800 20050
-F 0 "#PWR040" H 4800 19800 50  0001 C CNN
-F 1 "GND" V 4800 19850 50  0000 C CNN
-F 2 "" H 4800 20050 50  0001 C CNN
-F 3 "" H 4800 20050 50  0001 C CNN
-	1    4800 20050
+P 5100 19550
+F 0 "#PWR040" H 5100 19300 50  0001 C CNN
+F 1 "GND" V 5100 19350 50  0000 C CNN
+F 2 "" H 5100 19550 50  0001 C CNN
+F 3 "" H 5100 19550 50  0001 C CNN
+	1    5100 19550
 	0    1    -1   0
 $EndComp
@@
 	1    0    0    -1
 $EndComp
+$Comp
+L Connector:Screw_Terminal_01x06 J?
+U 1 1 5C4745D1
+P 5300 19350
+F 0 "J?" H 5380 19342 50  0000 L CNN
+F 1 "Screw_Terminal_01x06" H 5380 19251 50  0000 L CNN
+F 2 "" H 5300 19350 50  0001 C CNN
+F 3 "~" H 5300 19350 50  0001 C CNN
+	1    5300 19350
+	1    0    0    -1
+$EndComp

Commit message: Screw Terminals 4lyfe
Other:
- note added: "Mounting holes:\nM3 Screw holes.\n\nSymbol:\nThe sweet looking rocket logo on the back."
- note removed: "Mounting holes:\nM3 Screw holes.\n\nSymbol:\nThe rocket logo on the back."
Changed lines of the file:
@@
 Connectors:\nConnect to batteries and stuff
 Text Notes 1900 18800 0    50   ~ 0
-Mounting holes:\nM3 Screw holes.\n\nSymbol:\nThe rocket logo on the back.
+Mounting holes:\nM3 Screw holes.\n\nSymbol:\nThe sweet looking rocket logo on the back.
 Text Notes 2350 16300 0    50   ~ 0
 Connector:\n2x7 100mil header used to connect the different boards together
