File: Power Board/Power Board.sch (KiCad schematic (older format))
At the start: 148 parts, among them J1 Conn_02x03_Odd_Even, J6 Conn_01x02, J7 Conn_01x03, J8 Conn_02x07_Odd_Even, Q1 SI7157DP, Q2 SI7157DP, Q3 SI7157DP, Q4 SI7157DP, Q5 SI7157DP, Q6 SI7157DP, Q7 DMG2305UX, U1 LTC4417CGN, U10 LMR62014XMF, U11 TPS22810, U2 TPS564208DDCT, U3 LTC3130-1, U4 BQ2057WSNTR, U5 BQ29209DRBT, U6 LT6700CS6-1, U7 STS8C5H30L, U8 LTC4150, U9 ATxmega32E5-AU

Commit message: Made board bigger, started layout
Parts:
- J2: renamed from J?; footprint (none) -> Custom Parts:3PCV-06; Digikey Part Number (none) -> 3PCV-06-006-ND
Changed lines of the file:
@@
 	1    0    0    -1
 $EndComp
+Text Label 5100 19650 2    60   ~ 0
+VCC_IN
+Text Label 5100 19450 2    60   ~ 0
+BAT_BAK_VCC
 Text Label 5100 19150 2    60   ~ 0
-VCC_IN
+BAT_VCC_CONN
 Text Label 5100 19350 2    60   ~ 0
-BAT_BAK_VCC
-Text Label 5100 19450 2    60   ~ 0
-BAT_VCC_CONN
-Text Label 5100 19650 2    60   ~ 0
 UMB_VCC
 $Comp
@@
 $EndComp
 $Comp
-L Connector:Screw_Terminal_01x06 J?
+L Connector:Screw_Terminal_01x06 J2
 U 1 1 5C4745D1
 P 5300 19350
-F 0 "J?" H 5380 19342 50  0000 L CNN
+F 0 "J2" H 5380 19342 50  0000 L CNN
 F 1 "Screw_Terminal_01x06" H 5380 19251 50  0000 L CNN
-F 2 "" H 5300 19350 50  0001 C CNN
+F 2 "Custom Parts:3PCV-06" H 5300 19350 50  0001 C CNN
 F 3 "~" H 5300 19350 50  0001 C CNN
+F 4 "3PCV-06-006-ND" H 5300 19350 50  0001 C CNN "Digikey Part Number"
 	1    5300 19350
 	1    0    0    -1

Commit message: Started block layout
Parts:
- renumbered C11 to C10, C13 to C11, C14 to C12, C15 to C13, C16 to C14, C17 to C15, C18 to C16, C28 to C17, C29 to C18, C30 to C19, C19 to C20, C20 to C21, C21 to C22, C22 to C23, C23 to C24, C10 to C25, C12 to C26, C24 to C27, C25 to C28, C26 to C29, C27 to C30, D9 to D1, D14 to D10, D15 to D11, D16 to D12, D5 to D13, D6 to D14, D13 to D15, D8 to D16, D1 to D3, D10 to D4, D11 to D5, D3 to D6, D4 to D7, D7 to D8, D12 to D9, J8 to J1, J7 to J3, J6 to J4, J1 to J5, L5 to L3, L3 to L4, L4 to L5, R14 to R1, R6 to R10, R7 to R11, R8 to R12, R9 to R13, R30 to R14, R31 to R15, R32 to R16, R10 to R17, R11 to R18, R12 to R19, R15 to R2, R13 to R20, R57 to R21, R58 to R22, R59 to R23, R18 to R24, R19 to R25, R20 to R26, R21 to R27, R22 to R28, R23 to R29, R16 to R3, R24 to R30, R25 to R31, R26 to R32, R27 to R33, R28 to R34, R29 to R35, R33 to R36, R34 to R37, R35 to R38, R36 to R39, R17 to R4, R39 to R40, R40 to R41, R41 to R42, R42 to R43, R43 to R44, R44 to R45, R47 to R46, R48 to R47, R49 to R48, R50 to R49, R1 to R5, R51 to R50, R52 to R51, R53 to R52, R56 to R53, R37 to R54, R38 to R55, R45 to R56, R46 to R57, R54 to R58, R55 to R59, R2 to R6, R3 to R7, R4 to R8, R5 to R9, U8 to U10, U9 to U11, U10 to U4, U11 to U5, U4 to U6, U5 to U7, U6 to U8, U7 to U9
Other:
- moved on the sheet: U4
