File: Power Board/_autosave-Power Board.kicad_pcb (KiCad board)
At the start: 2 copper layers, 55.9 x 58.4 mm, 55 parts, among them J1 Conn_02x10_Odd_Even, J2 Conn_01x02, J3 Conn_01x02, J4 Conn_01x02, J5 Conn_01x02, Q1 SI7135DP, Q2 SI7135DP, Q3 SI7135DP, Q4 SI7135DP, Q5 SI7135DP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

Commit message: Removed Voltage sensing from main board, added 2 PTs
Other:
- board text added: "I'm aware this is bad"
