File: Power Board/Power Board.kicad_pcb (KiCad board)
At the start: 2 copper layers, 55 x 70 mm, 148 parts, among them J1 Conn_02x03_Odd_Even, J2 Screw_Terminal_01x06, J6 Conn_01x02, J7 Conn_01x03, J8 Conn_02x07_Odd_Even, Q1 SI7157DP, Q2 SI7157DP, Q3 SI7157DP, Q4 SI7157DP, Q5 SI7157DP, Q6 SI7157DP, Q7 DMG2305UX, U1 LTC4417CGN, U10 LMR62014XMF, U11 TPS22810, U2 TPS564208DDCT, U3 LTC3130-1, U4 BQ2057WSNTR, U5 BQ29209DRBT, U6 LT6700CS6-1, U7 STS8C5H30L, U8 LTC4150, U9 ATxmega32E5-AU

Commit message: Started block layout
Parts:
- removed the D8 at (302.9, 95.6)
- added D16: LED_G, LEDs:LED_0603, F.Cu at (382.1, 192.3)
- moved U8 176.5 mm to (436.1, 192.3)
- moved R35 175.9 mm to (455.1, 195.3)
- moved R33 173.5 mm to (449.1, 195.3)
- moved R34 173.3 mm to (455.1, 189.3)
- moved R32 170.6 mm to (449.1, 192.3)
- moved R31 167.2 mm to (449.1, 189.3)
- moved R28 166.9 mm to (444.1, 192.3)
- moved R29 164.6 mm to (444.1, 189.3)
- moved R30 163.6 mm to (444.1, 195.3)
- moved C24 159.8 mm to (429.1, 196.3)
- moved C23 159.4 mm to (429.1, 193.3)
- moved C22 158.5 mm to (429.1, 190.3)
- moved C21 155.3 mm to (429.1, 187.3)
- moved U5 155.0 mm to (445.5, 149.5)
- moved U7 154.6 mm to (422.1, 192.5)
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- renumbered C11 to C10, C13 to C11, C14 to C12, C15 to C13, C16 to C14, C17 to C15, C18 to C16, C28 to C17, C29 to C18, C30 to C19, C19 to C20, C20 to C21, C21 to C22, C22 to C23, C23 to C24, C10 to C25, C12 to C26, C24 to C27, C25 to C28, C26 to C29, C27 to C30, D9 to D1, D14 to D10, D15 to D11, D16 to D12, D5 to D13, D6 to D14, D13 to D15, D1 to D3, D10 to D4, D11 to D5, D3 to D6, D4 to D7, D7 to D8, D12 to D9, J8 to J1, J7 to J3, J6 to J4, J1 to J5, L5 to L3, L3 to L4, L4 to L5, R14 to R1, R6 to R10, R7 to R11, R8 to R12, R9 to R13, R30 to R14, R31 to R15, R32 to R16, R10 to R17, R11 to R18, R12 to R19, R15 to R2, R13 to R20, R57 to R21, R58 to R22, R59 to R23, R18 to R24, R19 to R25, R20 to R26, R21 to R27, R22 to R28, R23 to R29, R16 to R3, R24 to R30, R25 to R31, R26 to R32, R27 to R33, R28 to R34, R29 to R35, R33 to R36, R34 to R37, R35 to R38, R36 to R39, R17 to R4, R39 to R40, R40 to R41, R41 to R42, R42 to R43, R43 to R44, R44 to R45, R47 to R46, R48 to R47, R49 to R48, R50 to R49, R1 to R5, R51 to R50, R52 to R51, R53 to R52, R56 to R53, R37 to R54, R38 to R55, R45 to R56, R46 to R57, R54 to R58, R55 to R59, R2 to R6, R3 to R7, R4 to R8, R5 to R9, U8 to U10, U9 to U11, U10 to U4, U11 to U5, U4 to U6, U5 to U7, U6 to U8, U7 to U9
Connections:
- J1 pad 1: (no net) -> Net-(J1-Pad1)
- J1 pad 11: (no net) -> Net-(J1-Pad11)
- J1 pad 13: (no net) -> Net-(J1-Pad13)
- J1 pad 3: (no net) -> Net-(J1-Pad3)
- J1 pad 5: (no net) -> Net-(J1-Pad5)
- J1 pad 7: (no net) -> Net-(J1-Pad7)
- J1 pad 9: (no net) -> Net-(J1-Pad9)
- J5 pad 3: (no net) -> Net-(J5-Pad3)
- J5 pad 4: (no net) -> Net-(J5-Pad4)
- TH1 pad 1: (no net) -> Net-(TH1-Pad1)
- TH1 pad 2: (no net) -> Net-(TH1-Pad2)
- U1 pad 1: (no net) -> Net-(U1-Pad1)
- U1 pad 14: (no net) -> Net-(U1-Pad14)
- U11 pad 19: (no net) -> Net-(U11-Pad19)
- U2 pad 5: (no net) -> Net-(U2-Pad5)
- U3 pad 13: (no net) -> Net-(U3-Pad13)
- U5 pad 4: (no net) -> Net-(U5-Pad4)
- U5 pad 5: (no net) -> Net-(U5-Pad5)
- U8 pad 1: (no net) -> Net-(U8-Pad1)

Commit message: Finished grouping components
Parts:
- removed TH1: NXFT15XH103FA2B100, Custom Parts:Thermistor_Through_Hole_Tiny
- moved R45 116.6 mm to (374.1, 30.3)
- moved R40 107.2 mm to (364.1, 27.3)
- moved R44 105.4 mm to (369.1, 30.3)
- moved R53 103.5 mm to (369.1, 45.3)
- moved R42 100.7 mm to (374.1, 27.3)
- moved R49 100.2 mm to (364.1, 38.3)
- moved R52 97.6 mm to (369.1, 42.6)
- moved R43 95.7 mm to (364.1, 30.3)
- moved R41 93.5 mm to (369.1, 27.3)
- moved R47 92.5 mm to (369.1, 35.3)
- moved R48 92.2 mm to (374.1, 35.3)
- moved R51 86.5 mm to (374.1, 38.3)
- moved R50 81.9 mm to (369.1, 38.3)
- moved R58 81.0 mm to (372.1, 85.3)
- moved R54 79.6 mm to (372.1, 55.3), turned to 180 degrees
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
Commit message: Started routing of blocks
Parts:
- moved C20 25.9 mm to (360.7, 181.1), turned to 90 degrees
- moved R25 20.9 mm to (360.7, 183.9), turned to 270 degrees
- moved R27 18.7 mm to (359.1, 183.9), turned to 90 degrees
- moved R26 18.1 mm to (371.1, 182.9), turned to 180 degrees
- moved D16 13.6 mm to (371.1, 184.3), turned to 180 degrees
- moved U6 13.2 mm to (365.5, 182.5)
- moved R24 12.8 mm to (363.3, 177.5), turned to 180 degrees
- moved Q7 10.0 mm to (369.3, 177.5), turned to 180 degrees
Routing:
- net /BAT_CELL_2: track 0.00 -> 9.93 mm
- net /BAT_CHARGE_VCC: track 0.00 -> 9.08 mm
- net Net-(Q7-Pad3): track 0.00 -> 7.43 mm
- net Net-(Q7-Pad1): track 0.00 -> 4.56 mm
- net Net-(J4-Pad1): track 0.00 -> 3.80 mm
- net /CHARGE_STAT: track 0.00 -> 2.14 mm
- net Net-(D16-Pad1): track 0.00 -> 1.42 mm

Commit message: More blocks routed
Parts:
- moved U5 59.0 mm to (403.1, 108.5), turned to 180 degrees
- moved R22 18.6 mm to (409.4, 117.0), turned to 270 degrees
- moved C19 18.4 mm to (413.8, 110.5)
- moved R23 16.6 mm to (409.9, 113.2), turned to 180 degrees
- moved C18 14.6 mm to (411.1, 111.6)
- moved C14 14.4 mm to (333.4, 194.1), turned to 270 degrees
- moved L1 13.4 mm to (327.5, 145.5), turned to 90 degrees
- moved C26 13.2 mm to (405.1, 150.3), turned to 270 degrees
- moved C17 13.0 mm to (414.7, 116.9), turned to 90 degrees
- moved L3 12.6 mm to (421.0, 112.8), turned to 90 degrees
- moved D15 11.2 mm to (413.0, 108.5)
- moved C15 11.2 mm to (324.5, 193.9), turned to 270 degrees
- moved R21 11.0 mm to (412.6, 113.2)
- moved R37 10.3 mm to (402.4, 148.5), turned to 90 degrees
- moved D11 10.3 mm to (320.6, 191.6), turned to 90 degrees
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Routing:
- net /VCC_IN: track 0.00 -> 24.0 mm
- net /BAT_CELL_2: track 9.93 -> 28.6 mm
- net +3V3: track 0.00 -> 18.6 mm
- net Net-(D15-Pad2): track 0.00 -> 17.3 mm
- net Net-(C18-Pad1): track 0.00 -> 12.9 mm
- net Net-(C8-Pad2): track 0.00 -> 10.1 mm
- net Net-(C11-Pad2): track 0.00 -> 9.45 mm
- net GND: track 0.00 -> 9.22 mm
- net /UMB_VCC: track 0.00 -> 8.38 mm
- net Net-(C12-Pad1): track 0.00 -> 7.44 mm
- net /BAT_CELL_2_CONN: track 0.00 -> 6.89 mm
- net Net-(C18-Pad2): track 0.00 -> 5.27 mm
- net /LVL_POL: track 0.00 -> 3.60 mm
- net Net-(R17-Pad2): track 0.00 -> 3.50 mm
- net Net-(C11-Pad1): track 0.00 -> 2.94 mm
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
Commit message: Blocks blocks blocks
Parts:
- moved R35 64.4 mm to (392.8, 179.0), turned to 90 degrees
- moved R33 57.9 mm to (392.8, 181.6), turned to 90 degrees
- moved R31 47.6 mm to (402.1, 181.7), turned to 270 degrees
- moved R30 45.1 mm to (402.1, 178.9), turned to 270 degrees
- moved R34 40.2 mm to (416.2, 179.0), turned to 180 degrees
- moved R32 38.0 mm to (413.5, 179.0)
- moved R28 35.2 mm to (411.3, 179.5), turned to 90 degrees
- moved R29 34.2 mm to (410.7, 181.9), turned to 180 degrees
- moved L4 30.5 mm to (312.1, 98.3)
- moved C27 28.3 mm to (312.5, 96.2)
- moved C22 26.9 mm to (403.6, 181.7), turned to 270 degrees
- moved C24 26.9 mm to (405.9, 182.7)
- moved C21 26.9 mm to (403.6, 178.8), turned to 270 degrees
- moved U8 24.1 mm to (414.5, 181.7), turned to 180 degrees
- moved C23 23.7 mm to (409.8, 179.6), turned to 270 degrees
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Routing:
- net /BAT_CELL_2: track 28.6 -> 50.3 mm
- net Net-(R35-Pad1): track 0.00 -> 18.8 mm
- net /BAT_CELL_1: track 0.00 -> 10.3 mm
- net Net-(R33-Pad2): track 0.00 -> 8.24 mm
- net Net-(R29-Pad2): track 0.00 -> 6.75 mm
- net Net-(C28-Pad1): track 0.00 -> 6.74 mm
- net GND: track 9.22 -> 14.1 mm
- net Net-(C21-Pad2): track 0.00 -> 4.40 mm
- net Net-(C23-Pad1): track 0.00 -> 3.73 mm
- net Net-(C21-Pad1): track 0.00 -> 3.64 mm
- net Net-(C27-Pad2): track 0.00 -> 3.58 mm
- net Net-(R32-Pad2): track 0.00 -> 3.41 mm
- net Net-(C24-Pad1): track 0.00 -> 1.77 mm

Commit message: More changes
Parts:
- moved C28 51.9 mm to (368.7, 124.9)
- moved C29 51.9 mm to (378.7, 135.4)
- moved C30 51.9 mm to (368.7, 126.4)
- moved D17 51.9 mm to (369.2, 121.8)
- moved D18 51.9 mm to (380.1, 135.8)
- moved L4 51.9 mm to (357.4, 123.6)
- moved U11 51.9 mm to (372.6, 132.6)
- moved C27 51.9 mm to (357.8, 121.5)
- moved L5 51.9 mm to (368.8, 123.3)
- moved Q5 34.8 mm to (317.4, 18.4), turned to 180 degrees
- moved Q6 34.8 mm to (325.1, 18.4)
- moved Q4 34.5 mm to (325.1, 12.7)
- moved Q3 34.5 mm to (317.4, 12.7), turned to 180 degrees
- moved Q1 34.3 mm to (317.4, 7.03), turned to 180 degrees
- moved Q2 34.3 mm to (325.1, 7.03)
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Routing:
- net Net-(Q3-Pad2): track 0.00 -> 8.69 mm
- net Net-(Q5-Pad2): track 0.00 -> 8.68 mm
- net Net-(Q1-Pad2): track 0.00 -> 8.68 mm
- added copper zone on F.Cu, net Net-(C2-Pad1)
- added copper zone on F.Cu, net Net-(C3-Pad1)
- added copper zone on F.Cu, net Net-(C4-Pad1)
