File: Safing Remote/Safing Remote.sch (KiCad schematic (older format))
At the start: 4 parts

Commit message: Finished Safing Remote Schematic
Parts:
- removed U?: ATxmega32E5-AU, Package_QFP:TQFP-32_7x7mm_P0.8mm, symbol MCU_Microchip_ATmega:ATxmega32E5-AU
- removed U?: RFM95W-915S2, symbol RF_AM_FM:RFM95W-915S2
- added AE?: Antenna, symbol Device:Antenna
- added BT? (x2): Battery_Cell, symbol Device:Battery_Cell
- added C?: 0.1 µF, Capacitors_SMD:C_0805, symbol Device:C_Small
- added C?: 22 µF, Capacitors_SMD:C_0805, symbol Device:C_Small
- added C?: 47 µF, Capacitors_SMD:C_0805, symbol Device:C_Small
- added C? (x2): 0.1 µF, Capacitors_SMD:C_0603, symbol Device:C_Small
- added C? (x2): 10 µF, Capacitors_SMD:C_0603, symbol Device:C_Small
- added C?: 10 µF, Capacitors_SMD:C_0603, symbol Control-Board-rescue:C_Small-device
- added J?: Conn_Coaxial, symbol Connector:Conn_Coaxial
- added J?: Conn_02x03_Odd_Even, symbol Connector_Generic:Conn_02x03_Odd_Even
- added L?: 2.2 µH, symbol Device:L_Small
- added L?: 220 Ω @ 100 MHz, symbol Device:Ferrite_Bead_Small
- added L?: 10 µH, symbol Device:L_Small
- added R?: 33.2 kΩ, Resistors_SMD:R_0603, symbol Device:R_Small
- added R?: 10 kΩ, Resistors_SMD:R_0603, symbol Device:R_Small
- added R? (x7): 10 kΩ, symbol Device:R_Small
- added R?: 10 kΩ, Resistors_SMD:R_0603, symbol Control-Board-rescue:R_Small-device
- added R?: 121 kΩ, symbol Device:R_Small
- added SW?: SW_SPDT, symbol Switch:SW_SPDT
- added SW? (x5): SW_Push, symbol Switch:SW_Push
- added U?: TPS564208DDCT, TO_SOT_Packages_SMD:SOT-23-6, symbol Custom-Parts:TPS54308DDC
- added U?: ATxmega32E5-AU, Package_QFP:TQFP-32_7x7mm_P0.8mm, symbol MCU_Microchip_ATmega:ATxmega32E5-AU
- added U?: RFM95W-915S2, symbol RF_AM_FM:RFM96W-315S2
Connections:
- net labels added: +3V3, BEEP, GND, LCD_RX, LORA_CS, LORA_IRQ, LORA_RST, MISO1, MOSI1, SCK1, SW_DN, SW_EN, SW_LF, SW_RI, SW_UP, VCC_IN, VCC_IN_SENS
- wire segments 0 -> 73
- no-connect marks 0 -> 8
Other:
- note added: "3.3V dc-dc"
- note added: "Close to\npower supply"

Commit message: Little change
Other:
- note added: "Not mounted, just here so\nit shows up in the BOM"
Changed lines of the file:
@@
 Text Label 4050 5800 0    50   ~ 0
 LORA_RST
+Text Notes 10200 4700 0    50   ~ 0
+Not mounted, just here so\nit shows up in the BOM
 $EndSCHEMATC

Commit message: Started annotating, fixed a few errors
Parts:
- C?: symbol Control-Board-rescue:C_Small-device -> Device:C_Small
- R?: symbol Control-Board-rescue:R_Small-device -> Device:R_Small
- U?: symbol Custom-Parts:TPS54308DDC -> Custom_Parts:TPS54308DDC
Connections:
- wire segments 73 -> 71
Other:
- note added: "Beeper:\nLow power/volume buzzer to provide audible feedback."
- note added: "Button Array:\nUp, down, left, right, and enter buttons to control the remote"
- note added: "LCD Screen:\nConnector for the Sparkfun SerLCD. The actual module has more\nconnectors, this one is just the minimum required."
- note added: "MCU:\nATXMegaE5U to control all the functions.\nLow cost and small in order to\nminimize complexity."
- note added: "Power Supply:\nTakes in power from the two batteries and regulates it down to 3.3v. Uses\nthe same DC-DC converter as in the main power board, to minimize unique components.\ncomponents."
- note added: "RFM95 LoRa Module:\nLow power, long range radio to recieve communications from the backup\nradios in the rocket. Also cabable of sending commands to the rocket, if\nthat function is desired later"
- note added: "Voltage Divider:\nAllows the MCU to see if its batteries are dying"
Changed lines of the file:
@@
 EESchema Schematic File Version 4
-LIBS:Power Board-cache
-LIBS:Control Board-cache
+LIBS:Safing Remote-cache
 EELAYER 26 0
 EELAYER END
@@
 $EndComp
 $Comp
-L Custom-Parts:TPS54308DDC U?
+L Custom_Parts:TPS54308DDC U?
 U 1 1 5CA051C3
 P 2400 1200
@@
 	8950 4850 9350 4850
 $Comp
-L Control-Board-rescue:R_Small-device R?
-U 1 1 5CA53803
-P 7250 5250
-F 0 "R?" H 7280 5270 50  0000 L CNN
-F 1 "10 kΩ" H 7280 5210 50  0000 L CNN
-F 2 "Resistors_SMD:R_0603" H 7250 5250 50  0001 C CNN
-F 3 "" H 7250 5250 50  0001 C CNN
-F 4 "311-10.0KHRCT-ND" H 7280 5370 50  0001 C CNN "Digikey Part Number"
-	1    7250 5250
-	-1   0    0    1
-$EndComp
-Wire Wire Line
-	7950 5350 7250 5350
-Connection ~ 7250 5350
-Wire Wire Line
-	7250 5350 6950 5350
-$Comp
 L power:+3V3 #PWR?
 U 1 1 5CA5380D
@@
 	1    0    0    -1
 $EndComp
-Wire Wire Line
-	8450 4450 8450 4500
 $Comp
 L power:+3V3 #PWR?
@@
 NoConn ~ 8950 5050
 $Comp
-L Control-Board-rescue:C_Small-device C?
+L Device:C_Small C?
 U 1 1 5CA53822
 P 8350 4500
@@
 	0    -1   1    0
 $EndComp
-Connection ~ 8450 4500
-Wire Wire Line
-	8450 4500 8450 4650
 $Comp
 L power:GND #PWR?
@@
 Text Notes 10200 4700 0    50   ~ 0
 Not mounted, just here so\nit shows up in the BOM
+Text Notes 3400 800  0    50   ~ 0
+Power Supply:\nTakes in power from the two batteries and regulates it down to 3.3v. Uses\nthe same DC-DC converter as in the main power board, to minimize unique components.\ncomponents.
+Text Notes 5100 1600 0    50   ~ 0
+Beeper:\nLow power/volume buzzer to provide audible feedback.
+Text Notes 7800 700  0    50   ~ 0
+Button Array:\nUp, down, left, right, and enter buttons to control the remote
+Text Notes 4950 3250 0    50   ~ 0
+LCD Screen:\nConnector for the Sparkfun SerLCD. The actual module has more\nconnectors, this one is just the minimum required.
+Text Notes 7200 4300 0    50   ~ 0
+RFM95 LoRa Module:\nLow power, long range radio to recieve communications from the backup\nradios in the rocket. Also cabable of sending commands to the rocket, if\nthat function is desired later
+Text Notes 1050 4250 0    50   ~ 0
+MCU:\nATXMegaE5U to control all the functions.\nLow cost and small in order to\nminimize complexity.
+Text Notes 4750 5100 0    50   ~ 0
+Voltage Divider:\nAllows the MCU to see if its batteries are dying
+Wire Wire Line
+	6950 5350 7950 5350
+Wire Wire Line
+	8450 4450 8450 4650
+$Comp
+L Device:R_Small R?
+U 1 1 5CA53803
+P 7250 5250
+F 0 "R?" H 7280 5270 50  0000 L CNN
+F 1 "10 kΩ" H 7280 5210 50  0000 L CNN
+F 2 "Resistors_SMD:R_0603" H 7250 5250 50  0001 C CNN
+F 3 "" H 7250 5250 50  0001 C CNN
+F 4 "311-10.0KHRCT-ND" H 7280 5370 50  0001 C CNN "Digikey Part Number"
+	1    7250 5250
+	-1   0    0    1
+$EndComp
 $EndSCHEMATC

Commit message: Annotated Power Board Schematic
Other:
- note added: "Keep this trace\nshort and straight"
Changed lines of the file:
@@
 L Connector:Conn_Coaxial J?
 U 1 1 5C9B849C
-P 9550 4850
-F 0 "J?" H 9649 4826 50  0000 L CNN
-F 1 "Conn_Coaxial" H 9649 4735 50  0000 L CNN
-F 2 "" H 9550 4850 50  0001 C CNN
-F 3 " ~" H 9550 4850 50  0001 C CNN
-F 4 "CONSMA002-L-ND" H 9550 4850 50  0001 C CNN "Digikey Part Number"
-	1    9550 4850
+P 9800 4850
+F 0 "J?" H 9899 4826 50  0000 L CNN
+F 1 "Conn_Coaxial" H 9899 4735 50  0000 L CNN
+F 2 "" H 9800 4850 50  0001 C CNN
+F 3 " ~" H 9800 4850 50  0001 C CNN
+F 4 "CONSMA002-L-ND" H 9800 4850 50  0001 C CNN "Digikey Part Number"
+	1    9800 4850
 	1    0    0    -1
 $EndComp
@@
 	1    0    0    -1
 $EndComp
-Wire Wire Line
-	8950 4850 9350 4850
 $Comp
 L power:+3V3 #PWR?
@@
 L power:GND #PWR?
 U 1 1 5CA8ABAA
-P 9550 5050
-F 0 "#PWR?" H 9550 4800 50  0001 C CNN
-F 1 "GND" H 9550 4900 50  0000 C CNN
-F 2 "" H 9550 5050 50  0001 C CNN
-F 3 "" H 9550 5050 50  0001 C CNN
-	1    9550 5050
+P 9800 5050
+F 0 "#PWR?" H 9800 4800 50  0001 C CNN
+F 1 "GND" H 9800 4900 50  0000 C CNN
+F 2 "" H 9800 5050 50  0001 C CNN
+F 3 "" H 9800 5050 50  0001 C CNN
+	1    9800 5050
 	1    0    0    -1
 $EndComp
@@
 	-1   0    0    1
 $EndComp
+Text Notes 9150 4750 0    50   ~ 0
+Keep this trace\nshort and straight
+Wire Wire Line
+	8950 4850 9600 4850
 $EndSCHEMATC
