File: HotfireComms/HotfireComms.sch (KiCad schematic (older format))
At the start: 21 parts

Commit message: Fixed hotfire comms board shematic
Parts:
- removed H? (x3): Mounting_Hole, Mounting_Holes:MountingHole_3.2mm_M3, symbol Control-Board-rescue:Mounting_Hole-Mechanical
- added H? (x3): Mounting_Hole, Mounting_Holes:MountingHole_3.2mm_M3, symbol Mechanical:MountingHole
- C? (x3): symbol Control-Board-rescue:C_Small-device -> Device:C_Small
- D? (x2): symbol Control-Board-rescue:LED-device -> Device:LED
- H?: symbol Control-Board-rescue:Mounting_Hole-Mechanical -> Mechanical:MountingHole
- J?: symbol Control-Board-rescue:RJ45-Connector -> Connector:RJ45_Shielded
- J?: symbol Custom-Parts:Micro_SD_Card_SPI_MODE_Det -> Custom_Parts:Micro_SD_Card_SPI_MODE_Det
- R?: symbol Control-Board-rescue:R-device -> Device:R
- R?: symbol Control-Board-rescue:R_Small-device -> Device:R_Small
- U?: symbol Custom-Parts:ISL83490 -> Custom_Parts:ISL83490
Changed lines of the file:
@@
 EESchema Schematic File Version 4
-LIBS:Control Board-cache
+LIBS:HotfireComms-cache
 EELAYER 26 0
 EELAYER END
-$Descr A4 11693 8268
+$Descr A3 16535 11693
 encoding utf-8
 Sheet 1 1
@@
 $EndDescr
 $Comp
-L Custom-Parts:ISL83490 U?
+L Custom_Parts:ISL83490 U?
 U 1 1 5C733F14
 P 8150 5300
@@
 $EndComp
 $Comp
-L Control-Board-rescue:R-device R?
+L Device:R R?
 U 1 1 5C733F1C
 P 8900 5000
@@
 $EndComp
 $Comp
-L Control-Board-rescue:C_Small-device C?
+L Device:C_Small C?
 U 1 1 5C733F24
 P 7650 4500
@@
 L power:GND #PWR?
 U 1 1 5C733F5F
-P 10600 2150
-F 0 "#PWR?" H 10600 1900 50  0001 C CNN
-F 1 "GND" V 10600 1950 50  0000 C CNN
-F 2 "" H 10600 2150 50  0001 C CNN
-F 3 "" H 10600 2150 50  0001 C CNN
-	1    10600 2150
-	0    -1   1    0
-$EndComp
-$Comp
-L Control-Board-rescue:RJ45-Connector J?
+P 9500 2550
+F 0 "#PWR?" H 9500 2300 50  0001 C CNN
+F 1 "GND" V 9500 2350 50  0000 C CNN
+F 2 "" H 9500 2550 50  0001 C CNN
+F 3 "" H 9500 2550 50  0001 C CNN
+	1    9500 2550
+	0    1    -1   0
+$EndComp
+$Comp
+L Connector:RJ45_Shielded J?
 U 1 1 5C733F66
-P 10050 2500
-F 0 "J?" H 10126 3117 50  0000 C CNN
-F 1 "RJ45" H 10126 3026 50  0000 C CNN
-F 2 "Connectors:RJ45_8" H 10050 2500 50  0001 C CNN
-F 3 "" H 10050 2500 50  0001 C CNN
-F 4 "RJHSE-5080-ND" H -2100 -9700 50  0001 C CNN "Digikey Part Number"
-	1    10050 2500
-	1    0    0    -1
+P 10000 2550
+F 0 "J?" H 10076 3167 50  0000 C CNN
+F 1 "RJ45" H 10076 3076 50  0000 C CNN
+F 2 "Connectors:RJ45_8" H 10000 2550 50  0001 C CNN
+F 3 "" H 10000 2550 50  0001 C CNN
+F 4 "RJHSE-5080-ND" H -2150 -9650 50  0001 C CNN "Digikey Part Number"
+	1    10000 2550
+	0    1    1    0
 $EndComp
 $Comp
@@
 $EndComp
 $Comp
-L Control-Board-rescue:R_Small-device R?
+L Device:R_Small R?
 U 1 1 5C733F8D
 P 9450 950
@@
 $EndComp
 $Comp
-L Control-Board-rescue:Mounting_Hole-Mechanical H?
-U 1 1 5C733F97
-P 8150 1500
-F 0 "H?" H 8250 1546 50  0000 L CNN
-F 1 "Mounting_Hole" H 8250 1455 50  0000 L CNN
-F 2 "Mounting_Holes:MountingHole_3.2mm_M3" H 8150 1500 50  0001 C CNN
-F 3 "" H 8150 1500 50  0001 C CNN
-	1    8150 1500
-	1    0    0    -1
-$EndComp
-$Comp
-L Control-Board-rescue:Mounting_Hole-Mechanical H?
-U 1 1 5C733F9E
-P 8150 1700
-F 0 "H?" H 8250 1746 50  0000 L CNN
-F 1 "Mounting_Hole" H 8250 1655 50  0000 L CNN
-F 2 "Mounting_Holes:MountingHole_3.2mm_M3" H 8150 1700 50  0001 C CNN
-F 3 "" H 8150 1700 50  0001 C CNN
-	1    8150 1700
-	1    0    0    -1
-$EndComp
-$Comp
-L Control-Board-rescue:Mounting_Hole-Mechanical H?
-U 1 1 5C733FA5
-P 8150 1900
-F 0 "H?" H 8250 1946 50  0000 L CNN
-F 1 "Mounting_Hole" H 8250 1855 50  0000 L CNN
-F 2 "Mounting_Holes:MountingHole_3.2mm_M3" H 8150 1900 50  0001 C CNN
-F 3 "" H 8150 1900 50  0001 C CNN
-	1    8150 1900
-	1    0    0    -1
-$EndComp
-$Comp
-L Control-Board-rescue:Mounting_Hole-Mechanical H?
+L Mechanical:MountingHole H?
 U 1 1 5C733FAC
 P 8150 2100
@@
 $EndComp
 $Comp
-L Custom-Parts:Micro_SD_Card_SPI_MODE_Det J?
+L Custom_Parts:Micro_SD_Card_SPI_MODE_Det J?
 U 1 1 5C733FCB
 P 3350 2000
@@
 $EndComp
 $Comp
-L Control-Board-rescue:C_Small-device C?
+L Device:C_Small C?
 U 1 1 5C73401B
 P 1900 4000
@@
 SD_MISO
 $Comp
-L Control-Board-rescue:C_Small-device C?
+L Device:C_Small C?
 U 1 1 5C734038
 P 1750 4000
@@
 $EndComp
 $Comp
-L Control-Board-rescue:LED-device D?
+L Device:LED D?
 U 1 1 5C734060
 P 3900 6850
@@
 $EndComp
 $Comp
-L Control-Board-rescue:LED-device D?
+L Device:LED D?
 U 1 1 5C734068
 P 4300 6850
@@
 Wire Wire Line
 	7650 5000 7200 5000
+$Comp
+L Mechanical:MountingHole H?
+U 1 1 5BFBC168
+P 8150 1850
+F 0 "H?" H 8250 1896 50  0000 L CNN
+F 1 "Mounting_Hole" H 8250 1805 50  0000 L CNN
+F 2 "Mounting_Holes:MountingHole_3.2mm_M3" H 8150 1850 50  0001 C CNN
+F 3 "" H 8150 1850 50  0001 C CNN
+	1    8150 1850
+	1    0    0    -1
+$EndComp
+$Comp
+L Mechanical:MountingHole H?
+U 1 1 5BFBC19E
+P 8150 1600
+F 0 "H?" H 8250 1646 50  0000 L CNN
+F 1 "Mounting_Hole" H 8250 1555 50  0000 L CNN
+F 2 "Mounting_Holes:MountingHole_3.2mm_M3" H 8150 1600 50  0001 C CNN
+F 3 "" H 8150 1600 50  0001 C CNN
+	1    8150 1600
+	1    0    0    -1
+$EndComp
+$Comp
+L Mechanical:MountingHole H?
+U 1 1 5BFBC1D5
+P 8150 1350
+F 0 "H?" H 8250 1396 50  0000 L CNN
+F 1 "Mounting_Hole" H 8250 1305 50  0000 L CNN
+F 2 "Mounting_Holes:MountingHole_3.2mm_M3" H 8150 1350 50  0001 C CNN
+F 3 "" H 8150 1350 50  0001 C CNN
+	1    8150 1350
+	1    0    0    -1
+$EndComp
 $EndSCHEMATC

Commit message: Added FT232RL to hotfire comms board to allow it to be used at AGC end
AGC = Avionics Ground Station
Parts:
- added C? (x2): 0.1 uF, Capacitors_SMD:C_0603, symbol Device:C_Small
- added C?: 10 uF, Capacitors_SMD:C_0603, symbol Device:C_Small
- added C? (x2): 47 pF, Capacitors_SMD:C_0603, symbol Device:C_Small
- added D?: LED_G, LEDs:LED_0603, symbol Device:LED
- added D?: LED_R, LEDs:LED_0603, symbol Device:LED
- added J?: USB_B_Micro, symbol Connector:USB_B_Micro
- added R? (x2): 27 Ω, symbol Device:R_Small
- added R? (x2): 1 kΩ, symbol Device:R_Small
- added U?: FT232RL, Package_SO:SSOP-28_5.3x10.2mm_P0.65mm, symbol Interface_USB:FT232RL
- C? (x3): Digikey Part Number 445-5667-1-ND -> 1276-6717-6-ND
- J?: Digikey Part Number (none) -> 952-2219-ND
- J?: Digikey Part Number (none) -> WM24066CT-ND
- R?: Digikey Part Number 311-100HRCT-ND -> P100KHCT-ND
- R?: Digikey Part Number 311-10.0KHRCT-ND -> P10.0KHCT-ND
- R?: Digikey Part Number (none) -> P10.0KHCT-ND
- R?: Digikey Part Number (none) -> P1.00KHCT-ND
- R?: Digikey Part Number (none) -> P330HCT-ND
Connections:
- net labels added: +5V
- wire segments 47 -> 87
- no-connect marks 2 -> 14

Commit message: *AGS not AGC
Parts:
- gave numbers to parts that had none: 34
Connections:
- net labels added: AGS_RX, AGS_RX+, AGS_RX-, AGS_TX, AGS_TX+, AGS_TX-
- net labels removed: GSE_RX, GSE_RX+, GSE_RX-, GSE_TX, GSE_TX+, GSE_TX-

Commit message: Added some footprints to Hotfire Comms board
Parts:
- J1: footprint (none) -> Pin_Headers:Pin_Header_Straight_1x07_Pitch2.54mm
- R3, R4, R5, R6, R7, R8, R9: footprint (none) -> Resistors_SMD:R_0603
Changed lines of the file:
@@
 F 0 "J1" H 10250 1867 50  0000 C CNN
 F 1 "Conn_02x07_Counter_Clockwise" H 10250 1776 50  0000 C CNN
-F 2 "" H 10200 1350 50  0001 C CNN
+F 2 "Pin_Headers:Pin_Header_Straight_1x07_Pitch2.54mm" H 10200 1350 50  0001 C CNN
 F 3 "~" H 10200 1350 50  0001 C CNN
 F 4 "952-2219-ND" H 0   0   50  0001 C CNN "Digikey Part Number"
@@
 F 0 "R3" H 4559 5646 50  0000 L CNN
 F 1 "10 kΩ" H 4559 5555 50  0000 L CNN
-F 2 "" H 4500 5600 50  0001 C CNN
+F 2 "Resistors_SMD:R_0603" H 4500 5600 50  0001 C CNN
 F 3 "~" H 4500 5600 50  0001 C CNN
 F 4 "P10.0KHCT-ND" H 0   0   50  0001 C CNN "Digikey Part Number"
@@
 F 0 "R5" H 4359 6646 50  0000 L CNN
 F 1 "1 kΩ" H 4359 6555 50  0000 L CNN
-F 2 "" H 4300 6600 50  0001 C CNN
+F 2 "Resistors_SMD:R_0603" H 4300 6600 50  0001 C CNN
 F 3 "~" H 4300 6600 50  0001 C CNN
 F 4 "P1.00KHCT-ND" H 0   0   50  0001 C CNN "Digikey Part Number"
@@
 F 0 "R4" H 3959 6646 50  0000 L CNN
 F 1 "330 Ω" H 3959 6555 50  0000 L CNN
-F 2 "" H 3900 6600 50  0001 C CNN
+F 2 "Resistors_SMD:R_0603" H 3900 6600 50  0001 C CNN
 F 3 "~" H 3900 6600 50  0001 C CNN
 F 4 "P330HCT-ND" H 0   0   50  0001 C CNN "Digikey Part Number"
@@
 F 0 "R6" V 8404 8400 50  0000 C CNN
 F 1 "27 Ω" V 8495 8400 50  0000 C CNN
-F 2 "" H 8600 8400 50  0001 C CNN
+F 2 "Resistors_SMD:R_0603" H 8600 8400 50  0001 C CNN
 F 3 "~" H 8600 8400 50  0001 C CNN
 	1    8600 8400
@@
 F 0 "R7" V 8800 8500 50  0000 C CNN
 F 1 "27 Ω" V 8700 8500 50  0000 C CNN
-F 2 "" H 8600 8500 50  0001 C CNN
+F 2 "Resistors_SMD:R_0603" H 8600 8500 50  0001 C CNN
 F 3 "~" H 8600 8500 50  0001 C CNN
 	1    8600 8500
@@
 F 0 "R8" H 11159 8746 50  0000 L CNN
 F 1 "1 kΩ" H 11159 8655 50  0000 L CNN
-F 2 "" H 11100 8700 50  0001 C CNN
+F 2 "Resistors_SMD:R_0603" H 11100 8700 50  0001 C CNN
 F 3 "~" H 11100 8700 50  0001 C CNN
 F 4 "P1.00KHCT-ND" H 6800 2100 50  0001 C CNN "Digikey Part Number"
@@
 F 0 "R9" H 11459 8746 50  0000 L CNN
 F 1 "1 kΩ" H 11459 8655 50  0000 L CNN
-F 2 "" H 11400 8700 50  0001 C CNN
+F 2 "Resistors_SMD:R_0603" H 11400 8700 50  0001 C CNN
 F 3 "~" H 11400 8700 50  0001 C CNN
 F 4 "P1.00KHCT-ND" H 7100 2100 50  0001 C CNN "Digikey Part Number"

Commit message: Apparently connector footprints are odd-even by default, not counterclockwise
Parts:
- J1: value Conn_02x07_Counter_Clockwise -> Conn_02x07_Odd_Even; symbol Connector_Generic:Conn_02x07_Counter_Clockwise -> Connector_Generic:Conn_02x07_Odd_Even
Changed lines of the file:
@@
 $EndComp
 $Comp
-L Connector_Generic:Conn_02x07_Counter_Clockwise J1
+L Connector_Generic:Conn_02x07_Odd_Even J1
 U 1 1 5C733FBB
 P 10200 1350
 F 0 "J1" H 10250 1867 50  0000 C CNN
-F 1 "Conn_02x07_Counter_Clockwise" H 10250 1776 50  0000 C CNN
+F 1 "Conn_02x07_Odd_Even" H 10250 1776 50  0000 C CNN
 F 2 "Pin_Headers:Pin_Header_Straight_1x07_Pitch2.54mm" H 10200 1350 50  0001 C CNN
 F 3 "~" H 10200 1350 50  0001 C CNN
